File: HW/cross_band_handy_walkie_talkie_V1/cross_band_handy_walkie_talkie_V1.kicad_sch (KiCad schematic)
At the start: 29 parts

Commit message: F
Parts:
- added C10, C7, C8, C9: DNP, Capacitor_SMD:C_0603_1608Metric_Pad1.08x0.95mm_HandSolder, symbol Device:C_Small
- added J2, J3: Conn_Coaxial, Connector_Coaxial:SMA_Amphenol_901-144_Vertical, symbol Connector:Conn_Coaxial
- added R10, R11: filter, Resistor_SMD:R_1206_3216Metric_Pad1.30x1.75mm_HandSolder, symbol Device:R_Small
- added U3, U4: SA818S, Z_mycustom_footprint_lib:SA818S, symbol My_custom_lib:SA818S
- gave numbers to parts that had none: 28
Connections:
- net GPIO_37 is gone; now on net H/L2: U2.30 (SPIDQS/GPIO37/FSPIQ/SUBSPIQ)
- net GPIO_38 is gone; now on net PD2: U2.31 (GPIO38/FSPIWP/SUBSPIWP)
- net GPIO_39 is gone; now on net PTT2: U2.32 (MTCK/GPIO39/CLK_OUT3/SUBSPICS1)
- net +5V: now also U3.8 (VBATT), U4.8 (VBATT)
- net GND: now also C10.2, C7.2, C8.2, C9.2, J2.2 (Ext), J3.2 (Ext), U3.10 (GND), U3.9 (GND), U4.10 (GND), U4.9 (GND)
- net GPIO_11 renamed TX1
- net TX1: now also U3.16 (RXD_(RX))
- net GPIO_12 renamed RX1
- net RX1: now also U3.17 (TXD(TX))
- net GPIO_13 renamed PTT2
- net PTT2: now also U4.5 (PTT)
- net GPIO_14 renamed PD2
- net PD2: now also U4.6 (PD)
- net GPIO_15 renamed H/L2
- net H/L2: now also U4.7 (H/L)
- net GPIO_35 renamed RX2
- net RX2: now also U4.17 (TXD(TX))
- net GPIO_36 renamed TX2
- net TX2: now also U4.16 (RXD_(RX))
- net GPIO_40 renamed H/L1
- net H/L1: now also U3.7 (H/L)
- net GPIO_41 renamed PD1
- net PD1: now also U3.6 (PD)
- net GPIO_42 renamed PTT1
- net PTT1: now also U3.5 (PTT)
- new net: C9.1, R11.1, U4.12 (ANT)
- new net: C7.1, R10.1, U3.12 (ANT)
- new net: C8.1, J2.1 (In), R10.2
- new net: C10.1, J3.1 (In), R11.2
Other:
- moved on the sheet: C11, C12, C2, C3, C4, C5, C6, D1, D2, Q1A, Q1B, R12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

Commit message: h
Parts:
- added C14, C16, C18: 1u, Capacitor_SMD:C_0603_1608Metric_Pad1.08x0.95mm_HandSolder, symbol Device:C_Small
- added C15, C28, C29: 10u, Capacitor_SMD:C_0603_1608Metric_Pad1.08x0.95mm_HandSolder, symbol Device:C_Small
- added C17, C19, C22: 1uF, Capacitor_SMD:C_0805_2012Metric, symbol Device:C
- added C20: 1nF, Capacitor_SMD:C_0805_2012Metric, symbol Device:C
- added C21: 10uF, Capacitor_SMD:C_0805_2012Metric, symbol Device:C
- added C23: 1u-10u?, Capacitor_SMD:C_0603_1608Metric_Pad1.08x0.95mm_HandSolder, symbol Device:C_Small
- added C24: 47n, Capacitor_SMD:C_0603_1608Metric_Pad1.08x0.95mm_HandSolder, symbol Device:C_Small
- added C25: 47nF, Capacitor_SMD:C_0805_2012Metric, symbol Device:C
- added C26, C27: 4u7, Capacitor_SMD:C_0603_1608Metric_Pad1.08x0.95mm_HandSolder, symbol Device:C_Small
- added R14: 10, Resistor_SMD:R_0603_1608Metric_Pad0.98x0.95mm_HandSolder, symbol Device:R_Small
- added R15: 10R, Resistor_SMD:R_0805_2012Metric, symbol Device:R
- added RV1, RV2, RV3: 10k, Potentiometer_SMD:Potentiometer_Vishay_TS53YL_Vertical, symbol Device:R_POT
- added U5: LM386, symbol Amplifier_Audio:LM386
- added U6: LM386, Package_SO:SOIC-8_3.9x4.9mm_P1.27mm, symbol Amplifier_Audio:LM386
- added U7: LT1129-3.3_SO8, Package_SO:SOIC-8_3.9x4.9mm_P1.27mm, symbol Regulator_Linear:LT1129-3.3_SO8
- added U8: MAX9814, Package_DFN_QFN:DFN-14-1EP_3x3mm_P0.4mm_EP1.78x2.35mm, symbol Amplifier_Audio:MAX9814
Connections:
- net +3V3: now also C27.1, U7.1 (OUT), U7.2 (SENSE)
- net +5V: now also C15.1, C26.1, C28.2, C29.2, U5.6 (V+), U7.8 (IN)
- net GND: now also C14.2, C15.2, C20.2, C21.2, C24.2, C25.2, C26.2, C27.2, C28.1, C29.1, RV1.3, RV2.3, U5.2 (-), U5.4 (GND), U6.2 (-), U6.4 (GND), U7.3 (GND), U7.6 (GND), U7.7 (GND)
- net MIC_OUT: now reaches U3.18 (MIC_IN)
- net MIC_OUT: now also U4.18 (MIC_IN), C18.2
- new net: C22.1, U6.1 (GAIN)
- new net: C22.2, U6.8 (GAIN)
- new net: RV3.1, U5.1 (GAIN)
- new net: RV1.2, U5.3 (+)
- new net: C18.1, R14.2, U5.5
- new net: C14.1, U5.7 (BYPASS)
- new net: C23.1, U5.8 (GAIN)
- new net: C24.1, R14.1
- new net: C25.1, R15.2
- new net: U8.11 (GND), U8.15 (GND), U8.4 (GND), U8.7 (GND)
- new net: C20.1, RV2.2, U6.3 (+)
- new net: C21.1, U6.7 (BYPASS)
- new net: C16.2, RV1.1
- new net: C17.2, RV2.1
- new net: C19.1, R15.1, U6.5
- new net: C23.2, RV3.2
- new net AF_TRX: C17.1
- new net MIC_IN: C16.1
- new net SPKR: C19.2
- new net VCC: U6.6 (V+)
- no-connect marks 3 -> 4
Other:
- note added: "750mA max current"
- note added: "SPEAKER AMP"
- moved on the sheet: C1, C10, C2, C3, C4, C5, C6, C7, C8, C9, D1, D2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

Commit message: b
Parts:
- removed C10, C7, C8, C9: DNP, Capacitor_SMD:C_0603_1608Metric_Pad1.08x0.95mm_HandSolder, symbol Device:C_Small
- removed J2: Conn_Coaxial, Connector_Coaxial:SMA_Amphenol_901-144_Vertical, symbol Connector:Conn_Coaxial
- removed R10, R11: filter, Resistor_SMD:R_1206_3216Metric_Pad1.30x1.75mm_HandSolder, symbol Device:R_Small
- added C10: 2.2uF, Capacitor_SMD:C_0805_2012Metric, symbol Device:C
- added C30: 1uF, Capacitor_SMD:C_0805_2012Metric, symbol Device:C
- added C7, C8: 100nF, Capacitor_SMD:C_0805_2012Metric, symbol Device:C
- added C9: 470nF, Capacitor_SMD:C_0805_2012Metric, symbol Device:C
- added FL? (x2): LFCN-160, Filter:Filter_Mini-Circuits_FV1206, symbol RF_Filter:LFCN-160
- added J4, J5: Conn_01x03, Connector_PinHeader_2.54mm:PinHeader_1x03_P2.54mm_Vertical, symbol Connector_Generic:Conn_01x03
- added J6: Conn_01x03, Jumper:SolderJumper-3_P2.0mm_Open_TrianglePad1.0x1.5mm_NumberLabels, symbol Connector_Generic:Conn_01x03
- added J? (x6): pin, Connector_PinHeader_2.54mm:PinHeader_1x01_P2.54mm_Vertical, symbol Connector_Generic:Conn_01x01
- added J?: Conn_Coaxial, Connector_Coaxial:SMA_Amphenol_901-144_Vertical, symbol Connector:Conn_Coaxial
- added L1: Ferrit, Resistor_SMD:R_0805_2012Metric_Pad1.20x1.40mm_HandSolder, symbol Device:L
- added R16: #2.2k, Resistor_SMD:R_0805_2012Metric, symbol Device:R
- added R17: 150k, Resistor_SMD:R_0805_2012Metric, symbol Device:R
- added R18: 1k, Resistor_SMD:R_0805_2012Metric, symbol Device:R
- added R19: 100k, Resistor_SMD:R_0805_2012Metric, symbol Device:R
- added U? (x8): TS5A63157DBV, Package_TO_SOT_SMD:SOT-23-6, symbol Analog_Switch:TS5A63157DBV
- U8: LCSC (none) -> C41714
Connections:
- net +3V3: now also J4.3 (Pin_3), J5.3 (Pin_3), L1.1
- net AF_TRX: no longer C17.1
- net GND: now also U8.11 (GND), U8.13 (MICBIAS), U8.15 (GND), U8.4 (GND), U8.7 (GND), U8.8 (MICIN), C10.2, C30.1, C7.1, C8.1, C9.2, FL?.2 (GND), FL?.2 (GND), FL?.4 (GND), FL?.4 (GND), J4.1 (Pin_1), J5.1 (Pin_1), J?.2 (Ext), R16.1, R17.1, R19.2
- net MIC_IN: now also J?.1 (Pin_1), U?.4, U?.4; no longer C16.1
- net at U4.12 (ANT): now also FL?.1 (IN)
- net at U3.12 (ANT): now also FL?.1 (IN)
- net at U3.3 (AF(Audio_OUT)): now also U?.3
- net at U4.3 (AF(Audio_OUT)): now also U?.1
- net at J3.1 (In): now also FL?.3 (OUT)
- net at U8.1 (CT): now also C7.2
- net at U8.10 (GAIN): now also R18.1
- net at U8.12 (BIAS): now also C9.1
- net at U8.14 (TH): now also R17.2, R19.1
- net -SLEEP: now reaches U8.2 (~{SHDN})
- net at U8.3 (CG): now also C10.1
- net at U8.5 (VDD): now also C30.2, L1.2
- net at U8.6 (MICOUT): now also J6.1 (Pin_1), J?.1 (Pin_1), U?.3
- net MIC_AR: now reaches U8.9 (A/R)
- net MIC_AR: now also J5.2 (Pin_2)
- removed net MIC_OUT: C18.2, U3.18 (MIC_IN), U4.18 (MIC_IN)
- new net: U3.18 (MIC_IN), U?.1
- new net: U4.18 (MIC_IN), U?.3
- new net: FL?.3 (OUT), J?.1 (In)
- new net AUDIO_IN: C16.1, J?.1 (Pin_1), U?.4
- new net AUDIO_OUT: C18.2, J?.1 (Pin_1), U?.3, U?.4
- new net MIC-AMP_IN: C8.2, R16.2
- new net MIC-DIGI_IN: J6.3 (Pin_3)
- new net MIC_GAIN: J4.2 (Pin_2), R18.2
- new net TRX_MIC: J6.2 (Pin_2)
- new net esp audio: J?.1 (Pin_1), J?.1 (Pin_1), U?.1, U?.1
Other:
- note added: "???"
- note added: "MIC AMP"
- note added: "VDD: 1:2000 NC: 1:4000 GND: 1:500"
- note added: "VDD: 40dB NC: 60dB GND: 50dB"
- moved on the sheet: C1, C11, C12, C13, C14, C15, C16, C17, C18, C19, C20, C21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

Commit message: Update cross_band_handy_walkie_talkie_V1.kicad_sch
Parts:
- removed U2: ESP32-S3-WROOM-1, Espressif:ESP32-S3-WROOM-1, symbol Espressif:ESP32-S3-WROOM-1
- added U?: ESP32-A1S_, symbol My_custom_lib:ESP32-A1S_
Other:
- note added: "danger pins: IO_0 IO_2"
Changed lines of the file:
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@@
     (stroke (width 0) (type default) (color 0 0 0 0))
   )
-  (wire (pts (xy 204.47 -88.9) (xy 227.33 -88.9))
-    (stroke (width 0) (type default) (color 0 0 0 0))
-  )
   (wire (pts (xy 200.66 530.86) (xy 198.12 530.86))
     (stroke (width 0) (type default) (color 0 0 0 0))
@@
     (stroke (width 0) (type default) (color 0 0 0 0))
   )
-  (wire (pts (xy 204.47 -86.36) (xy 227.33 -86.36))
-    (stroke (width 0) (type default) (color 0 0 0 0))
-  )
   (wire (pts (xy 368.3 210.82) (xy 365.76 210.82))
     (stroke (width 0) (type default) (color 0 0 0 0))
@@
     (effects (font (size 1 1) italic) (justify right bottom))
   )
+  (text "danger pins:\nIO_0 IO_2" (at 49.53 -85.09 0)
+    (effects (font (size 1.27 1.27)) (justify left bottom))
+  )
   (text "VDD: 40dB\nNC:	 60dB\nGND: 50dB" (at -127 334.645 180)
     (effects (font (size 1 1) italic) (justify right bottom))
@@
     )
   )
-  (hierarchical_label "USB_OTG_D-" (shape input) (at 227.33 -86.36 0)
-    (effects (font (size 1.27 1.27)) (justify left))
-  )
-  (hierarchical_label "USB_OTG_D+" (shape input) (at 227.33 -88.9 0)
-    (effects (font (size 1.27 1.27)) (justify left))
-  )
   (symbol (lib_id "Device:C_Small") (at 326.39 46.99 0) (unit 1)
     (in_bom yes) (on_board yes)
@@
     (pin "1")
   )
+  (symbol (lib_id "My_custom_lib:ESP32-A1S_") (at 147.32 -64.77 0) (unit 1)
+    (in_bom yes) (on_board yes) (fields_autoplaced)
+    (property "Reference" "U?" (id 0) (at 154.4194 -100.33 0)
+      (effects (font (size 1.27 1.27)) (justify left))
+    )
+    (property "Value" "ESP32-A1S_" (id 1) (at 154.4194 -97.79 0)
+      (effects (font (size 1.27 1.27)) (justify left))
+    )
+    (property "Footprint" "" (id 2) (at 162.56 -99.06 0)
+      (effects (font (size 1.27 1.27)) hide)
+    )
+    (property "Datasheet" "" (id 3) (at 162.56 -99.06 0)
+      (effects (font (size 1.27 1.27)) hide)
+    )
+    (pin "1")
+    (pin "10")
+    (pin "11")
+    (pin "12")
+    (pin "13")
+    (pin "14")
+    (pin "15")
+    (pin "16")
+    (pin "17")
+    (pin "18")
+    (pin "19")
+    (pin "2")
+    (pin "20")
+    (pin "21")
+    (pin "22")
+    (pin "23")
+    (pin "24")
+    (pin "25")
+    (pin "26")
+    (pin "27")
+    (pin "28")
+    (pin "29")
+    (pin "3")
+    (pin "30")
+    (pin "31")
+    (pin "32")
+    (pin "33")
+    (pin "34")
+    (pin "35")
+    (pin "36")
+    (pin "37")
+    (pin "4")
+    (pin "5")
+    (pin "6")
+    (pin "7")
+    (pin "8")
+    (pin "9")
+  )
   (symbol (lib_id "Device:R_Small") (at 351.79 63.5 0) (unit 1)
     (in_bom yes) (on_board yes) (fields_autoplaced)
@@
     (pin "2")
   )
-  (symbol (lib_id "Espressif:ESP32-S3-WROOM-1") (at 146.05 -58.42 0) (unit 1)
-    (in_bom yes) (on_board yes) (fields_autoplaced)
-    (property "Reference" "U2" (id 0) (at 147.32 -96.52 0))
-    (property "Value" "ESP32-S3-WROOM-1" (id 1) (at 147.32 -93.98 0))
-    (property "Footprint" "Espressif:ESP32-S3-WROOM-1" (id 2) (at 146.05 -25.4 0)
-      (effects (font (size 1.27 1.27)) hide)
-    )
-    (property "Datasheet" "https://www.espressif.com/sites/default/files/documentation/esp32-s3-wroom-1_wroom-1u_datasheet_en.pdf" (id 3) (at 146.05 -22.86 0)
-      (effects (font (size 1.27 1.27)) hide)
-    )
-    (pin "1")
-    (pin "10")
-    (pin "11")
-    (pin "12")
-    (pin "13")
-    (pin "14")
-    (pin "15")
-    (pin "16")
-    (pin "17")
-    (pin "18")
-    (pin "19")
-    (pin "2")
-    (pin "20")
-    (pin "21")
-    (pin "22")
-    (pin "23")
-    (pin "24")
-    (pin "25")
-    (pin "26")
-    (pin "27")
-    (pin "28")
-    (pin "29")
-    (pin "3")
-    (pin "30")
-    (pin "31")
-    (pin "32")
-    (pin "33")
-    (pin "34")
-    (pin "35")
-    (pin "36")
-    (pin "37")
-    (pin "38")
-    (pin "39")
-    (pin "4")
-    (pin "40")
-    (pin "41")
-    (pin "5")
-    (pin "6")
-    (pin "7")
-    (pin "8")
-    (pin "9")
-  )
   (symbol (lib_id "Device:C") (at 389.89 375.285 90) (unit 1)
     (in_bom yes) (on_board yes)
@@
       (reference "U1") (unit 1) (value "CP2102N-Axx-xQFN24") (footprint "Package_DFN_QFN:QFN-24-1EP_4x4mm_P0.5mm_EP2.6x2.6mm")
     )
-    (path "/b21d272b-ac72-4a0a-82c6-e660fe64ac9b"
-      (reference "U2") (unit 1) (value "ESP32-S3-WROOM-1") (footprint "Espressif:ESP32-S3-WROOM-1")
-    )
     (path "/0b39b014-49bc-4a91-b379-91f371838ebc"
       (reference "U3") (unit 1) (value "SA818S") (footprint "Z_mycustom_footprint_lib:SA818S")
@@
       (reference "U?") (unit 1) (value "TS5A63157DBV") (footprint "Package_TO_SOT_SMD:SOT-23-6")
     )
+    (path "/37e5f2cc-01ff-4ce7-b945-a93c063adff0"
+      (reference "U?") (unit 1) (value "ESP32-A1S_") (footprint "")
+    )
     (path "/429c7a58-b354-4d2d-87ce-4a3a713dc9eb"

Commit message: v
Parts:
- removed C17, C19, C22: 1uF, Capacitor_SMD:C_0805_2012Metric, symbol Device:C
- removed C20: 1nF, Capacitor_SMD:C_0805_2012Metric, symbol Device:C
- removed C21: 10uF, Capacitor_SMD:C_0805_2012Metric, symbol Device:C
- removed C25: 47nF, Capacitor_SMD:C_0805_2012Metric, symbol Device:C
- removed R15: 10R, Resistor_SMD:R_0805_2012Metric, symbol Device:R
- removed RV2: 10k, Potentiometer_SMD:Potentiometer_Vishay_TS53YL_Vertical, symbol Device:R_POT
- removed U6: LM386, Package_SO:SOIC-8_3.9x4.9mm_P1.27mm, symbol Amplifier_Audio:LM386
- removed U?: ESP32-A1S_, symbol My_custom_lib:ESP32-A1S_
- added H1, H2, H3, H4: hole, MountingHole:MountingHole_3.2mm_M3_DIN965_Pad_TopBottom, symbol Mechanical:MountingHole_Pad
- added U2: ESP32-A1S, Z_mycustom_footprint_lib:ESP32-A1S, symbol My_custom_lib:ESP32-A1S
- gave numbers to parts that had none: 13
Connections:
- net +3V3: now also U10.5 (V+), U11.5 (V+), U6.5 (V+), U9.5 (V+), U2.2 (3V3)
- net BOOT: now also U2.6 (IO_0)
- net EN: now also U2.35 (EN)
- net GND: now also U10.2 (GND), U11.2 (GND), U6.2 (GND), U9.2 (GND), H1.1, H2.1, H3.1, H4.1, U2.1 (GND), U2.19 (GND), U2.20 (GND), U2.38 (GND)
- net GPIO_21: now also U2.34 (IO_21)
- net PTT1: now also U2.9 (IO_13)
- net PTT2: now also U2.7 (IO_14)
- net RX1: now also U2.8 (IO_12)
- net RX2: now also U2.12 (IO_4)
- net TX1: now also U2.29 (IO_5)
- net TX2: now also U2.11 (IO_2)
- net UART0_RX: now also U2.37 (RXD0)
- net UART0_TX: now also U2.36 (TXD0)
- net AUDIO_ON1: now reaches U3.1 (Audio_ON)
- net AUDIO_ON1: now also U2.10 (IO_15)
- net switch3: now reaches U11.6
- net AUDIO_ON2: now reaches U4.1 (Audio_ON)
- net AUDIO_ON2: now also U2.30 (IO_18)
- net switch4: now reaches U10.6
- net switch2: now reaches U9.6
- net switch1: now reaches U6.6
- new net GPIO_19: U2.32 (IO_19)
- new net GPIO_22: U2.33 (IO_22)
- new net GPIO_23: U2.31 (IO_23)
- new net GPIO_34: U2.5 (IO_34)
Other:
- note removed: "SPEAKER AMP"
- moved on the sheet: C1, C10, C11, C12, C13, C14, C15, C16, C18, C2, C23, C24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

Commit message: Update cross_band_handy_walkie_talkie_V1.kicad_sch
Parts:
- removed C26, C27: 4u7, Capacitor_SMD:C_0603_1608Metric_Pad1.08x0.95mm_HandSolder, symbol Device:C_Small
- removed U4: SA818S, Z_mycustom_footprint_lib:SA818S, symbol My_custom_lib:SA818S
- removed U7: LT1129-3.3_SO8, Package_SO:SOIC-8_3.9x4.9mm_P1.27mm, symbol Regulator_Linear:LT1129-3.3_SO8
- added C? (x5): 100n, Capacitor_SMD:C_0603_1608Metric_Pad1.08x0.95mm_HandSolder, symbol Device:C_Small
- added C? (x4): 10u, Capacitor_SMD:C_0603_1608Metric_Pad1.08x0.95mm_HandSolder, symbol Device:C_Small
- added C? (x2): 100n, Capacitor_SMD:C_0805_2012Metric, symbol Device:C
- added C?: 470n, Capacitor_SMD:C_0805_2012Metric, symbol Device:C
- added C?: 2u2, Capacitor_SMD:C_0805_2012Metric, symbol Device:C
- added J? (x2): Conn_01x03, Connector_PinHeader_2.54mm:PinHeader_1x03_P2.54mm_Vertical, symbol Connector_Generic:Conn_01x03
- added J?: Conn_01x03, Jumper:SolderJumper-3_P2.0mm_Open_TrianglePad1.0x1.5mm_NumberLabels, symbol Connector_Generic:Conn_01x03
- added L?: Ferrit, Resistor_SMD:R_0805_2012Metric_Pad1.20x1.40mm_HandSolder, symbol Device:L
- added R?: 1k, Resistor_SMD:R_0805_2012Metric, symbol Device:R
- added R?: 2k2, Resistor_SMD:R_0805_2012Metric, symbol Device:R
- added R?: 150k, Resistor_SMD:R_0805_2012Metric, symbol Device:R
- added R?: 100k, Resistor_SMD:R_0805_2012Metric, symbol Device:R
- added U?: AMS1117-3.3, Package_TO_SOT_SMD:SOT-223-3_TabPin2, symbol Regulator_Linear:AMS1117-3.3
- added U?: SA818S, Z_mycustom_footprint_lib:SA818S, symbol My_custom_lib:SA818S
- added U?: PCA9554APW, Package_SO:TSSOP-16_4.4x5mm_P0.65mm, symbol My_custom_lib:PCA9554APW
- added U?: PCA9555PW, Package_SO:TSSOP-24_4.4x7.8mm_P0.65mm, symbol Interface_Expansion:PCA9555PW
- added U?: MAX9814, Package_DFN_QFN:DFN-14-1EP_3x3mm_P0.4mm_EP1.78x2.35mm, symbol Amplifier_Audio:MAX9814
- U10, U11, U6, U9: LCSC (none) -> C2673185
- U2: LCSC (none) -> C277945
- U3: LCSC (none) -> C3001549
- U5: footprint (none) -> Package_SO:SOIC-8-1EP_3.9x4.9mm_P1.27mm_EP2.41x3.3mm_ThermalVias; LCSC (none) -> C383071
Connections:
- net +3V3: now also C?.1, C?.1, C?.1, C?.1, C?.1, C?.1, C?.1, J?.3 (Pin_3), J?.3 (Pin_3), L?.2, U?.16 (VCC), U?.2 (VO)
- net +5V: now also C?.1, U?.3 (VI), U?.8 (VBATT)
- net -SLEEP: now also U?.2 (~{SHDN})
- net AUDIO_ON2: now also U?.1 (Audio_ON)
- net GND: now also C?.1, C?.1, C?.2, C?.2, C?.2, C?.2, C?.2, C?.2, C?.2, C?.2, C?.2, C?.2, C?.2, J?.1 (Pin_1), J?.1 (Pin_1), R?.1, R?.2, U?.1 (A0), U?.1 (GND), U?.10 (GND), U?.11 (GND), U?.15 (GND), U?.2 (A1), U?.3 (A2), U?.4 (GND), U?.7 (GND), U?.8 (GND), U?.8 (MICIN), U?.9 (GND)
- net H/L1: now also U?.5 (IO_1)
- net H/L2: now also U?.7 (H/L), U?.7 (IO_3)
- net MIC-AMP_IN: now also C?.2, R?.2
- net MIC-DIGI_IN: now also J?.3 (Pin_3)
- net MIC_AR: now also J?.2 (Pin_2), U?.9 (A/R)
- net MIC_GAIN: now also J?.2 (Pin_2), R?.2
- net PD1: now also U?.4 (IO_0)
- net PD2: now also U?.6 (IO_2), U?.6 (PD)
- net PTT2: now also U?.5 (PTT)
- net RX2: now also U?.17 (TXD(TX))
- net TRX_MIC: now also J?.2 (Pin_2)
- net TX2: now also U?.16 (RXD_(RX))
- net switch1: now also U?.9 (IO_4)
- net switch2: now also U?.10 (IO_5)
- net switch3: now also U?.11 (IO_6)
- net switch4: now also U?.12 (IO_7)
- net at U11.1: now also U?.3 (AF(Audio_OUT))
- net at FL1.1 (IN): now also U?.12 (ANT)
- net at U10.3: now also U?.18 (MIC_IN)
- net GPIO_19 renamed SDA
- net SDA: now also U?.15 (SDA)
- net GPIO_21 renamed SCL
- net SCL: now also U?.14 (SCL)
- new net: C?.2, U?.1 (CT)
- new net: C?.1, L?.1, U?.5 (VDD)
- new net: R?.1, U?.13 (MICBIAS)
- new net: R?.1, R?.2, U?.14 (TH)
- new net: C?.1, U?.12 (BIAS)
- new net: C?.1, U?.3 (CG)
- new net: J?.1 (Pin_1), U?.6 (MICOUT)
- new net MIC_GAIN_pin: R?.1, U?.10 (GAIN)
- no-connect marks 4 -> 5
Other:
- note added: "https://lcsc.com/product-detail/Audio-Power-OpAmps_HGSEMI-LM386M-1-TR_C383071.html https://lcsc.com/product-detail/Audio-Power-OpAmps_Texas-Instruments-LM386MX-1-NOPB_C23573.html"
- note added: "https://lcsc.com/products/Analog-Switches-Multiplexers_618.html"
- note added: "https://lcsc.com/products/Audio-Connectors_590.html?keyword=audio%20jack"
- note added: "https://lcsc.com/products/Variable-Resistors-Potentiometers_520.html"

Commit message: j
Parts:
- removed C1, C2, C? (x5): 100n, Capacitor_SMD:C_0603_1608Metric_Pad1.08x0.95mm_HandSolder, symbol Device:C_Small
- removed C28, C29, C? (x4): 10u, Capacitor_SMD:C_0603_1608Metric_Pad1.08x0.95mm_HandSolder, symbol Device:C_Small
- removed C7, C8: 100nF, Capacitor_SMD:C_0805_2012Metric, symbol Device:C
- removed C? (x2): 100n, Capacitor_SMD:C_0805_2012Metric, symbol Device:C
- removed Q1: BC847BS, symbol Device:Q_Dual_NPN_NPN_E1B1C2E2B2C1
- added C10, C14, C25, C26, C32, C33, C9: 10u, Capacitor_SMD:C_0805_2012Metric, symbol Device:C_Small
- added C11, C12, C16, C17, C18, C31, C34, C35, C36, C37, C38, C4, C5: 100n, Capacitor_SMD:C_0603_1608Metric_Pad1.08x0.95mm_HandSolder, symbol Device:C_Small
- added Q1, Q2: MMBT3904, Package_TO_SOT_SMD:SOT-23, symbol Device:Q_NPN_BEC
- C1: renamed from C5; LCSC (none) -> C14663
- C13: value 100n -> 10u; footprint Capacitor_SMD:C_0603_1608Metric_Pad1.08x0.95mm_HandSolder -> Capacitor_SMD:C_0805_2012Metric; LCSC (none) -> C15850
- C15: value 10u -> 100n; LCSC (none) -> C14663
- C2: renamed from C4; footprint Capacitor_SMD:C_0603_1608Metric_Pad1.08x0.95mm_HandSolder -> Capacitor_SMD:C_0805_2012Metric; LCSC (none) -> C15850
- C3: footprint Capacitor_SMD:C_0603_1608Metric_Pad1.08x0.95mm_HandSolder -> Capacitor_SMD:C_0805_2012Metric; LCSC (none) -> C15850
- D1, D2: footprint LED_SMD:LED_0603_1608Metric_Pad1.05x0.95mm_HandSolder -> LED_SMD:LED_0805_2012Metric; LCSC (none) -> C2297
- gave numbers to parts that had none: 15
- renumbered C9 to C19, C10 to C20, C30 to C23, C14 to C24, C16 to C27, C18 to C28, C23 to C29, C24 to C30, C11 to C7, C12 to C8, J9 to J10, J6 to J11, J10 to J12, J11 to J13, J3 to J14, J12 to J15, J4 to J2, J5 to J3, J2 to J6, J7 to J8, J8 to J9, L1 to L2, R6 to R10, R13 to R11, R16 to R12, R17 to R14, R18 to R16, R19 to R18, R8 to R2, R14 to R20, R2 to R3, R9 to R4, R7 to R5, R3 to R6, R12 to R7, R4 to R8, R5 to R9, RV3 to RV2, U5 to U10, U10 to U11, U11 to U12, U3 to U14, U8 to U6, U6 to U8
Connections:
- net +3V3: now also C10.1, C12.1, C14.1, C35.1, C36.1, C37.1, C38.1
- net +5V: now also C25.1, C26.1, C31.1, C32.1, C33.1, C34.2, C9.1; no longer C15.1
- net BASE1: now also Q1.1 (B)
- net BASE2: now also Q2.1 (B)
- net BOOT: now also C11.1, Q2.3 (C); no longer C13.1
- net EN: now also Q1.3 (C)
- net GND: now also C10.2, C11.2, C12.2, C14.2, C16.2, C17.2, C18.2, C25.2, C26.2, C31.2, C32.2, C33.2, C34.1, C35.2, C36.2, C37.2, C38.2, C4.2, C5.2, C9.2
- net MIC-AMP_IN: now also C17.1, C18.1
- net VDD_CP: now also C4.1
- net ~{DTR}: now also Q2.2 (E)
- net ~{RST_CP}: now also C5.1
- net ~{RTS}: now also Q1.2 (E)
- net at U7.1 (CT): now also C16.1
- net at L1.1, U7.5 (VDD): now also C13.1
- net at U6.1 (CT): now also C15.1
Other:
- note added: "15ms delay needed (10-20ms is fine)"
