File: HW/cross_band_handy_walkie_talkie_V1/cross_band_handy_walkie_talkie_V1.kicad_sch (KiCad schematic)
At the start: 103 parts, among them J1 USB_OTG, J10 pin, J11 Conn_01x03, J12 pin, J13 pin, J14 Conn_Coaxial, J15 Conn_Coaxial, J2 Conn_01x03, J3 Conn_01x03, J4 Conn_01x03, J5 Conn_01x03, J6 pin, J7 Conn_01x03, J8 pin, J9 pin, Q1 MMBT3904, Q2 MMBT3904, SW1 MCU_RESET, U1 CP2102N-Axx-xQFN24, U10 LM386, U11 TS5A63157DBV, U12 TS5A63157DBV, U13 SA818S, U14 SA818S, U2 ESP32-A1S, U3 AMS1117-3.3, U4 PCA9554APW, U5 PCA9555PW, U6 MAX9814, U7 MAX9814, U8 TS5A63157DBV, U9 TS5A63157DBV

Commit message: t
Parts:
- removed C17: 100n, Capacitor_SMD:C_0603_1608Metric_Pad1.08x0.95mm_HandSolder, symbol Device:C_Small
- removed C19: 470nF, Capacitor_SMD:C_0805_2012Metric, symbol Device:C
- removed C20: 2.2uF, Capacitor_SMD:C_0805_2012Metric, symbol Device:C
- removed C23: 1uF, Capacitor_SMD:C_0805_2012Metric, symbol Device:C
- removed FB1: MH2029-401Y, Resistor_SMD:R_0805_2012Metric_Pad1.20x1.40mm_HandSolder, symbol Device:FerriteBead_Small
- removed J1: USB_OTG, symbol Connector:USB_OTG
- removed J10, J12, J13, J6, J8, J9: pin, Connector_PinHeader_2.54mm:PinHeader_1x01_P2.54mm_Vertical, symbol Connector_Generic:Conn_01x01
- removed J11: Conn_01x03, Jumper:SolderJumper-3_P2.0mm_Open_TrianglePad1.0x1.5mm_NumberLabels, symbol Connector_Generic:Conn_01x03
- removed L1, L2: Ferrit, Resistor_SMD:R_0805_2012Metric_Pad1.20x1.40mm_HandSolder, symbol Device:L
- removed R1: 1k, Resistor_SMD:R_0603_1608Metric_Pad0.98x0.95mm_HandSolder, symbol Device:R_Small
- removed R12: #2.2k, Resistor_SMD:R_0805_2012Metric, symbol Device:R
- removed R14: 150k, Resistor_SMD:R_0805_2012Metric, symbol Device:R
- removed R16: 1k, Resistor_SMD:R_0805_2012Metric, symbol Device:R
- removed R18: 100k, Resistor_SMD:R_0805_2012Metric, symbol Device:R
- removed R3: 22k, Resistor_SMD:R_0603_1608Metric_Pad0.98x0.95mm_HandSolder, symbol Device:R_Small
- removed R5: 1Meg, Resistor_SMD:R_0603_1608Metric_Pad0.98x0.95mm_HandSolder, symbol Device:R_Small
- removed R6: 47k, Resistor_SMD:R_0603_1608Metric_Pad0.98x0.95mm_HandSolder, symbol Device:R_Small
- removed R8: 10k, Resistor_SMD:R_0603_1608Metric_Pad0.98x0.95mm_HandSolder, symbol Device:R_Small
- removed U1: CP2102N-Axx-xQFN24, Package_DFN_QFN:QFN-24-1EP_4x4mm_P0.5mm_EP2.6x2.6mm, symbol Interface_USB:CP2102N-Axx-xQFN24
- removed U5: PCA9555PW, Package_SO:TSSOP-24_4.4x7.8mm_P0.65mm, symbol Interface_Expansion:PCA9555PW
- removed U6: MAX9814, Package_DFN_QFN:DFN-14-1EP_3x3mm_P0.4mm_EP1.78x2.35mm, symbol Amplifier_Audio:MAX9814
- added FB2: MH2029-401Y, Resistor_SMD:R_0805_2012Metric_Pad1.20x1.40mm_HandSolder, symbol Device:FerriteBead_Small
- added J1: AudioPlug3, symbol Connector:AudioPlug3
- added J6: USB_C_Receptacle, Connector_USB:USB_C_Receptacle_HRO_TYPE-C-31-M-12, symbol Connector:USB_C_Receptacle
- added L1: L_Small, Inductor_SMD:L_0805_2012Metric, symbol Device:L_Small
- added R12, R14: 5k1, Resistor_SMD:R_0603_1608Metric_Pad0.98x0.95mm_HandSolder, symbol Device:R_Small
- added R16: 1Meg, Resistor_SMD:R_0603_1608Metric_Pad0.98x0.95mm_HandSolder, symbol Device:R_Small
- added U1: CH340C, Package_SO:SOIC-16_3.9x9.9mm_P1.27mm, symbol Interface_USB:CH340C
- C15: value 100n -> 10p; LCSC C14663 -> (none)
- C5: value 100n -> 10u; footprint Capacitor_SMD:C_0603_1608Metric_Pad1.08x0.95mm_HandSolder -> Capacitor_SMD:C_0805_2012Metric; LCSC C14663 -> C15850
- C6: value 10p -> 100n; LCSC (none) -> C14663
- J2, J3: Remarks Mouser: 649-54201-G0803ALF -> (none)
- J7: footprint Jumper:SolderJumper-3_P2.0mm_Open_TrianglePad1.0x1.5mm_NumberLabels -> Connector_PinHeader_2.54mm:PinHeader_1x03_P2.54mm_Vertical
- RV1, RV2: LCSC (none) -> C118956
Connections:
- net GPIO_34 is gone; now on net -SLEEP: U2.5 (IO_34)
- net RXT is gone; now on net UART0_TX: R10.1
- net TXT is gone; now on net UART0_RX: R9.1
- net VDD_CP is gone; now on net +5V: C4.1
- net VIO is gone; now on net +3V3: D1.2 (A), D2.2 (A)
- net ~{RST_CP} is gone; now on net +5V: C5.1
- net +3V3: now also L1.2; no longer J2.3 (Pin_3), J3.3 (Pin_3)
- net +5V: now also C33.2, C34.1, FB2.2, U1.16 (VCC); no longer C33.1, C34.2
- net AUDIO_IN: now also J3.2 (Pin_2)
- net AUDIO_OUT: now also J3.1 (Pin_1)
- net D+: now also J6.A6 (D+), J6.B6 (D+), U1.5 (UD+)
- net D-: now also J6.A7 (D-), J6.B7 (D-), U1.6 (UD-)
- net GND: now also C33.1, C34.2, J1.S, J6.A1 (GND), J6.A12 (GND), J6.B1 (GND), J6.B12 (GND), R12.2, R14.2, R16.1, U1.1 (GND); no longer C33.2, C34.1, J2.1 (Pin_1), J3.1 (Pin_1), R13.1
- net MIC_AR: no longer J3.2 (Pin_2)
- net MIC_GAIN: no longer J2.2 (Pin_2)
- net MIC_IN: now also J2.2 (Pin_2)
- net UART0_RX: now also U1.2 (TXD)
- net UART0_TX: now also U1.3 (RXD)
- net VBUS: now also FB2.1, J6.A4 (VBUS), J6.A9 (VBUS), J6.B4 (VBUS), J6.B9 (VBUS)
- net esp audio: now also J2.3 (Pin_3), J3.3 (Pin_3)
- net at C6.1: now also U1.4 (V3)
- net at C15.1: now also J6.S1 (SHIELD), R16.2
- net +3.3VA: now reaches C13.1, U7.5 (VDD)
- net +3.3VA: now also L1.1
- net at U7.13 (MICBIAS): now also R13.1, R15.2; no longer R15.1
- net at R17.1, U7.14 (TH): now also R15.1; no longer R15.2
- net at U8.3: now also J2.1 (Pin_1), J7.1 (Pin_1), U7.6 (MICOUT)
- new net: J6.A5 (CC1), R12.1
- new net: J6.B5 (CC2), R14.1
- no-connect marks 5 -> 19
Other:
- moved on the sheet: C1, C12, C13, C14, C16, C18, C2, C21, C22, C24, C25, C26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
