File: HW/cross_band_handy_walkie_talkie_V1/cross_band_handy_walkie_talkie_V1.kicad_sch (KiCad schematic)
At the start: 84 parts, among them J1 AudioPlug3, J14 Conn_Coaxial, J15 Conn_Coaxial, J2 Conn_01x03, J3 Conn_01x03, J4 Conn_01x03, J5 Conn_01x03, J6 USB_C_Receptacle, J7 Conn_01x03, Q1 MMBT3904, Q2 MMBT3904, SW1 MCU_RESET, U1 CH340C, U10 LM386, U11 TS5A63157DBV, U12 TS5A63157DBV, U13 SA818S, U14 SA818S, U2 ESP32-A1S, U3 AMS1117-3.3, U4 PCA9554APW, U7 MAX9814, U8 TS5A63157DBV, U9 TS5A63157DBV

Commit message: f
Parts:
- removed J1: AudioPlug3, symbol Connector:AudioPlug3
- added J8: RFShield_OnePiece, RF_Shielding:Wuerth_36103205_20x20mm, symbol Device:RFShield_OnePiece
- RV1, RV2: footprint Potentiometer_SMD:Potentiometer_Vishay_TS53YL_Vertical -> Potentiometer_THT:Potentiometer_Bourns_3266W_Vertical
Connections:
- net GND: now also J8.1 (Shield)
- net MIC_out: now reaches J2.1 (Pin_1), J7.1 (Pin_1), U7.6 (MICOUT), U8.3
- net ant3: now reaches FL2.1 (IN), U14.12 (ANT)
- net ant4: now reaches FL2.3 (OUT), J15.1 (In)
- net ant1: now reaches FL1.1 (IN), U13.12 (ANT)
- net ant2: now reaches FL1.3 (OUT), J14.1 (In)
- net MIC_BIAS: now reaches R13.1, R15.2, U7.13 (MICBIAS)
- net cc1: now reaches J6.A5 (CC1), R12.1
- net cc2: now reaches J6.B5 (CC2), R14.1
- net BIAS: now reaches C21.1, U7.12 (BIAS)
- net CG: now reaches C22.1, U7.3 (CG)
Other:
- moved on the sheet: C1, C10, C11, C12, C13, C14, C15, C16, C18, C2, C21, C22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

Commit message: R
Parts:
- added J1: Conn_01x06, Connector_PinHeader_2.54mm:PinHeader_1x06_P2.54mm_Vertical, symbol Connector_Generic:Conn_01x06
Connections:
- net +3V3: now also J1.1 (Pin_1)
- net GND: now also J1.2 (Pin_2), J1.5 (Pin_5)
- net MIC-AMP_IN: now also J1.6 (Pin_6)
- new net EXT_SPEAKER+: J1.3 (Pin_3)
- new net MIC_EST_PTT: J1.4 (Pin_4)
Other:
- note added: "SA181-1"
- note added: "SA181-2"
Changed lines of the file:
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@@
     (stroke (width 0) (type default) (color 0 0 0 0))
   )
+  (wire (pts (xy 255.27 288.29) (xy 237.49 288.29))
+    (stroke (width 0) (type default) (color 0 0 0 0))
+  )
   (wire (pts (xy 139.7 208.28) (xy 139.7 210.82))
     (stroke (width 0) (type default) (color 0 0 0 0))
@@
     (stroke (width 0) (type default) (color 0 0 0 0))
   )
+  (wire (pts (xy 237.49 283.21) (xy 255.27 283.21))
+    (stroke (width 0) (type default) (color 0 0 0 0))
+  )
   (wire (pts (xy 281.94 104.14) (xy 281.94 106.68))
     (stroke (width 0) (type default) (color 0 0 0 0))
@@
     (stroke (width 0) (type default) (color 0 0 0 0))
   )
+  (wire (pts (xy 92.71 60.96) (xy 85.09 60.96))
+    (stroke (width 0) (type default) (color 0 0 0 0))
+  )
   (wire (pts (xy 464.82 254) (xy 464.82 256.54))
     (stroke (width 0) (type default) (color 0 0 0 0))
@@
     (stroke (width 0) (type default) (color 0 0 0 0))
   )
+  (wire (pts (xy 255.27 290.83) (xy 237.49 290.83))
+    (stroke (width 0) (type default) (color 0 0 0 0))
+  )
   (wire (pts (xy 363.22 45.72) (xy 340.36 45.72))
     (stroke (width 0) (type default) (color 0 0 0 0))
@@
     (stroke (width 0) (type default) (color 0 0 0 0))
   )
+  (wire (pts (xy 237.49 285.75) (xy 259.08 285.75))
+    (stroke (width 0) (type default) (color 0 0 0 0))
+  )
   (wire (pts (xy 157.48 340.36) (xy 162.56 340.36))
     (stroke (width 0) (type default) (color 0 0 0 0))
@@
     (stroke (width 0) (type default) (color 0 0 0 0))
   )
+  (wire (pts (xy 95.25 101.6) (xy 87.63 101.6))
+    (stroke (width 0) (type default) (color 0 0 0 0))
+  )
   (wire (pts (xy 167.64 157.48) (xy 167.64 160.02))
     (stroke (width 0) (type default) (color 0 0 0 0))
@@
     (stroke (width 0) (type default) (color 0 0 0 0))
   )
+  (wire (pts (xy 242.57 295.91) (xy 237.49 295.91))
+    (stroke (width 0) (type default) (color 0 0 0 0))
+  )
+  (wire (pts (xy 259.08 293.37) (xy 237.49 293.37))
+    (stroke (width 0) (type default) (color 0 0 0 0))
+  )
   (wire (pts (xy 180.34 53.34) (xy 185.42 53.34))
     (stroke (width 0) (type default) (color 0 0 0 0))
@@
     (effects (font (size 1.27 1.27) bold italic) (justify left bottom))
   )
+  (text "SA181-2\n" (at 179.07 378.46 0)
+    (effects (font (size 1.27 1.27)) (justify left bottom))
+  )
   (text "VDD: 1:2000\nNC: 1:4000\nGND: 1:500\n\n\n" (at 96.52 222.25 180)
     (effects (font (size 1 1) italic) (justify right bottom))
   )
+  (text "SA181-1\n" (at 101.6 378.46 0)
+    (effects (font (size 1.27 1.27)) (justify left bottom))
+  )
   (text "15ms delay needed (10-20ms is fine)" (at 378.46 83.185 0)
     (effects (font (size 1.27 1.27)) (justify left bottom))
@@
     (effects (font (size 0.5 0.5)) (justify left bottom))
   )
+  (label "MIC_EST_PTT" (at 255.27 288.29 180)
+    (effects (font (size 1.27 1.27)) (justify right bottom))
+  )
   (label "MIC_GAIN" (at 50.8 218.44 180)
     (effects (font (size 1.27 1.27)) (justify right bottom))
@@
     (effects (font (size 1.27 1.27)) (justify left bottom))
   )
+  (label "MIC-AMP_IN" (at 255.27 283.21 180)
+    (effects (font (size 1.27 1.27)) (justify right bottom))
+  )
   (label "GPIO_18" (at 38.1 104.14 180)
     (effects (font (size 1.27 1.27)) (justify right bottom))
@@
     (effects (font (size 1.27 1.27)) (justify left bottom))
   )
+  (label "EXT_SPEAKER+" (at 255.27 290.83 180)
+    (effects (font (size 1.27 1.27)) (justify right bottom))
+  )
   (label "MIC-DIGI_IN" (at 142.24 248.92 0)
     (effects (font (size 1.27 1.27)) (justify left bottom))
@@
     )
   )
+  (global_label "AUDIO_OUT" (shape input) (at 92.71 60.96 0) (fields_autoplaced)
+    (effects (font (size 1.27 1.27) (thickness 0.254) bold italic) (justify left))
+    (property "Intersheet References" "${INTERSHEET_REFS}" (id 0) (at 105.7896 60.833 0)
+      (effects (font (size 1.27 1.27) (thickness 0.254) bold italic) (justify left) hide)
+    )
+  )
   (global_label "UART0_TX" (shape input) (at 35.56 60.96 180) (fields_autoplaced)
     (effects (font (size 1.27 1.27)) (justify right))
@@
     )
   )
+  (global_label "MIC_IN" (shape input) (at 95.25 101.6 0) (fields_autoplaced)
+    (effects (font (size 1.27 1.27) (thickness 0.254) bold italic) (justify left))
+    (property "Intersheet References" "${INTERSHEET_REFS}" (id 0) (at 104.3381 101.727 0)
+      (effects (font (size 1.27 1.27) (thickness 0.254) bold italic) (justify left) hide)
+    )
+  )
   (global_label "H{slash}L1" (shape input) (at 121.92 363.22 0) (fields_autoplaced)
     (effects (font (size 1.27 1.27)) (justify left))
@@
     (pin "1")
   )
+  (symbol (lib_id "power:GND") (at 259.08 285.75 0) (unit 1)
+    (in_bom yes) (on_board yes)
+    (property "Reference" "#PWR0111" (id 0) (at 259.08 292.1 0)
+      (effects (font (size 1.27 1.27)) hide)
+    )
+    (property "Value" "GND" (id 1) (at 259.207 290.1442 0)
+      (effects (font (size 1.27 1.27)) hide)
+    )
+    (property "Footprint" "" (id 2) (at 259.08 285.75 0)
+      (effects (font (size 1.27 1.27)) hide)
+    )
+    (property "Datasheet" "" (id 3) (at 259.08 285.75 0)
+      (effects (font (size 1.27 1.27)) hide)
+    )
+    (pin "1")
+  )
   (symbol (lib_id "Device:LED_Small") (at 144.78 86.36 90) (unit 1)
     (in_bom yes) (on_board yes) (fields_autoplaced)
@@
     (pin "4")
   )
+  (symbol (lib_id "power:+3V3") (at 242.57 295.91 270) (unit 1)
+    (in_bom yes) (on_board yes)
+    (property "Reference" "#PWR?" (id 0) (at 238.76 295.91 0)
+      (effects (font (size 1.27 1.27)) hide)
+    )
+    (property "Value" "+3V3" (id 1) (at 248.92 295.91 90))
+    (property "Footprint" "" (id 2) (at 242.57 295.91 0)
+      (effects (font (size 1.27 1.27)) hide)
+    )
+    (property "Datasheet" "" (id 3) (at 242.57 295.91 0)
+      (effects (font (size 1.27 1.27)) hide)
+    )
+    (pin "1")
+  )
   (symbol (lib_id "power:+3V3") (at 314.96 104.14 0) (mirror y) (unit 1)
     (in_bom yes) (on_board yes) (fields_autoplaced)
@@
     (pin "3")
   )
+  (symbol (lib_id "power:GND") (at 259.08 293.37 0) (unit 1)
+    (in_bom yes) (on_board yes)
+    (property "Reference" "#PWR?" (id 0) (at 259.08 299.72 0)
+      (effects (font (size 1.27 1.27)) hide)
+    )
+    (property "Value" "GND" (id 1) (at 259.207 297.7642 0)
+      (effects (font (size 1.27 1.27)) hide)
+    )
+    (property "Footprint" "" (id 2) (at 259.08 293.37 0)
+      (effects (font (size 1.27 1.27)) hide)
+    )
+    (property "Datasheet" "" (id 3) (at 259.08 293.37 0)
+      (effects (font (size 1.27 1.27)) hide)
+    )
+    (pin "1")
+  )
   (symbol (lib_id "power:GND") (at 139.7 287.02 0) (unit 1)
     (in_bom yes) (on_board yes) (fields_autoplaced)
@@
     (pin "2")
   )
+  (symbol (lib_id "Connector_Generic:Conn_01x06") (at 232.41 290.83 180) (unit 1)
+    (in_bom yes) (on_board yes)
+    (property "Reference" "J1" (id 0) (at 224.79 287.02 0))
+    (property "Value" "Conn_01x06" (id 1) (at 224.79 289.56 0))
+    (property "Footprint" "Connector_PinHeader_2.54mm:PinHeader_1x06_P2.54mm_Vertical" (id 2) (at 232.41 290.83 0)
+      (effects (font (size 1.27 1.27)) hide)
+    )
+    (property "Datasheet" "~" (id 3) (at 232.41 290.83 0)
+      (effects (font (size 1.27 1.27)) hide)
+    )
+    (pin "1")
+    (pin "2")
+    (pin "3")
+    (pin "4")
+    (pin "5")
+    (pin "6")
+  )
   (symbol (lib_id "Device:C_Small") (at 353.06 88.9 0) (unit 1)
     (in_bom yes) (on_board yes) (fields_autoplaced)
@@
       (reference "#PWR0110") (unit 1) (value "GND") (footprint "")
     )
+    (path "/62117082-fc2f-4665-97bc-c5bb8317f0a4"
+      (reference "#PWR0111") (unit 1) (value "GND") (footprint "")
+    )
+    (path "/d6272214-7378-427b-afc6-1030437be5e1"
+      (reference "#PWR?") (unit 1) (value "+3V3") (footprint "")
+    )
+    (path "/e25fec8d-1484-40a1-ab82-dc651a34b03a"
+      (reference "#PWR?") (unit 1) (value "GND") (footprint "")
+    )
     (path "/8c509600-7f9c-4bfc-84b1-320113255391"
       (reference "C1") (unit 1) (value "100n") (footprint "Capacitor_SMD:C_0603_1608Metric_Pad1.08x0.95mm_HandSolder")
@@
       (reference "H4") (unit 1) (value "hole") (footprint "MountingHole:MountingHole_3.2mm_M3_DIN965_Pad_TopBottom")
     )
+    (path "/f698f558-b26f-43d1-b14b-2a6416d2b11f"
+      (reference "J1") (unit 1) (value "Conn_01x06") (footprint "Connector_PinHeader_2.54mm:PinHeader_1x06_P2.54mm_Vertical")
+    )
     (path "/0013baf7-b1e0-4773-aa1b-0b3d8e0bb22e"

Commit message: k
Parts:
- added D3: D_Small, Diode_SMD:D_SOD-123, symbol Device:D_Small
- added J9: Conn_01x02, Connector_PinHeader_2.54mm:PinHeader_1x02_P2.54mm_Vertical, symbol Connector_Generic:Conn_01x02
- added JP1: Jumper_3_Bridged12, Connector_PinHeader_2.54mm:PinHeader_1x03_P2.54mm_Vertical, symbol Jumper:Jumper_3_Bridged12
- added R1, R3: 5k1, Resistor_SMD:R_0603_1608Metric_Pad0.98x0.95mm_HandSolder, symbol Device:R_Small
Connections:
- net GND: now also J9.1 (Pin_1)
- net MIC_EST_PTT: now also JP1.2 (C)
- net PTT1: now also R3.1
- net PTT2: now also R1.2
- net VBUS: now also D3.1 (K)
- new net: JP1.1 (A), R3.2
- new net: JP1.3 (B), R1.1
- new net: D3.2 (A), J9.2 (Pin_2)

Commit message: n
Parts:
- added C17, C19: 1u, Capacitor_SMD:C_0603_1608Metric_Pad1.08x0.95mm_HandSolder, symbol Device:C_Small
- added D4: LED_Small, LED_SMD:LED_0805_2012Metric, symbol Device:LED_Small
- added FID1: Fiducial, Fiducial:Fiducial_0.5mm_Mask1mm, symbol Mechanical:Fiducial
- added FID2: Fiducial, Symbol:KiCad-Logo2_5mm_SilkScreen, symbol Mechanical:Fiducial
- added FID3: Fiducial, Symbol:WEEE-Logo_4.2x6mm_SilkScreen, symbol Mechanical:Fiducial
- added J10: Conn_01x02, Connector_PinHeader_2.54mm:PinHeader_1x02_P2.54mm_Vertical, symbol Connector_Generic:Conn_01x02
- added R5: 300, Resistor_SMD:R_0603_1608Metric_Pad0.98x0.95mm_HandSolder, symbol Device:R_Small
- J14, J15: value Conn_Coaxial -> SMA
Connections:
- net AUDIO_OUT: now also C19.2; no longer C28.2
- net GND: now also J10.1 (Pin_1), R5.1
- net GPIO_23: now also D4.2 (A)
- net MIC_IN: now also C17.2
- net at U2.21 (LINE_INR): now also U2.22 (LINE_INL), C19.1
- net at U2.27 (HPOUT_L): now also U2.28 (HPOUT_R), C17.1
- net EXT_SPEAKER+ renamed AMPLIFIED_AUDIO_OUT
- net AMPLIFIED_AUDIO_OUT: now also C28.2, J10.2 (Pin_2)
- new net: D4.1 (K), R5.2
Other:
- note added: "3V3 LOD"
- note added: "ANALOG BIDIRECTIONAL SWITCHES"
- note added: "AUDIO IO"
- note added: "AUDIO POWER AMPLIFIER"
- note added: "CONTROL"
- note added: "MCU+PROGRAMING"
- note added: "MIC AMPLIFIER"
- note added: "MISCELANIOUS"
- note added: "RF MODULES"
- moved on the sheet: C1, C10, C11, C12, C15, C2, C24, C25, C26, C27, C28, C29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

Commit message: g
Parts:
- added C20: 1u, Capacitor_SMD:C_0603_1608Metric_Pad1.08x0.95mm_HandSolder, symbol Device:C_Small
Connections:
- net MIC_out: now also C20.1; no longer J2.1 (Pin_1), U8.3
- new net: C20.2, J2.1 (Pin_1), U8.3
Other:
- moved on the sheet: C15, C21, C22, C4, C5, D4, R16, R17, R5

Commit message: m
Other:
- note added: "3V3 LDO"
- note removed: "3V3 LOD"
Changed lines of the file:
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@@
     (stroke (width 0) (type default) (color 0 0 0 0))
   )
-  (text "3V3 LOD" (at 285.75 203.2 0)
+  (text "3V3 LDO" (at 285.75 203.2 0)
     (effects (font (size 5 5)) (justify left bottom))
   )

Commit message: f
Parts:
- removed J10: Conn_01x02, Connector_PinHeader_2.54mm:PinHeader_1x02_P2.54mm_Vertical, symbol Connector_Generic:Conn_01x02
- removed J7: Conn_01x03, Connector_PinHeader_2.54mm:PinHeader_1x03_P2.54mm_Vertical, symbol Connector_Generic:Conn_01x03
- added J7: Conn_01x04, Connector_PinHeader_2.54mm:PinHeader_1x04_P2.54mm_Vertical, symbol Connector_Generic:Conn_01x04
Connections:
- net AUDIO_OUT: now also J3.3 (Pin_3); no longer J3.1 (Pin_1)
- net GND: now also J3.1 (Pin_1), U9.1, J7.1 (Pin_1)
- net MIC-DIGI_IN: now also J7.2 (Pin_2)
- net at C17.1, U2.28 (HPOUT_R): no longer U2.27 (HPOUT_L)
- net MIC_IN renamed RF_AUDIO_INPUT
- net RF_AUDIO_INPUT: no longer C17.2
- net MIC_out: no longer names the net of C20.1
- net MIC_out: now also J7.3 (Pin_3); no longer U7.6 (MICOUT)
- net esp audio renamed esp_audio_OUTPUT
- net esp_audio_OUTPUT: now also C17.2; no longer J3.3 (Pin_3), U9.1
- new net MIC_AMPLIFIER_OUTPUT: J7.4 (Pin_4), U7.6 (MICOUT)
- no-connect marks 19 -> 32
Other:
- title: (none) -> Cross band handy walkie talkie
- moved on the sheet: J2, J3, U8A

Commit message: k
Parts:
- added TP1, TP10, TP2, TP3, TP4, TP5, TP6, TP7, TP8, TP9: TestPoint, TestPoint:TestPoint_Pad_1.5x1.5mm, symbol Connector:TestPoint
Connections:
- net GND: now also TP10.1
- net GPIO_22: now also TP7.1
- net HBIAS: now reaches U2.13 (HBIAS)
- net HBIAS: now also TP6.1
- net MIC2P: now reaches U2.14 (MIC2_N)
- net MIC2P: now also TP5.1
- net MIC2N: now reaches U2.15 (MIC2_P)
- net MIC2N: now also TP4.1
- net MBIAS: now reaches U2.16 (MBIAS)
- net MBIAS: now also TP3.1
- net MIC1P: now reaches U2.17 (MIC1P)
- net MIC1P: now also TP2.1
- net MIC1N: now reaches U2.18 (MIC1N)
- net MIC1N: now also TP1.1
- net SENSOR_VN: now reaches U2.3 (SENSOR_VN)
- net SENSOR_VN: now also TP9.1
- net SENSOR_VP: now reaches U2.4 (SENSOR_VP)
- net SENSOR_VP: now also TP8.1
- no-connect marks 32 -> 25
