File: HW/cross_band_handy_walkie_talkie_V1/cross_band_handy_walkie_talkie_V1.kicad_sch (KiCad schematic)
At the start: 108 parts, among them J1 Conn_01x06, J14 SMA, J15 SMA, J2 Conn_01x03, J3 Conn_01x03, J4 Conn_01x03, J5 Conn_01x03, J6 USB_C_Receptacle, J7 Conn_01x04, J8 RFShield_OnePiece, J9 Conn_01x02, Q1 MMBT3904, Q2 MMBT3904, SW1 MCU_RESET, U1 CH340C, U10 LM386, U11 TS5A63157DBV, U12 TS5A63157DBV, U13 SA818S, U14 SA818S, U2 ESP32-A1S, U3 AMS1117-3.3, U4 PCA9554APW, U7 MAX9814, U8 TS5A63157DBV, U9 TS5A63157DBV

Commit message: g
Parts:
- C15: value 10p -> 15p; LCSC (none) -> C1644
- C17, C19, C20, C24, C27, C28: LCSC (none) -> C15849
- C29: value 1u-10u? -> 1u; LCSC (none) -> C15849
- C30: LCSC (none) -> C1622
- C8: LCSC (none) -> C1644
- R1, R12, R14, R3: LCSC (none) -> C23186
- R10, R5, R9: LCSC (none) -> C23025
- R11, R2, R4: LCSC (none) -> C25804
- R16, R7: LCSC (none) -> C22935
- R17: LCSC C17407 -> C149504
- SW1: LCSC (none) -> C318884
Other:
- moved on the sheet: C8
Changed lines of the file:
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@@
   (junction (at 190.5 388.62) (diameter 0) (color 0 0 0 0)
   )
+  (junction (at 278.13 113.03) (diameter 0) (color 0 0 0 0)
+  )
   (junction (at 139.7 208.28) (diameter 0) (color 0 0 0 0)
   )
@@
   (junction (at 269.24 113.03) (diameter 0) (color 0 0 0 0)
   )
-  (junction (at 276.86 113.03) (diameter 0) (color 0 0 0 0)
-  )
   (junction (at 181.61 62.23) (diameter 0) (color 0 0 0 0)
   )
@@
     (stroke (width 0) (type default) (color 0 0 0 0))
   )
-  (wire (pts (xy 276.86 123.19) (xy 276.86 125.73))
+  (wire (pts (xy 278.13 123.19) (xy 278.13 125.73))
     (stroke (width 0) (type default) (color 0 0 0 0))
   )
@@
     (stroke (width 0) (type default) (color 0 0 0 0))
   )
-  (wire (pts (xy 276.86 118.11) (xy 276.86 113.03))
+  (wire (pts (xy 278.13 118.11) (xy 278.13 113.03))
     (stroke (width 0) (type default) (color 0 0 0 0))
   )
@@
     (stroke (width 0) (type default) (color 0 0 0 0))
   )
-  (wire (pts (xy 276.86 113.03) (xy 289.56 113.03))
-    (stroke (width 0) (type default) (color 0 0 0 0))
-  )
   (polyline (pts (xy 260.35 321.31) (xy 260.35 400.05))
     (stroke (width 0) (type default) (color 0 0 0 0))
@@
     (stroke (width 0) (type default) (color 0 0 0 0))
   )
+  (wire (pts (xy 278.13 113.03) (xy 289.56 113.03))
+    (stroke (width 0) (type default) (color 0 0 0 0))
+  )
   (wire (pts (xy 99.06 345.44) (xy 104.14 345.44))
     (stroke (width 0) (type default) (color 0 0 0 0))
@@
     (stroke (width 0) (type default) (color 0 0 0 0))
   )
-  (wire (pts (xy 269.24 113.03) (xy 276.86 113.03))
+  (wire (pts (xy 269.24 113.03) (xy 278.13 113.03))
     (stroke (width 0) (type default) (color 0 0 0 0))
   )
@@
       (effects (font (size 1.27 1.27)) hide)
     )
+    (property "LCSC" "C25804" (id 4) (at 273.05 78.74 90)
+      (effects (font (size 1.27 1.27)) hide)
+    )
     (pin "1")
     (pin "2")
@@
       (effects (font (size 1.27 1.27)) hide)
     )
+    (property "LCSC" "C15849" (id 4) (at 160.02 233.68 90)
+      (effects (font (size 1.27 1.27)) hide)
+    )
     (pin "1")
     (pin "2")
@@
       (effects (font (size 1.27 1.27)) hide)
     )
+    (property "LCSC" "C22935" (id 4) (at 231.14 138.43 0)
+      (effects (font (size 1.27 1.27)) hide)
+    )
     (pin "1")
     (pin "2")
@@
       (effects (font (size 1.27 1.27)) hide)
     )
+    (property "LCSC" "C1622" (id 4) (at 368.3 278.13 0)
+      (effects (font (size 1.27 1.27)) hide)
+    )
     (pin "1")
     (pin "2")
@@
       (effects (font (size 1.27 1.27)) hide)
     )
+    (property "LCSC" "C22935" (id 4) (at 264.16 113.03 90)
+      (effects (font (size 1.27 1.27)) hide)
+    )
     (pin "1")
     (pin "2")
@@
       (effects (font (size 1.27 1.27)) hide)
     )
+    (property "LCSC" "C15849" (id 4) (at 83.82 133.35 90)
+      (effects (font (size 1.27 1.27)) hide)
+    )
     (pin "1")
     (pin "2")
@@
       (effects (font (size 1.27 1.27)) hide)
     )
+    (property "LCSC" "C23186" (id 4) (at 212.09 276.86 90)
+      (effects (font (size 1.27 1.27)) hide)
+    )
     (pin "1")
     (pin "2")
@@
       (effects (font (size 1.27 1.27)) (justify left))
     )
-    (property "Value" "10p" (id 1) (at 228.6 139.7 0)
+    (property "Value" "15p" (id 1) (at 228.6 139.7 0)
       (effects (font (size 1.27 1.27)) (justify left))
     )
@@
       (effects (font (size 1.27 1.27)) hide)
     )
+    (property "LCSC" "C1644" (id 4) (at 222.25 138.43 0)
+      (effects (font (size 1.27 1.27)) hide)
+    )
     (pin "1")
     (pin "2")
@@
       (effects (font (size 1.27 1.27)) hide)
     )
+    (property "LCSC" "C23025" (id 4) (at 154.94 138.43 0)
+      (effects (font (size 1.27 1.27)) hide)
+    )
     (pin "1")
     (pin "2")
@@
       (effects (font (size 1.27 1.27)) hide)
     )
+    (property "LCSC" "C318884" (id 4) (at 289.56 118.11 90)
+      (effects (font (size 1.27 1.27)) hide)
+    )
     (pin "1")
     (pin "2")
@@
       (effects (font (size 1.27 1.27)) hide)
     )
+    (property "LCSC" "C25804" (id 4) (at 271.78 140.97 90)
+      (effects (font (size 1.27 1.27)) hide)
+    )
     (pin "1")
     (pin "2")
@@
       (effects (font (size 1.27 1.27)) hide)
     )
+    (property "LCSC" "C15849" (id 4) (at 309.88 255.27 90)
+      (effects (font (size 1.27 1.27)) hide)
+    )
     (pin "1")
     (pin "2")
@@
       (effects (font (size 1.27 1.27)) hide)
     )
+    (property "LCSC" "C15849" (id 4) (at 83.82 118.11 90)
+      (effects (font (size 1.27 1.27)) hide)
+    )
     (pin "1")
     (pin "2")
@@
       (effects (font (size 1.27 1.27)) hide)
     )
+    (property "LCSC" "C23025" (id 4) (at 171.45 138.43 0)
+      (effects (font (size 1.27 1.27)) hide)
+    )
     (pin "1")
     (pin "2")
@@
       (effects (font (size 1.27 1.27)) hide)
     )
-    (property "LCSC" "C17407" (id 4) (at 68.58 260.35 0)
+    (property "LCSC" "C149504" (id 4) (at 68.58 260.35 0)
       (effects (font (size 1.27 1.27)) hide)
     )
@@
       (effects (font (size 1.27 1.27)) hide)
     )
+    (property "LCSC" "C15849" (id 4) (at 350.52 252.73 0)
+      (effects (font (size 1.27 1.27)) hide)
+    )
     (pin "1")
     (pin "2")
@@
       (effects (font (size 1.27 1.27)) (justify left))
     )
-    (property "Value" "1u-10u?" (id 1) (at 355.6 279.4 0)
+    (property "Value" "1u" (id 1) (at 355.6 279.4 0)
       (effects (font (size 1.27 1.27)) (justify left))
     )
@@
       (effects (font (size 1.27 1.27)) hide)
     )
+    (property "LCSC" "C15849" (id 4) (at 353.06 278.13 0)
+      (effects (font (size 1.27 1.27)) hide)
+    )
     (pin "1")
     (pin "2")
@@
       (effects (font (size 1.27 1.27)) hide)
     )
+    (property "LCSC" "C15849" (id 4) (at 378.46 265.43 90)
+      (effects (font (size 1.27 1.27)) hide)
+    )
     (pin "1")
     (pin "2")
@@
     (pin "1")
   )
-  (symbol (lib_id "power:GND") (at 276.86 125.73 0) (unit 1)
+  (symbol (lib_id "power:GND") (at 278.13 125.73 0) (unit 1)
     (in_bom yes) (on_board yes) (fields_autoplaced)
-    (property "Reference" "#PWR020" (id 0) (at 276.86 132.08 0)
+    (property "Reference" "#PWR020" (id 0) (at 278.13 132.08 0)
       (effects (font (size 1.27 1.27)) hide)
     )
-    (property "Value" "GND" (id 1) (at 276.86 130.81 0)
+    (property "Value" "GND" (id 1) (at 278.13 130.81 0)
       (effects (font (size 1.27 1.27)) hide)
     )
-    (property "Footprint" "" (id 2) (at 276.86 125.73 0)
+    (property "Footprint" "" (id 2) (at 278.13 125.73 0)
       (effects (font (size 1.27 1.27)) hide)
     )
-    (property "Datasheet" "" (id 3) (at 276.86 125.73 0)
+    (property "Datasheet" "" (id 3) (at 278.13 125.73 0)
       (effects (font (size 1.27 1.27)) hide)
     )
@@
       (effects (font (size 1.27 1.27)) hide)
     )
+    (property "LCSC" "C23186" (id 4) (at 189.23 69.85 90)
+      (effects (font (size 1.27 1.27)) hide)
+    )
     (pin "1")
     (pin "2")
@@
       (effects (font (size 1.27 1.27)) hide)
     )
+    (property "LCSC" "C23186" (id 4) (at 186.69 276.86 90)
+      (effects (font (size 1.27 1.27)) hide)
+    )
     (pin "1")
     (pin "2")
@@
       (effects (font (size 1.27 1.27)) hide)
     )
+    (property "LCSC" "C23186" (id 4) (at 189.23 67.31 90)
+      (effects (font (size 1.27 1.27)) hide)
+    )
     (pin "1")
     (pin "2")
@@
       (effects (font (size 1.27 1.27)) hide)
     )
+    (property "LCSC" "C23025" (id 4) (at 149.86 138.43 0)
+      (effects (font (size 1.27 1.27)) hide)
+    )
     (pin "1")
     (pin "2")
@@
       (effects (font (size 1.27 1.27)) hide)
     )
+    (property "LCSC" "C25804" (id 4) (at 273.05 60.96 90)
+      (effects (font (size 1.27 1.27)) hide)
+    )
     (pin "1")
     (pin "2")
@@
     (pin "6")
   )
-  (symbol (lib_id "Device:C_Small") (at 276.86 120.65 0) (unit 1)
+  (symbol (lib_id "Device:C_Small") (at 278.13 120.65 0) (unit 1)
     (in_bom yes) (on_board yes) (fields_autoplaced)
-    (property "Reference" "C8" (id 0) (at 279.4 119.3862 0)
+    (property "Reference" "C8" (id 0) (at 280.67 119.3862 0)
       (effects (font (size 1.27 1.27)) (justify left))
     )
-    (property "Value" "15n" (id 1) (at 279.4 121.9262 0)
+    (property "Value" "15n" (id 1) (at 280.67 121.9262 0)
       (effects (font (size 1.27 1.27)) (justify left))
     )
-    (property "Footprint" "Capacitor_SMD:C_0603_1608Metric_Pad1.08x0.95mm_HandSolder" (id 2) (at 276.86 120.65 0)
+    (property "Footprint" "Capacitor_SMD:C_0603_1608Metric_Pad1.08x0.95mm_HandSolder" (id 2) (at 278.13 120.65 0)
+      (effects (font (size 1.27 1.27)) hide)
+    )
+    (property "Datasheet" "~" (id 3) (at 278.13 120.65 0)
       (effects (font (size 1.27 1.27)) hide)
     )
-    (property "Datasheet" "~" (id 3) (at 276.86 120.65 0)
+    (property "LCSC" "C1644" (id 4) (at 278.13 120.65 0)
       (effects (font (size 1.27 1.27)) hide)
     )
@@
     )
     (path "/42afdb3d-94ce-48ca-995e-1afadc59de21"
-      (reference "C15") (unit 1) (value "10p") (footprint "Capacitor_SMD:C_0603_1608Metric_Pad1.08x0.95mm_HandSolder")
+      (reference "C15") (unit 1) (value "15p") (footprint "Capacitor_SMD:C_0603_1608Metric_Pad1.08x0.95mm_HandSolder")
     )
     (path "/2bdcbae0-d12a-462d-b7e3-bf20d9c57840"
@@
     )
     (path "/9ae5d04d-cbac-4f5d-8e42-4a41d9fbade2"
-      (reference "C29") (unit 1) (value "1u-10u?") (footprint "Capacitor_SMD:C_0603_1608Metric_Pad1.08x0.95mm_HandSolder")
+      (reference "C29") (unit 1) (value "1u") (footprint "Capacitor_SMD:C_0603_1608Metric_Pad1.08x0.95mm_HandSolder")
     )
     (path "/28e4fe5b-ce72-4a20-8aa4-41762ee2dcb8"

Commit message: v1
Parts:
- added U5: SRV05-4, Package_TO_SOT_SMD:SOT-23-6, symbol Power_Protection:SRV05-4
- U3: LCSC C347222 -> C6186
Connections:
- net +5V: now also U5.5 (VP)
- net D+: now also U5.1 (IO1)
- net D-: now also U5.6 (IO4)
- net GND: now also U5.2 (VN)
- no-connect marks 25 -> 27
Changed lines of the file:
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@@
   (no_connect (at 146.05 90.17))
   (no_connect (at 146.05 97.79))
+  (no_connect (at 100.33 58.42))
   (no_connect (at 199.39 118.11))
   (no_connect (at 199.39 102.87))
@@
   (no_connect (at 199.39 97.79))
   (no_connect (at 74.93 130.81))
+  (no_connect (at 125.73 53.34))
   (no_connect (at 146.05 87.63))
   (no_connect (at 529.59 254))
@@
     (stroke (width 0) (type default) (color 0 0 0 0))
   )
+  (wire (pts (xy 95.25 53.34) (xy 100.33 53.34))
+    (stroke (width 0) (type default) (color 0 0 0 0))
+  )
   (wire (pts (xy 45.72 238.76) (xy 48.26 238.76))
     (stroke (width 0) (type default) (color 0 0 0 0))
@@
     (stroke (width 0) (type default) (color 0 0 0 0))
   )
+  (wire (pts (xy 113.03 40.64) (xy 113.03 43.18))
+    (stroke (width 0) (type default) (color 0 0 0 0))
+  )
   (polyline (pts (xy 469.9 295.91) (xy 570.23 295.91))
     (stroke (width 0) (type default) (color 0 0 0 0))
@@
     (stroke (width 0) (type default) (color 0 0 0 0))
   )
+  (wire (pts (xy 130.81 58.42) (xy 125.73 58.42))
+    (stroke (width 0) (type default) (color 0 0 0 0))
+  )
   (wire (pts (xy 345.44 387.35) (xy 342.9 387.35))
     (stroke (width 0) (type default) (color 0 0 0 0))
@@
     (stroke (width 0) (type default) (color 0 0 0 0))
   )
+  (wire (pts (xy 113.03 69.85) (xy 113.03 68.58))
+    (stroke (width 0) (type default) (color 0 0 0 0))
+  )
   (wire (pts (xy 158.75 72.39) (xy 158.75 69.85))
     (stroke (width 0) (type default) (color 0 0 0 0))
@@
     )
   )
+  (global_label "D-" (shape input) (at 130.81 58.42 0) (fields_autoplaced)
+    (effects (font (size 1.27 1.27)) (justify left))
+    (property "Intersheet References" "${INTERSHEET_REFS}" (id 0) (at 136.0655 58.3406 0)
+      (effects (font (size 1.27 1.27)) (justify left) hide)
+    )
+  )
   (global_label "AUDIO_ON1" (shape input) (at 111.76 360.68 0) (fields_autoplaced)
     (effects (font (size 1.27 1.27) (thickness 0.254) bold italic) (justify left))
@@
     )
   )
+  (global_label "D+" (shape input) (at 95.25 53.34 180) (fields_autoplaced)
+    (effects (font (size 1.27 1.27)) (justify right))
+    (property "Intersheet References" "${INTERSHEET_REFS}" (id 0) (at 89.9945 53.4194 0)
+      (effects (font (size 1.27 1.27)) (justify right) hide)
+    )
+  )
   (global_label "PTT2" (shape input) (at 497.84 256.54 0) (fields_autoplaced)
     (effects (font (size 1.27 1.27) (thickness 0.254) bold italic) (justify left))
@@
       (effects (font (size 1.27 1.27)) hide)
     )
-    (property "LCSC" "C347222" (id 4) (at 265.43 196.85 0)
+    (property "LCSC" "C6186" (id 4) (at 265.43 196.85 0)
       (effects (font (size 1.27 1.27)) hide)
     )
@@
     (pin "1")
   )
+  (symbol (lib_id "power:GND") (at 113.03 69.85 0) (unit 1)
+    (in_bom yes) (on_board yes) (fields_autoplaced)
+    (property "Reference" "#PWR0116" (id 0) (at 113.03 76.2 0)
+      (effects (font (size 1.27 1.27)) hide)
+    )
+    (property "Value" "GND" (id 1) (at 113.03 74.93 0)
+      (effects (font (size 1.27 1.27)) hide)
+    )
+    (property "Footprint" "" (id 2) (at 113.03 69.85 0)
+      (effects (font (size 1.27 1.27)) hide)
+    )
+    (property "Datasheet" "" (id 3) (at 113.03 69.85 0)
+      (effects (font (size 1.27 1.27)) hide)
+    )
+    (pin "1")
+  )
   (symbol (lib_id "Device:C_Small") (at 252.73 201.93 0) (unit 1)
     (in_bom yes) (on_board yes)
@@
     (pin "1")
   )
+  (symbol (lib_id "Power_Protection:SRV05-4") (at 113.03 55.88 0) (unit 1)
+    (in_bom yes) (on_board yes) (fields_autoplaced)
+    (property "Reference" "U5" (id 0) (at 115.7987 40.64 0)
+      (effects (font (size 1.27 1.27)) (justify left))
+    )
+    (property "Value" "SRV05-4" (id 1) (at 115.7987 43.18 0)
+      (effects (font (size 1.27 1.27)) (justify left))
+    )
+    (property "Footprint" "Package_TO_SOT_SMD:SOT-23-6" (id 2) (at 130.81 67.31 0)
+      (effects (font (size 1.27 1.27)) hide)
+    )
+    (property "Datasheet" "http://www.onsemi.com/pub/Collateral/SRV05-4-D.PDF" (id 3) (at 113.03 55.88 0)
+      (effects (font (size 1.27 1.27)) hide)
+    )
+    (property "LCSC" "C85364" (id 4) (at 113.03 55.88 0)
+      (effects (font (size 1.27 1.27)) hide)
+    )
+    (pin "1")
+    (pin "2")
+    (pin "3")
+    (pin "4")
+    (pin "5")
+    (pin "6")
+  )
   (symbol (lib_id "Device:R_Small") (at 189.23 69.85 270) (mirror x) (unit 1)
     (in_bom yes) (on_board yes)
@@
     (pin "1")
   )
+  (symbol (lib_id "power:+5V") (at 113.03 40.64 0) (mirror y) (unit 1)
+    (in_bom yes) (on_board yes) (fields_autoplaced)
+    (property "Reference" "#PWR0117" (id 0) (at 113.03 44.45 0)
+      (effects (font (size 1.27 1.27)) hide)
+    )
+    (property "Value" "+5V" (id 1) (at 113.03 35.56 0))
+    (property "Footprint" "" (id 2) (at 113.03 40.64 0)
+      (effects (font (size 1.27 1.27)) hide)
+    )
+    (property "Datasheet" "" (id 3) (at 113.03 40.64 0)
+      (effects (font (size 1.27 1.27)) hide)
+    )
+    (pin "1")
+  )
   (symbol (lib_id "Device:C_Small") (at 45.72 251.46 0) (unit 1)
     (in_bom yes) (on_board yes)
@@
       (reference "#PWR0115") (unit 1) (value "GND") (footprint "")
     )
+    (path "/af344fe8-6186-4007-aaac-c341a0133aea"
+      (reference "#PWR0116") (unit 1) (value "GND") (footprint "")
+    )
+    (path "/e610498a-8389-462d-98dc-3a2e8b4478ce"
+      (reference "#PWR0117") (unit 1) (value "+5V") (footprint "")
+    )
     (path "/8c509600-7f9c-4bfc-84b1-320113255391"
       (reference "C1") (unit 1) (value "100n") (footprint "Capacitor_SMD:C_0603_1608Metric_Pad1.08x0.95mm_HandSolder")
@@
       (reference "U4") (unit 1) (value "PCA9554APW") (footprint "Package_SO:TSSOP-16_4.4x5mm_P0.65mm")
     )
+    (path "/b4c25313-7d10-4dcb-a1da-1a9d03412eab"
+      (reference "U5") (unit 1) (value "SRV05-4") (footprint "Package_TO_SOT_SMD:SOT-23-6")
+    )
     (path "/e3ceac9e-20a1-4164-83dd-2889cc9f32ae"

Commit message: r
Parts:
- added JP2, JP3: ., Jumper:SolderJumper-3_P2.0mm_Open_TrianglePad1.0x1.5mm_NumberLabels, symbol Jumper:Jumper_3_Bridged12
- added R6: 300, Resistor_SMD:R_0603_1608Metric_Pad0.98x0.95mm_HandSolder, symbol Device:R_Small
- added TP11, TP12, TP13: TestPoint, TestPoint:TestPoint_Pad_1.5x1.5mm, symbol Connector:TestPoint
- C8: value 15n -> 1u; LCSC C1644 -> C15849
- R7: value 1Meg -> 10k; LCSC C22935 -> C25804
Connections:
- net -SLEEP: no longer U2.5 (IO_34)
- net GND: now also JP2.3 (B), JP3.3 (B), TP11.1, TP12.1, TP13.1; no longer C18.2, U7.8 (MICIN)
- net MIC-AMP_IN: no longer C18.1
- net MIC_BIAS: now also C18.2
- net PD1: now also JP2.1 (A); no longer U14.6 (PD)
- net PD2: now also JP3.1 (A); no longer U13.6 (PD)
- net RX1: no longer U2.8 (IO_12)
- net TX2: no longer U2.11 (IO_2)
- net UART0_TX: now also R6.1; no longer U1.3 (RXD)
- net ~{DTR}: now also U1.13 (~{DTR})
- net ~{RTS}: now also U1.14 (~{RTS})
- new net: JP2.2 (C), U14.6 (PD)
- new net: JP3.2 (C), U13.6 (PD)
- new net: R6.2, U1.3 (RXD)
- new net GPIO_02: U2.11 (IO_2)
- new net GPIO_12: U2.8 (IO_12)
- new net GPIO_34: U2.5 (IO_34)
- new net MIC_in: C18.1, U7.8 (MICIN)
- no-connect marks 27 -> 24
Other:
- note added: "10k & 1u"
- note added: "danger pin"
- note added: "danger pin, must be high on boot"
- note added: "input only"
- moved on the sheet: C20
