File: HW/cross_band_handy_walkie_talkie_V1/cross_band_handy_walkie_talkie_V1.kicad_pcb (KiCad board)
At the start: 2 copper layers, 37 parts, among them J2 Conn_Coaxial, J3 Conn_Coaxial, Q1 BC847BS, SW1 MCU_RESET, U1 CP2102N-Axx-xQFN24, U2 ESP32-S3-WROOM-1, U3 SA818S, U4 SA818S

Commit message: b
Parts:
- removed U2: ESP32-S3-WROOM-1, Espressif:ESP32-S3-WROOM-1
- added C14: 1u, Capacitor_SMD:C_0603_1608Metric_Pad1.08x0.95mm_HandSolder, F.Cu at (119.8, 162.7)
- added C15: 10u, Capacitor_SMD:C_0603_1608Metric_Pad1.08x0.95mm_HandSolder, F.Cu at (108.1, 172.3)
- added C16: 1u, Capacitor_SMD:C_0603_1608Metric_Pad1.08x0.95mm_HandSolder, F.Cu at (112.5, 171.2)
- added C17: 1uF, Capacitor_SMD:C_0805_2012Metric, F.Cu at (91.1, 182.5)
- added C18: 1u, Capacitor_SMD:C_0603_1608Metric_Pad1.08x0.95mm_HandSolder, F.Cu at (99.9, 181.2)
- added C19: 1uF, Capacitor_SMD:C_0805_2012Metric, F.Cu at (103.7, 169.5)
- added C20: 1nF, Capacitor_SMD:C_0805_2012Metric, F.Cu at (86.7, 182.5)
- added C21: 10uF, Capacitor_SMD:C_0805_2012Metric, F.Cu at (111.0, 162.9)
- added C22: 1uF, Capacitor_SMD:C_0805_2012Metric, F.Cu at (100.1, 175.9)
- added C23: 1u-10u?, Capacitor_SMD:C_0603_1608Metric_Pad1.08x0.95mm_HandSolder, F.Cu at (104.5, 177.7)
- added C24: 47n, Capacitor_SMD:C_0603_1608Metric_Pad1.08x0.95mm_HandSolder, F.Cu at (100.0, 178.7)
- added C25: 47nF, Capacitor_SMD:C_0805_2012Metric, F.Cu at (104.0, 166.5)
- added C26: 4u7, Capacitor_SMD:C_0603_1608Metric_Pad1.08x0.95mm_HandSolder, F.Cu at (108.8, 174.8)
- added C27: 4u7, Capacitor_SMD:C_0603_1608Metric_Pad1.08x0.95mm_HandSolder, F.Cu at (95.5, 183.4)
- added C28: 10u, Capacitor_SMD:C_0603_1608Metric_Pad1.08x0.95mm_HandSolder, F.Cu at (104.5, 175.2)
- added C29: 10u, Capacitor_SMD:C_0603_1608Metric_Pad1.08x0.95mm_HandSolder, F.Cu at (117.2, 165.6)
- added C30: 1uF, Capacitor_SMD:C_0805_2012Metric, F.Cu at (108.4, 166.5)
- added J4: Conn_01x03, Connector_PinHeader_2.54mm:PinHeader_1x03_P2.54mm_Vertical, F.Cu at (82.0, 163.8)
- added J5: Conn_01x03, Connector_PinHeader_2.54mm:PinHeader_1x03_P2.54mm_Vertical, F.Cu at (82.0, 173.5)
- added J6: Conn_01x03, Jumper:SolderJumper-3_P2.0mm_Open_TrianglePad1.0x1.5mm_NumberLabels, F.Cu at (105.3, 163.2)
- added JP1: jumper, Connector_PinHeader_2.54mm:PinHeader_1x03_P2.54mm_Vertical, F.Cu at (122.3, 148.8)
- added JP2: jumper, Connector_PinHeader_2.54mm:PinHeader_1x03_P2.54mm_Vertical, F.Cu at (117.6, 148.8)
- added L1: Ferrit, Resistor_SMD:R_0805_2012Metric_Pad1.20x1.40mm_HandSolder, F.Cu at (82.1, 182.5)
- added R14: 10, Resistor_SMD:R_0603_1608Metric_Pad0.98x0.95mm_HandSolder, F.Cu at (112.8, 168.6)
- added R15: 10R, Resistor_SMD:R_0805_2012Metric, F.Cu at (112.9, 165.9)
- added R16: #2.2k, Resistor_SMD:R_0805_2012Metric, F.Cu at (103.7, 172.5)
- added R17: 150k, Resistor_SMD:R_0805_2012Metric, F.Cu at (115.4, 162.9)
- added R18: 1k, Resistor_SMD:R_0805_2012Metric, F.Cu at (108.2, 169.5)
- added R19: 100k, Resistor_SMD:R_0805_2012Metric, F.Cu at (95.6, 180.7)
- added RV1: 10k, Potentiometer_SMD:Potentiometer_Vishay_TS53YL_Vertical, F.Cu at (88.9, 171.3)
- added RV2: 10k, Potentiometer_SMD:Potentiometer_Vishay_TS53YL_Vertical, F.Cu at (88.9, 164.7)
- added RV3: 10k, Potentiometer_SMD:Potentiometer_Vishay_TS53YL_Vertical, F.Cu at (97.6, 164.7)
- added U6: LM386, Package_SO:SOIC-8_3.9x4.9mm_P1.27mm, F.Cu at (97.3, 171.2)
- added U7: LT1129-3.3_SO8, Package_SO:SOIC-8_3.9x4.9mm_P1.27mm, F.Cu at (88.6, 177.8)
- added U8: MAX9814, Package_DFN_QFN:DFN-14-1EP_3x3mm_P0.4mm_EP1.78x2.35mm, F.Cu at (95.3, 176.9)
- C10: value DNP -> 2.2uF; footprint Capacitor_SMD:C_0603_1608Metric_Pad1.08x0.95mm_HandSolder -> Capacitor_SMD:C_0805_2012Metric
- C7, C8: value DNP -> 100nF; footprint Capacitor_SMD:C_0603_1608Metric_Pad1.08x0.95mm_HandSolder -> Capacitor_SMD:C_0805_2012Metric
- C9: value DNP -> 470nF; footprint Capacitor_SMD:C_0603_1608Metric_Pad1.08x0.95mm_HandSolder -> Capacitor_SMD:C_0805_2012Metric
- U4: moved to B.Cu
- turned U4 to 180 degrees
Connections:
- C7 pad 1: Net-(C7-Pad1) -> GND
- C7 pad 2: GND -> Net-(C7-Pad2)
- C8 pad 1: Net-(C8-Pad1) -> GND
- C8 pad 2: GND -> /MIC-AMP_IN
- J2 pad 1: Net-(C8-Pad1) -> Net-(J2-Pad1)
- J3 pad 1: Net-(C10-Pad1) -> Net-(J3-Pad1)
- R10 pad 1: Net-(C7-Pad1) -> Net-(R10-Pad1)
- R10 pad 2: Net-(C8-Pad1) -> Net-(J2-Pad1)
- R11 pad 1: Net-(C9-Pad1) -> Net-(R11-Pad1)
- R11 pad 2: Net-(C10-Pad1) -> Net-(J3-Pad1)
- U3 pad 1: unconnected-(U3-Pad1) -> Net-(U3-Pad1)
- U3 pad 12: Net-(C7-Pad1) -> Net-(R10-Pad1)
- U3 pad 3: unconnected-(U3-Pad3) -> Net-(U3-Pad3)
- U4 pad 1: unconnected-(U4-Pad1) -> Net-(U4-Pad1)
- U4 pad 12: Net-(C9-Pad1) -> Net-(R11-Pad1)
- U4 pad 3: unconnected-(U4-Pad3) -> Net-(U4-Pad3)
Other:
- board outline added: 125.4 x 69.7 mm

Commit message: v
Parts:
- removed C17, C19, C22: 1uF, Capacitor_SMD:C_0805_2012Metric
- removed C20: 1nF, Capacitor_SMD:C_0805_2012Metric
- removed C21: 10uF, Capacitor_SMD:C_0805_2012Metric
- removed C25: 47nF, Capacitor_SMD:C_0805_2012Metric
- removed JP1, JP2: jumper, Connector_PinHeader_2.54mm:PinHeader_1x03_P2.54mm_Vertical
- removed R10, R11: filter, Resistor_SMD:R_1206_3216Metric_Pad1.30x1.75mm_HandSolder
- removed R15: 10R, Resistor_SMD:R_0805_2012Metric
- removed RV2: 10k, Potentiometer_SMD:Potentiometer_Vishay_TS53YL_Vertical
- added FL1: LFCN-160, Filter:Filter_Mini-Circuits_FV1206, B.Cu at (143.2, 69.0)
- added FL2: LFCN-160, Filter:Filter_Mini-Circuits_FV1206, B.Cu at (57.5, 89.6)
- added H1: hole, MountingHole:MountingHole_3.2mm_M3_DIN965_Pad_TopBottom, F.Cu at (55.0, 55.0)
- added H2: hole, MountingHole:MountingHole_3.2mm_M3_DIN965_Pad_TopBottom, F.Cu at (145.0, 95.0)
- added H3: hole, MountingHole:MountingHole_3.2mm_M3_DIN965_Pad_TopBottom, F.Cu at (55.0, 95.0)
- added H4: hole, MountingHole:MountingHole_3.2mm_M3_DIN965_Pad_TopBottom, F.Cu at (145.0, 55.0)
- added J10: pin, Connector_PinHeader_2.54mm:PinHeader_1x01_P2.54mm_Vertical, F.Cu at (239.5, 118.9)
- added J11: pin, Connector_PinHeader_2.54mm:PinHeader_1x01_P2.54mm_Vertical, F.Cu at (247.0, 114.2)
- added J12: Conn_Coaxial, Connector_Coaxial:SMA_Amphenol_901-144_Vertical, F.Cu at (55.2, 81.6)
- added J7: pin, Connector_PinHeader_2.54mm:PinHeader_1x01_P2.54mm_Vertical, F.Cu at (242.3, 114.2)
- added J8: pin, Connector_PinHeader_2.54mm:PinHeader_1x01_P2.54mm_Vertical, F.Cu at (252.2, 107.4)
- added J9: pin, Connector_PinHeader_2.54mm:PinHeader_1x01_P2.54mm_Vertical, F.Cu at (244.1, 118.9)
- added U10: TS5A63157DBV, Package_TO_SOT_SMD:SOT-23-6, F.Cu at (229.8, 118.2)
- added U11: TS5A63157DBV, Package_TO_SOT_SMD:SOT-23-6, F.Cu at (242.6, 109.7)
- added U2: ESP32-A1S, Z_mycustom_footprint_lib:ESP32-A1S, F.Cu at (84.3, 58.4)
- added U9: TS5A63157DBV, Package_TO_SOT_SMD:SOT-23-6, F.Cu at (249.4, 73.0)
- J2: value Conn_Coaxial -> pin; footprint Connector_Coaxial:SMA_Amphenol_901-144_Vertical -> Connector_PinHeader_2.54mm:PinHeader_1x01_P2.54mm_Vertical
- U3: moved to B.Cu
- U6: value LM386 -> TS5A63157DBV; footprint Package_SO:SOIC-8_3.9x4.9mm_P1.27mm -> Package_TO_SOT_SMD:SOT-23-6
- moved D2 247.1 mm to (258.6, 72.0)
- moved R13 236.4 mm to (262.3, 77.1)
- moved C11 235.2 mm to (260.3, 108.7)
- moved C13 233.4 mm to (252.8, 82.4)
- moved C7 230.0 mm to (249.1, 76.7)
- moved U1 223.9 mm to (231.1, 108.2)
- moved FB1 219.6 mm to (234.8, 117.4)
- moved C9 217.1 mm to (251.5, 111.2)
- moved R3 216.3 mm to (272.2, 99.3)
- moved C1 216.2 mm to (248.6, 120.8)
- moved D1 208.4 mm to (229.1, 121.7)
- moved R9 202.6 mm to (263.0, 74.5)
- moved J2 202.1 mm to (247.5, 107.4)
- moved C12 199.5 mm to (267.3, 72.0)
- moved C2 196.3 mm to (272.2, 101.8)
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Connections:
- net VCC renamed /switch1
- C18 pad 2: /AUDIO_OUT -> AUDIO_OUT
- J2 pad 1: Net-(J2-Pad1) -> /esp audio
- U3 pad 1: Net-(U3-Pad1) -> AUDIO_ON1
- U3 pad 18: unconnected-(U3-Pad18) -> Net-(U3-Pad18)
- U4 pad 1: Net-(U4-Pad1) -> AUDIO_ON2
- U4 pad 18: unconnected-(U4-Pad18) -> Net-(U4-Pad18)
- U6 pad 1: Net-(C22-Pad1) -> /esp audio
- U6 pad 3: Net-(C20-Pad1) -> Net-(J6-Pad1)
- U6 pad 4: GND -> MIC_IN
- U6 pad 5: Net-(C19-Pad1) -> +3V3
Routing:
- added copper zone on In1.Cu, net GND
- added copper zone on In2.Cu, net GND
Other:
- board size 125.4 x 69.7 mm -> 100 x 50 mm
- copper layers 2 -> 4

Commit message: j
Parts:
- removed RV3: 10k, Potentiometer_SMD:Potentiometer_Vishay_TS53YL_Vertical
- added C17: 100n, Capacitor_SMD:C_0603_1608Metric_Pad1.08x0.95mm_HandSolder, F.Cu at (253.8, 71.0)
- added C19: 470nF, Capacitor_SMD:C_0805_2012Metric, F.Cu at (257.6, 55.1)
- added C20: 2.2uF, Capacitor_SMD:C_0805_2012Metric, F.Cu at (245.0, 70.7)
- added C21: 470n, Capacitor_SMD:C_0805_2012Metric, F.Cu at (262.0, 55.1)
- added C22: 2u2, Capacitor_SMD:C_0805_2012Metric, F.Cu at (227.2, 88.6)
- added C25: 10u, Capacitor_SMD:C_0805_2012Metric, F.Cu at (254.0, 62.8)
- added C31: 100n, Capacitor_SMD:C_0603_1608Metric_Pad1.08x0.95mm_HandSolder, F.Cu at (262.8, 63.0)
- added C32: 10u, Capacitor_SMD:C_0805_2012Metric, F.Cu at (235.7, 78.0)
- added C33: 10u, Capacitor_SMD:C_0805_2012Metric, F.Cu at (240.6, 73.7)
- added C34: 100n, Capacitor_SMD:C_0603_1608Metric_Pad1.08x0.95mm_HandSolder, F.Cu at (258.2, 66.3)
- added C35: 100n, Capacitor_SMD:C_0603_1608Metric_Pad1.08x0.95mm_HandSolder, F.Cu at (258.1, 71.3)
- added C36: 100n, Capacitor_SMD:C_0603_1608Metric_Pad1.08x0.95mm_HandSolder, F.Cu at (240.3, 87.3)
- added C37: 100n, Capacitor_SMD:C_0603_1608Metric_Pad1.08x0.95mm_HandSolder, F.Cu at (231.6, 88.2)
- added C38: 100n, Capacitor_SMD:C_0603_1608Metric_Pad1.08x0.95mm_HandSolder, F.Cu at (270.8, 54.9)
- added J13: pin, Connector_PinHeader_2.54mm:PinHeader_1x01_P2.54mm_Vertical, F.Cu at (253.0, 55.9)
- added J14: Conn_Coaxial, Connector_Coaxial:SMA_Amphenol_901-144_Vertical, F.Cu at (145.0, 77.0)
- added J15: Conn_Coaxial, Connector_Coaxial:SMA_Amphenol_901-144_Vertical, F.Cu at (55.5, 81.5)
- added L2: Ferrit, Resistor_SMD:R_0805_2012Metric_Pad1.20x1.40mm_HandSolder, F.Cu at (225.3, 71.3)
- added Q2: MMBT3904, Package_TO_SOT_SMD:SOT-23, F.Cu at (231.3, 74.1)
- added R10: 300, Resistor_SMD:R_0603_1608Metric_Pad0.98x0.95mm_HandSolder, F.Cu at (267.2, 57.8)
- added R11: 10k, Resistor_SMD:R_0603_1608Metric_Pad0.98x0.95mm_HandSolder, F.Cu at (258.1, 68.8)
- added R15: 150k, Resistor_SMD:R_0805_2012Metric, F.Cu at (266.4, 55.1)
- added R20: 10, Resistor_SMD:R_0603_1608Metric_Pad0.98x0.95mm_HandSolder, F.Cu at (262.8, 60.5)
- added RV2: 10k, Potentiometer_SMD:Potentiometer_Vishay_TS53YL_Vertical, F.Cu at (227.5, 66.6)
- added U12: TS5A63157DBV, Package_TO_SOT_SMD:SOT-23-6, F.Cu at (234.2, 69.6)
- added U13: SA818S, Z_mycustom_footprint_lib:SA818S, B.Cu at (129.8, 78.2)
- added U14: SA818S, Z_mycustom_footprint_lib:SA818S, B.Cu at (70.8, 79.5)
- added U5: PCA9555PW, Package_SO:TSSOP-24_4.4x7.8mm_P0.65mm, F.Cu at (232.7, 58.3)
- C10: value 2.2uF -> 10u
- C11: value DNP -> 100n
- C12: value 15n -> 100n
- C13, C2: value 100n -> 10u; footprint Capacitor_SMD:C_0603_1608Metric_Pad1.08x0.95mm_HandSolder -> Capacitor_SMD:C_0805_2012Metric
- C14: value 1u -> 10u; footprint Capacitor_SMD:C_0603_1608Metric_Pad1.08x0.95mm_HandSolder -> Capacitor_SMD:C_0805_2012Metric
- C15, C4: value 10u -> 100n
- C16, C18: value 1u -> 100n
- C23: value 1u-10u? -> 1uF; footprint Capacitor_SMD:C_0603_1608Metric_Pad1.08x0.95mm_HandSolder -> Capacitor_SMD:C_0805_2012Metric
- C24: value 47n -> 1u
- C26: value 4u7 -> 10u; footprint Capacitor_SMD:C_0603_1608Metric_Pad1.08x0.95mm_HandSolder -> Capacitor_SMD:C_0805_2012Metric
- C27: value 4u7 -> 1u
- C28: value 10u -> 1u
- C29: value 10u -> 1u-10u?
- C3: footprint Capacitor_SMD:C_0603_1608Metric_Pad1.08x0.95mm_HandSolder -> Capacitor_SMD:C_0805_2012Metric
- C30: value 1uF -> 47n; footprint Capacitor_SMD:C_0805_2012Metric -> Capacitor_SMD:C_0603_1608Metric_Pad1.08x0.95mm_HandSolder
- C7: value 100nF -> DNP; footprint Capacitor_SMD:C_0805_2012Metric -> Capacitor_SMD:C_0603_1608Metric_Pad1.08x0.95mm_HandSolder
- C8: value 100nF -> 15n; footprint Capacitor_SMD:C_0805_2012Metric -> Capacitor_SMD:C_0603_1608Metric_Pad1.08x0.95mm_HandSolder
- C9: value 470nF -> 10u
- J11, J7: value pin -> Conn_01x03; footprint Connector_PinHeader_2.54mm:PinHeader_1x01_P2.54mm_Vertical -> Jumper:SolderJumper-3_P2.0mm_Open_TrianglePad1.0x1.5mm_NumberLabels
- J12: value Conn_Coaxial -> pin; footprint Connector_Coaxial:SMA_Amphenol_901-144_Vertical -> Connector_PinHeader_2.54mm:PinHeader_1x01_P2.54mm_Vertical
- J2: value pin -> Conn_01x03; footprint Connector_PinHeader_2.54mm:PinHeader_1x01_P2.54mm_Vertical -> Connector_PinHeader_2.54mm:PinHeader_1x03_P2.54mm_Vertical
- J3: value Conn_Coaxial -> Conn_01x03; footprint Connector_Coaxial:SMA_Amphenol_901-144_Vertical -> Connector_PinHeader_2.54mm:PinHeader_1x03_P2.54mm_Vertical
- J6: value Conn_01x03 -> pin; footprint Jumper:SolderJumper-3_P2.0mm_Open_TrianglePad1.0x1.5mm_NumberLabels -> Connector_PinHeader_2.54mm:PinHeader_1x01_P2.54mm_Vertical
- Q1: value BC847BS -> MMBT3904; footprint Package_TO_SOT_SMD:SOT-363_SC-70-6_Handsoldering -> Package_TO_SOT_SMD:SOT-23
- R12: value 1Meg -> #2.2k; footprint Resistor_SMD:R_0603_1608Metric_Pad0.98x0.95mm_HandSolder -> Resistor_SMD:R_0805_2012Metric
- R13: value 10k -> 2k2; footprint Resistor_SMD:R_0603_1608Metric_Pad0.98x0.95mm_HandSolder -> Resistor_SMD:R_0805_2012Metric
- R14: value 10 -> 150k; footprint Resistor_SMD:R_0603_1608Metric_Pad0.98x0.95mm_HandSolder -> Resistor_SMD:R_0805_2012Metric
- R16: value #2.2k -> 1k
- R17: value 150k -> 100k
- R18: value 1k -> 100k
- R19: value 100k -> 1k
- R2: value 22k -> 10k
- R3: value 47k -> 22k
- R5: value 300 -> 1Meg
- R6: value 300 -> 47k
- R9: value 10k -> 300
- U10: value TS5A63157DBV -> LM386; footprint Package_TO_SOT_SMD:SOT-23-6 -> Package_SO:SOIC-8-1EP_3.9x4.9mm_P1.27mm_EP2.41x3.3mm_ThermalVias
- U3: value SA818S -> AMS1117-3.3; footprint Z_mycustom_footprint_lib:SA818S -> Package_TO_SOT_SMD:SOT-223-3_TabPin2; moved to F.Cu
- U4: value SA818S -> PCA9554APW; footprint Z_mycustom_footprint_lib:SA818S -> Package_SO:TSSOP-16_4.4x5mm_P0.65mm; moved to F.Cu
- U6: value TS5A63157DBV -> MAX9814; footprint Package_TO_SOT_SMD:SOT-23-6 -> Package_DFN_QFN:DFN-14-1EP_3x3mm_P0.4mm_EP1.78x2.35mm
- U7: value LT1129-3.3_SO8 -> MAX9814; footprint Package_SO:SOIC-8_3.9x4.9mm_P1.27mm -> Package_DFN_QFN:DFN-14-1EP_3x3mm_P0.4mm_EP1.78x2.35mm
- U8: value MAX9814 -> TS5A63157DBV; footprint Package_DFN_QFN:DFN-14-1EP_3x3mm_P0.4mm_EP1.78x2.35mm -> Package_TO_SOT_SMD:SOT-23-6
- moved J12 181.0 mm to (236.0, 74.2)
- moved U3 143.5 mm to (213.4, 66.0), turned to 0 degrees
- moved U4 83.1 mm to (212.8, 83.2), turned to 0 degrees
- moved J3 79.8 mm to (221.4, 55.9)
- moved U10 62.4 mm to (241.3, 56.8)
- moved R14 59.1 mm to (258.4, 58.1)
- moved C30 58.6 mm to (262.5, 68.8)
- moved J9 58.5 mm to (249.5, 60.6)
- moved C4 57.9 mm to (271.5, 60.3)
- moved J2 55.7 mm to (226.0, 55.9)
- moved C5 54.7 mm to (267.2, 60.5)
- moved U11 54.1 mm to (248.1, 55.8)
- moved D1 52.1 mm to (215.3, 71.5)
- moved SW1 51.6 mm to (214.0, 57.8)
- moved U8 49.0 mm to (239.7, 62.3)
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Connections:
- C1 pad 1: /VDD_CP -> +3V3
- C10 pad 1: Net-(C10-Pad1) -> +3V3
- C11 pad 1: /EN -> /BOOT
- C12 pad 1: /EN -> +3V3
- C13 pad 1: /BOOT -> Net-(C13-Pad1)
- C14 pad 1: Net-(C14-Pad1) -> +3V3
- C15 pad 1: +5V -> Net-(U6-Pad1)
- C16 pad 1: /AUDIO_IN -> Net-(C16-Pad1)
- C16 pad 2: Net-(C16-Pad2) -> GND
- C18 pad 1: Net-(C18-Pad1) -> /MIC-AMP_IN
- C18 pad 2: AUDIO_OUT -> GND
- C2 pad 1: /~{RST_CP} -> +3V3
- C23 pad 1: Net-(C23-Pad1) -> GND
- C27 pad 1: +3V3 -> /AUDIO_IN
- C27 pad 2: GND -> Net-(C27-Pad2)
- C28 pad 1: GND -> Net-(C28-Pad1)
- C28 pad 2: +5V -> AUDIO_OUT
- C29 pad 1: GND -> Net-(C29-Pad1)
- C29 pad 2: +5V -> Net-(C29-Pad2)
- C30 pad 1: GND -> Net-(C30-Pad1)
- C30 pad 2: Net-(C30-Pad2) -> GND
- C4 pad 1: +3V3 -> /VDD_CP
- C5 pad 1: +3V3 -> /~{RST_CP}
- C7 pad 1: GND -> /EN
- C7 pad 2: Net-(C7-Pad2) -> GND
- C8 pad 1: GND -> /EN
- C8 pad 2: /MIC-AMP_IN -> GND
- C9 pad 1: Net-(C9-Pad1) -> +5V
- FL1 pad 1: Net-(U4-Pad12) -> Net-(FL1-Pad1)
- FL1 pad 3: Net-(J3-Pad1) -> Net-(FL1-Pad3)
- FL2 pad 1: Net-(U3-Pad12) -> Net-(FL2-Pad1)
- J10 pad 1: AUDIO_OUT -> /esp audio
- J11 pad 1: /AUDIO_IN -> Net-(J11-Pad1)
- J12 pad 1: Net-(FL2-Pad3) -> AUDIO_OUT
- J2 pad 1: /esp audio -> GND
- J3 pad 1: Net-(J3-Pad1) -> GND
- J3 pad 2: GND -> /MIC_AR
- J6 pad 1: Net-(J6-Pad1) -> /esp audio
- J7 pad 1: MIC_IN -> Net-(J7-Pad1)
- J8 pad 1: Net-(J6-Pad1) -> MIC_IN
- J9 pad 1: /esp audio -> Net-(J11-Pad1)
- L1 pad 1: +3V3 -> Net-(C13-Pad1)
- L1 pad 2: Net-(C30-Pad2) -> +3V3
- Q1 pad 1: /~{RTS} -> /BASE1
- Q1 pad 2: /BASE1 -> /~{RTS}
- Q1 pad 3: /BOOT -> /EN
- R12 pad 1: /EN -> GND
- R12 pad 2: +3V3 -> /MIC-AMP_IN
- R13 pad 1: /BOOT -> GND
- R13 pad 2: +3V3 -> /MIC-AMP_IN
- R14 pad 1: Net-(C24-Pad1) -> GND
- R14 pad 2: Net-(C18-Pad1) -> Net-(R14-Pad2)
- R16 pad 1: GND -> Net-(R16-Pad1)
- R16 pad 2: /MIC-AMP_IN -> /MIC_GAIN
- R17 pad 1: GND -> Net-(R15-Pad2)
- R17 pad 2: Net-(R17-Pad2) -> GND
- R18 pad 1: Net-(R18-Pad1) -> Net-(R14-Pad2)
- R18 pad 2: /MIC_GAIN -> GND
- R19 pad 1: Net-(R17-Pad2) -> /MIC_GAIN_pin
- R19 pad 2: GND -> /MIC_GAIN
- R2 pad 1: +5V -> /BASE1
- R2 pad 2: /VBUS_DETECT_CP -> /~{DTR}
- R3 pad 1: /VBUS_DETECT_CP -> +5V
- R3 pad 2: GND -> /VBUS_DETECT_CP
- R4 pad 1: Net-(R4-Pad1) -> /~{RTS}
- R4 pad 2: GND -> /BASE2
- R5 pad 1: /TXT -> GND
- R5 pad 2: Net-(D1-Pad1) -> Net-(C6-Pad1)
- R6 pad 1: /RXT -> /VBUS_DETECT_CP
- R6 pad 2: Net-(D2-Pad1) -> GND
- R7 pad 1: GND -> /EN
- R7 pad 2: Net-(C6-Pad1) -> +3V3
- R8 pad 1: /BASE1 -> Net-(R8-Pad1)
- R8 pad 2: /~{DTR} -> GND
- R9 pad 1: /~{RTS} -> /TXT
- R9 pad 2: /BASE2 -> Net-(D1-Pad1)
- RV1 pad 1: Net-(C16-Pad2) -> Net-(C27-Pad2)
- U1 pad 15: Net-(R4-Pad1) -> Net-(R8-Pad1)
- U10 pad 1: Net-(U3-Pad18) -> Net-(RV2-Pad1)
- U10 pad 3: Net-(U4-Pad18) -> Net-(RV1-Pad2)
- U10 pad 4: MIC_IN -> GND
- U10 pad 5: +3V3 -> Net-(C28-Pad1)
- U10 pad 6: /switch4 -> +5V
- U11 pad 1: Net-(U4-Pad3) -> Net-(U11-Pad1)
- U11 pad 3: Net-(U3-Pad3) -> Net-(U11-Pad3)
- U11 pad 4: AUDIO_OUT -> MIC_IN
- U11 pad 6: /switch3 -> /switch4
- U2 pad 32: /GPIO_19 -> SDA
- U2 pad 34: /GPIO_21 -> SCL
- U3 pad 1: AUDIO_ON1 -> GND
- U3 pad 2: unconnected-(U3-Pad2) -> +3V3
- U3 pad 3: Net-(U3-Pad3) -> +5V
- U4 pad 1: AUDIO_ON2 -> GND
- U4 pad 10: GND -> /switch2
- U4 pad 11: unconnected-(U4-Pad11) -> /switch3
- U4 pad 12: Net-(U4-Pad12) -> /switch4
- U4 pad 14: unconnected-(U4-Pad14) -> SCL
- U4 pad 15: unconnected-(U4-Pad15) -> SDA
- U4 pad 16: TX2 -> +3V3
- U4 pad 2: unconnected-(U4-Pad2) -> GND
- U4 pad 3: Net-(U4-Pad3) -> GND
- U4 pad 4: unconnected-(U4-Pad4) -> PD1
- U4 pad 5: PTT2 -> H/L1
- U4 pad 8: +5V -> GND
- U4 pad 9: GND -> /switch1
- U6 pad 1: /esp audio -> Net-(U6-Pad1)
- U6 pad 2: GND -> /-SLEEP
- U6 pad 3: Net-(J6-Pad1) -> Net-(C20-Pad1)
- U6 pad 4: MIC_IN -> GND
- U6 pad 5: +3V3 -> Net-(C23-Pad2)
- U6 pad 6: /switch1 -> Net-(J11-Pad1)
- U7 pad 1: +3V3 -> Net-(C16-Pad1)
- U7 pad 2: +3V3 -> /-SLEEP
- U7 pad 3: GND -> Net-(C22-Pad1)
- U7 pad 4: unconnected-(U7-Pad4) -> GND
- U7 pad 5: unconnected-(U7-Pad5) -> Net-(C13-Pad1)
- U7 pad 6: GND -> Net-(J7-Pad1)
- U7 pad 8: +5V -> GND
- U8 pad 1: Net-(C7-Pad2) -> /esp audio
- U8 pad 2: /-SLEEP -> GND
- U8 pad 3: Net-(C10-Pad1) -> Net-(J11-Pad1)
- U8 pad 4: GND -> MIC_IN
- U8 pad 5: Net-(C30-Pad2) -> +3V3
- U8 pad 6: Net-(J6-Pad1) -> /switch1
Routing:
- added copper zone on B.Cu, net GND
- added copper zone on F.Cu, net GND
Other:
- outline, holes or cut-outs redrawn

Commit message: t
Parts:
- removed C17: 100n, Capacitor_SMD:C_0603_1608Metric_Pad1.08x0.95mm_HandSolder
- removed C19: 470nF, Capacitor_SMD:C_0805_2012Metric
- removed C20: 2.2uF, Capacitor_SMD:C_0805_2012Metric
- removed C23: 1uF, Capacitor_SMD:C_0805_2012Metric
- removed FB1: MH2029-401Y, Resistor_SMD:R_0805_2012Metric_Pad1.20x1.40mm_HandSolder
- removed J10, J12, J13, J8, J9: pin, Connector_PinHeader_2.54mm:PinHeader_1x01_P2.54mm_Vertical
- removed J11: Conn_01x03, Jumper:SolderJumper-3_P2.0mm_Open_TrianglePad1.0x1.5mm_NumberLabels
- removed L2: Ferrit, Resistor_SMD:R_0805_2012Metric_Pad1.20x1.40mm_HandSolder
- removed R1: 1k, Resistor_SMD:R_0603_1608Metric_Pad0.98x0.95mm_HandSolder
- removed R18: 100k, Resistor_SMD:R_0805_2012Metric
- removed R3: 22k, Resistor_SMD:R_0603_1608Metric_Pad0.98x0.95mm_HandSolder
- removed R5: 1Meg, Resistor_SMD:R_0603_1608Metric_Pad0.98x0.95mm_HandSolder
- removed R6: 47k, Resistor_SMD:R_0603_1608Metric_Pad0.98x0.95mm_HandSolder
- removed R8: 10k, Resistor_SMD:R_0603_1608Metric_Pad0.98x0.95mm_HandSolder
- removed RV1, RV2: 10k, Potentiometer_SMD:Potentiometer_Vishay_TS53YL_Vertical
- removed U5: PCA9555PW, Package_SO:TSSOP-24_4.4x7.8mm_P0.65mm
- removed U6: MAX9814, Package_DFN_QFN:DFN-14-1EP_3x3mm_P0.4mm_EP1.78x2.35mm
- added FB2: MH2029-401Y, Resistor_SMD:R_0805_2012Metric_Pad1.20x1.40mm_HandSolder, F.Cu at (123.8, 90.2)
- C15: value 100n -> 10p
- C5: value 100n -> 10u; footprint Capacitor_SMD:C_0603_1608Metric_Pad1.08x0.95mm_HandSolder -> Capacitor_SMD:C_0805_2012Metric
- C6: value 10p -> 100n
- D1, D2: footprint LED_SMD:LED_0603_1608Metric_Pad1.05x0.95mm_HandSolder -> LED_SMD:LED_0805_2012Metric
- J6: value pin -> USB_C_Receptacle; footprint Connector_PinHeader_2.54mm:PinHeader_1x01_P2.54mm_Vertical -> Connector_USB:USB_C_Receptacle_HRO_TYPE-C-31-M-12
- J7: footprint Jumper:SolderJumper-3_P2.0mm_Open_TrianglePad1.0x1.5mm_NumberLabels -> Connector_PinHeader_2.54mm:PinHeader_1x03_P2.54mm_Vertical
- L1: value Ferrit -> L_Small; footprint Resistor_SMD:R_0805_2012Metric_Pad1.20x1.40mm_HandSolder -> Inductor_SMD:L_0805_2012Metric
- R12: value #2.2k -> 5k1; footprint Resistor_SMD:R_0805_2012Metric -> Resistor_SMD:R_0603_1608Metric_Pad0.98x0.95mm_HandSolder
- R14: value 150k -> 5k1; footprint Resistor_SMD:R_0805_2012Metric -> Resistor_SMD:R_0603_1608Metric_Pad0.98x0.95mm_HandSolder
- R16: value 1k -> 1Meg; footprint Resistor_SMD:R_0805_2012Metric -> Resistor_SMD:R_0603_1608Metric_Pad0.98x0.95mm_HandSolder
- U1: value CP2102N-Axx-xQFN24 -> CH340C; footprint Package_DFN_QFN:QFN-24-1EP_4x4mm_P0.5mm_EP2.6x2.6mm -> Package_SO:SOIC-16_3.9x9.9mm_P1.27mm
- moved C38 203.7 mm to (67.2, 62.8), turned to 180 degrees
- moved C34 184.8 mm to (75.0, 90.5)
- moved U11 180.9 mm to (67.2, 60.2)
- moved C3 175.5 mm to (78.5, 59.0), turned to 90 degrees
- moved C1 172.1 mm to (82.2, 59.0), turned to 90 degrees
- moved U12 167.1 mm to (67.1, 67.2)
- moved C33 166.7 mm to (75.0, 92.5), turned to 180 degrees
- moved C37 166.2 mm to (67.1, 64.2), turned to 180 degrees
- moved C2 160.5 mm to (80.5, 59.0), turned to 90 degrees
- moved R20 160.2 mm to (106.0, 93.0), turned to -90 degrees
- moved C30 157.9 mm to (106.0, 89.5), turned to 90 degrees
- moved C25 151.0 mm to (107.0, 97.3), turned to -90 degrees
- moved R9 145.8 mm to (127.0, 76.3), turned to 90 degrees
- moved U8 145.7 mm to (95.8, 85.2), turned to 180 degrees
- moved C24 144.6 mm to (110.8, 97.3), turned to -90 degrees
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Connections:
- net Net-(C13-Pad1) renamed +3.3VA
- C15 pad 1: Net-(U6-Pad1) -> Net-(C15-Pad1)
- C33 pad 1: +5V -> GND
- C33 pad 2: GND -> +5V
- C34 pad 1: GND -> +5V
- C34 pad 2: +5V -> GND
- C4 pad 1: /VDD_CP -> +5V
- C5 pad 1: /~{RST_CP} -> +5V
- D1 pad 2: /VIO -> +3V3
- D2 pad 2: /VIO -> +3V3
- J2 pad 1: GND -> Net-(J2-Pad1)
- J2 pad 2: /MIC_GAIN -> MIC_IN
- J2 pad 3: +3V3 -> /esp audio
- J3 pad 1: GND -> AUDIO_OUT
- J3 pad 2: /MIC_AR -> /AUDIO_IN
- J3 pad 3: +3V3 -> /esp audio
- J7 pad 1: Net-(J7-Pad1) -> Net-(J2-Pad1)
- R10 pad 1: /RXT -> UART0_TX
- R12 pad 1: GND -> Net-(J6-PadA5)
- R12 pad 2: /MIC-AMP_IN -> GND
- R13 pad 1: GND -> Net-(R13-Pad1)
- R14 pad 1: GND -> Net-(J6-PadB5)
- R14 pad 2: Net-(R14-Pad2) -> GND
- R15 pad 2: Net-(R15-Pad2) -> Net-(R13-Pad1)
- R16 pad 1: Net-(R16-Pad1) -> GND
- R16 pad 2: /MIC_GAIN -> Net-(C15-Pad1)
- R17 pad 1: Net-(R15-Pad2) -> Net-(R15-Pad1)
- R9 pad 1: /TXT -> UART0_RX
- U1 pad 1: /~{RI} -> GND
- U1 pad 13: /RXT -> unconnected-(U1-Pad13)
- U1 pad 14: /TXT -> unconnected-(U1-Pad14)
- U1 pad 15: Net-(R8-Pad1) -> unconnected-(U1-Pad15)
- U1 pad 16: unconnected-(U1-Pad16) -> +5V
- U1 pad 2: GND -> UART0_RX
- U1 pad 3: D+ -> UART0_TX
- U1 pad 4: D- -> Net-(C6-Pad1)
- U1 pad 5: /VIO -> D+
- U1 pad 6: /VDD_CP -> D-
- U1 pad 7: /VDD_CP -> unconnected-(U1-Pad7)
- U1 pad 8: /VBUS_DETECT_CP -> unconnected-(U1-Pad8)
- U1 pad 9: /~{RST_CP} -> unconnected-(U1-Pad9)
- U2 pad 5: /GPIO_34 -> /-SLEEP
- U7 pad 13: Net-(R15-Pad1) -> Net-(R13-Pad1)
- U7 pad 14: Net-(R15-Pad2) -> Net-(R15-Pad1)
- U7 pad 6: Net-(J7-Pad1) -> Net-(J2-Pad1)
- U8 pad 3: Net-(J11-Pad1) -> Net-(J2-Pad1)
Other:
- board text added: "jack here"

Commit message: f
Parts:
- added J8: RFShield_OnePiece, RF_Shielding:Wuerth_36103205_20x20mm, F.Cu at (72.0, 79.2)
- added RV1: 10k, Potentiometer_THT:Potentiometer_Bourns_3266W_Vertical, F.Cu at (113.2, 78.7)
- added RV2: 10k, Potentiometer_THT:Potentiometer_Bourns_3266W_Vertical, F.Cu at (118.8, 96.5)
- moved C36 159.3 mm to (104.8, 90.0), turned to -90 degrees
- moved J5 158.7 mm to (69.8, 94.8), turned to -90 degrees
- moved R19 158.0 mm to (75.3, 83.5)
- moved C22 148.9 mm to (66.9, 80.2)
- moved C35 148.9 mm to (103.2, 85.8), turned to -90 degrees
- moved C18 148.8 mm to (75.5, 76.2)
- moved R15 148.8 mm to (74.5, 78.8)
- moved R13 148.8 mm to (76.5, 78.8)
- moved C13 148.8 mm to (67.8, 83.0)
- moved C14 148.8 mm to (66.8, 85.8)
- moved C16 148.8 mm to (69.5, 78.1)
- moved R17 148.8 mm to (72.5, 78.2)
- moved U7 148.8 mm to (71.0, 81.8)
- moved C21 148.8 mm to (75.3, 81.5)
- moved L1 148.7 mm to (65.8, 83.0)
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Connections:
- net Net-(C21-Pad1) renamed /BIAS
- net Net-(C22-Pad1) renamed /CG
- net Net-(FL1-Pad1) renamed /ant1
- net Net-(FL1-Pad3) renamed /ant2
- net Net-(FL2-Pad1) renamed /ant3
- net Net-(FL2-Pad3) renamed /ant4
- net Net-(J2-Pad1) renamed /MIC_out
- net Net-(J6-PadA5) renamed /cc1
- net Net-(J6-PadB5) renamed /cc2
- net Net-(R13-Pad1) renamed /MIC_BIAS
Routing:
- net +5V: track 0.00 -> 163.7 mm, vias 0 -> 9
- net +3V3: track 0.00 -> 133.3 mm, vias 0 -> 2
- net GND: track 0.00 -> 103.2 mm, vias 0 -> 51
- net MIC_IN: track 0.00 -> 69.1 mm, vias 0 -> 5
- net /switch4: track 0.00 -> 63.7 mm, vias 0 -> 3
- net /MIC_out: track 0.00 -> 58.7 mm, vias 0 -> 2
- net H/L1: track 0.00 -> 55.7 mm, vias 0 -> 5
- net TX1: track 0.00 -> 54.2 mm, vias 0 -> 2
- net /BOOT: track 0.00 -> 45.9 mm, vias 0 -> 2
- net UART0_TX: track 0.00 -> 40.3 mm, vias 0 -> 2
- net UART0_RX: track 0.00 -> 40.1 mm, vias 0 -> 2
- net PTT2: track 0.00 -> 33.2 mm, vias 0 -> 2
- net /EN: track 0.00 -> 33.2 mm
- net RX1: track 0.00 -> 31.3 mm, vias 0 -> 2
- net /-SLEEP: track 0.00 -> 30.6 mm, vias 0 -> 2
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
Commit message: Update cross_band_handy_walkie_talkie_V1.kicad_pcb
Parts:
- moved R7 1.67 mm to (124.8, 63.4), turned to -90 degrees
- moved R11 0.11 mm to (129.3, 68.5)
- moved C12 0.10 mm to (119.5, 72.2)
Routing:
- net Net-(U11-Pad3): track 0.00 -> 103.7 mm, vias 0 -> 4
- net +3V3: track 133.3 -> 201.0 mm, vias 2 -> 5
- net PD1: track 0.00 -> 55.5 mm, vias 0 -> 3
- net TX2: track 0.00 -> 52.5 mm, vias 0 -> 2
- net RX2: track 0.00 -> 52.0 mm, vias 0 -> 2
- net Net-(U12-Pad3): track 0.00 -> 37.3 mm, vias 0 -> 4
- net /switch2: track 0.00 -> 30.4 mm, vias 0 -> 3
- net AUDIO_ON2: track 0.00 -> 26.7 mm, vias 0 -> 1
- net Net-(U12-Pad1): track 0.00 -> 21.2 mm, vias 0 -> 1
- net AUDIO_OUT: track 14.3 -> 33.2 mm, vias 0 -> 1
- net H/L2: track 0.00 -> 9.22 mm, vias 0 -> 2
- net PD2: track 0.00 -> 4.91 mm, vias 0 -> 1
- net +5V: track 163.7 -> 167.9 mm, vias 9 -> 8
- net PTT1: track 24.8 -> 21.0 mm
- net /switch1: track 30.0 -> 32.8 mm
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