File: HW/cross_band_handy_walkie_talkie_V1/cross_band_handy_walkie_talkie_V1.kicad_pcb (KiCad board)
At the start: 4 copper layers, 100 x 50 mm, 84 parts, among them J14 Conn_Coaxial, J15 Conn_Coaxial, J2 Conn_01x03, J3 Conn_01x03, J4 Conn_01x03, J5 Conn_01x03, J6 USB_C_Receptacle, J7 Conn_01x03, J8 RFShield_OnePiece, Q1 MMBT3904, Q2 MMBT3904, SW1 MCU_RESET, U1 CH340C, U10 LM386, U11 TS5A63157DBV, U12 TS5A63157DBV, U13 SA818S, U14 SA818S, U2 ESP32-A1S, U3 AMS1117-3.3, U4 PCA9554APW, U7 MAX9814, U8 TS5A63157DBV, U9 TS5A63157DBV

Commit message: R
Parts:
- added J1: Conn_01x06, Connector_PinHeader_2.54mm:PinHeader_1x06_P2.54mm_Vertical, F.Cu at (82.2, 93.4)
- moved J14 89.7 mm to (55.0, 75.0)
- moved J15 89.4 mm to (144.9, 75.0), turned to 180 degrees
- moved FL1 87.4 mm to (56.2, 65.8), turned to -135 degrees
- moved FL2 86.7 mm to (143.8, 82.6), turned to 45 degrees
- moved U13 60.0 mm to (69.8, 75.6)
- moved U14 59.6 mm to (129.8, 72.0)
- moved C34 51.1 mm to (125.8, 88.0), turned to 0 degrees
- moved C32 51.1 mm to (74.1, 59.4), turned to 180 degrees
- moved C31 50.9 mm to (74.2, 57.5), turned to 180 degrees
- moved C33 50.9 mm to (125.8, 89.8), turned to 180 degrees
- moved U11 23.1 mm to (66.7, 85.3), turned to 0 degrees
- moved C38 23.0 mm to (69.7, 86.3), turned to -90 degrees
- moved J4 13.0 mm to (85.3, 88.0)
- moved C5 9.89 mm to (137.3, 78.0), turned to 180 degrees
- moved C4 8.79 mm to (137.3, 79.8), turned to 180 degrees
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Routing:
- net Net-(U11-Pad3): track 103.7 -> 5.44 mm, vias 4 -> 1
- net +5V: track 167.9 -> 72.0 mm, vias 8 -> 6
- net Net-(U11-Pad1): track 2.88 -> 88.9 mm, vias 1 -> 3
- net PD2: track 4.91 -> 54.7 mm, vias 1 -> 2
- net PD1: track 55.5 -> 14.8 mm, vias 3 -> 1
- net +3V3: track 201.0 -> 166.3 mm, vias 5 -> 3
- net H/L1: track 55.7 -> 22.5 mm, vias 5 -> 1
- net /switch1: track 32.8 -> 0.00 mm, vias 2 -> 0
- net /switch2: track 30.4 -> 0.00 mm, vias 3 -> 0
- net Net-(U12-Pad3): track 37.3 -> 10.1 mm, vias 4 -> 1
- net TX1: track 54.2 -> 30.1 mm, vias 2 -> 1
- net AUDIO_ON1: track 15.6 -> 38.8 mm
- net Net-(U12-Pad1): track 21.2 -> 0.00 mm, vias 1 -> 0
- net TX2: track 52.5 -> 33.9 mm, vias 2 -> 1
- net MIC_IN: track 69.9 -> 51.6 mm, vias 5 -> 2
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Other:
- board text added: "SA181-1"
- board text added: "SA181-2"
- board text removed: "jack here"

Commit message: k
Parts:
- added D3: D_Small, Diode_SMD:D_SOD-123, B.Cu at (143.8, 88.8)
- added J9: Conn_01x02, Connector_PinHeader_2.54mm:PinHeader_1x02_P2.54mm_Vertical, F.Cu at (147.4, 86.9)
- added JP1: Jumper_3_Bridged12, Connector_PinHeader_2.54mm:PinHeader_1x03_P2.54mm_Vertical, F.Cu at (94.9, 87.6)
- added R1: 5k1, Resistor_SMD:R_0603_1608Metric_Pad0.98x0.95mm_HandSolder, F.Cu at (90.7, 84.8)
- added R3: 5k1, Resistor_SMD:R_0603_1608Metric_Pad0.98x0.95mm_HandSolder, F.Cu at (94.1, 84.8)
- moved J5 3.47 mm to (73.2, 95.6)
- moved C35 0.16 mm to (103.2, 85.6)
Routing:
- net H/L2: track 0.00 -> 60.5 mm, vias 0 -> 3
- net +5V: track 72.0 -> 123.1 mm, vias 6 -> 10
- net Net-(U12-Pad1): track 0.00 -> 47.4 mm, vias 0 -> 5
- net /switch2: track 0.00 -> 35.1 mm, vias 0 -> 2
- net /MIC-AMP_IN: track 1.69 -> 36.8 mm, vias 0 -> 2
- net /switch1: track 0.00 -> 30.4 mm, vias 0 -> 3
- net PTT2: track 18.1 -> 32.4 mm, vias 1 -> 3
- net PTT1: track 34.7 -> 48.7 mm, vias 3 -> 5
- net +3V3: track 166.3 -> 177.1 mm
- net VBUS: track 14.1 -> 24.3 mm
- net /MIC_EST_PTT: track 0.00 -> 6.85 mm
- net Net-(J9-Pad2): track 0.00 -> 4.80 mm
- net Net-(JP1-Pad1): track 0.00 -> 2.85 mm
- net Net-(JP1-Pad3): track 0.00 -> 2.81 mm
- net Net-(C24-Pad1): track 0.00 -> 2.61 mm
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