File: HW/cross_band_handy_walkie_talkie_V1/cross_band_handy_walkie_talkie_V1.kicad_pcb (KiCad board)
At the start: 4 copper layers, 100 x 50 mm, 90 parts, among them J1 Conn_01x06, J14 Conn_Coaxial, J15 Conn_Coaxial, J2 Conn_01x03, J3 Conn_01x03, J4 Conn_01x03, J5 Conn_01x03, J6 USB_C_Receptacle, J7 Conn_01x03, J8 RFShield_OnePiece, J9 Conn_01x02, Q1 MMBT3904, Q2 MMBT3904, SW1 MCU_RESET, U1 CH340C, U10 LM386, U11 TS5A63157DBV, U12 TS5A63157DBV, U13 SA818S, U14 SA818S, U2 ESP32-A1S, U3 AMS1117-3.3, U4 PCA9554APW, U7 MAX9814, U8 TS5A63157DBV, U9 TS5A63157DBV

Commit message: n
Parts:
- added C17: 1u, Capacitor_SMD:C_0603_1608Metric_Pad1.08x0.95mm_HandSolder, F.Cu at (100.4, 83.4)
- added C19: 1u, Capacitor_SMD:C_0603_1608Metric_Pad1.08x0.95mm_HandSolder, F.Cu at (116.4, 81.2)
- added D4: LED_Small, LED_SMD:LED_0805_2012Metric, F.Cu at (117.2, 60.5)
- added FID1: Fiducial, Fiducial:Fiducial_0.5mm_Mask1mm, F.Cu at (146.2, 64.8)
- added FID2: Fiducial, Symbol:KiCad-Logo2_5mm_SilkScreen, B.Cu at (99.6, 72.6)
- added FID3: Fiducial, Symbol:WEEE-Logo_4.2x6mm_SilkScreen, B.Cu at (90.2, 72.6)
- added J10: Conn_01x02, Connector_PinHeader_2.54mm:PinHeader_1x02_P2.54mm_Vertical, F.Cu at (107.8, 97.9)
- added R5: 300, Resistor_SMD:R_0603_1608Metric_Pad0.98x0.95mm_HandSolder, F.Cu at (120.8, 60.6)
- J14, J15: value Conn_Coaxial -> SMA
- moved RV2 3.81 mm to (120.8, 93.3), turned to 90 degrees
- moved C24 2.43 mm to (117.3, 95.8), turned to 0 degrees
- moved C29 1.91 mm to (119.2, 89.6)
- moved J2 1.75 mm to (99.0, 94.0)
- moved J7 1.72 mm to (99.0, 97.8)
- moved C28 1.13 mm to (107.8, 92.6), turned to 180 degrees
- moved C25 1.10 mm to (112.6, 97.0)
- moved C26 1.10 mm to (114.6, 97.0)
- moved RV1 0.72 mm to (113.2, 78.0)
- moved C27 0.60 mm to (114.6, 81.2), turned to 90 degrees
- moved J3 0.30 mm to (117.0, 84.8)
- moved R20 0.20 mm to (110.4, 93.4)
Connections:
- C28 pad 2: AUDIO_OUT -> /AMPLIFIED_AUDIO_OUT
- J1 pad 3: /EXT_SPEAKER+ -> /AMPLIFIED_AUDIO_OUT
- U2 pad 21: unconnected-(U2-Pad21) -> Net-(C19-Pad1)
- U2 pad 22: unconnected-(U2-Pad22) -> Net-(C19-Pad1)
- U2 pad 27: unconnected-(U2-Pad27) -> Net-(C17-Pad1)
- U2 pad 28: unconnected-(U2-Pad28) -> Net-(C17-Pad1)
Routing:
- net /AMPLIFIED_AUDIO_OUT: track 0.00 -> 25.6 mm
- net /GPIO_23: track 0.00 -> 19.4 mm, vias 0 -> 2
- net Net-(C17-Pad1): track 0.00 -> 19.4 mm
- net Net-(C19-Pad1): track 0.00 -> 11.5 mm
- net GND: track 115.1 -> 123.0 mm, vias 57 -> 63
- net MIC_IN: track 51.6 -> 56.5 mm
- net Net-(C29-Pad2): track 3.54 -> 7.56 mm
- net Net-(RV2-Pad1): track 9.16 -> 6.78 mm
- net Net-(C29-Pad1): track 3.05 -> 5.03 mm
- net PD2: track 55.0 -> 56.9 mm
- net Net-(D4-Pad1): track 0.00 -> 1.80 mm
- net +5V: track 123.1 -> 124.6 mm
- net /esp audio: track 17.6 -> 19.0 mm
- net AUDIO_OUT: track 32.7 -> 33.9 mm
- net /AUDIO_IN: track 11.7 -> 11.0 mm
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Other:
- rule solder_mask_min_width: 0.25 -> 0.2

Commit message: g
Parts:
- added C20: 1u, Capacitor_SMD:C_0603_1608Metric_Pad1.08x0.95mm_HandSolder, F.Cu at (96.4, 97.3)
- added kibuzzard-639A1F7F: G***, kibuzzard-639A1F7F, F.Cu at (84.6, 97.6)
- added kibuzzard-639A1F7F: G***, kibuzzard-639A1F7F, F.Cu at (77.4, 95.6)
- added kibuzzard-639A1F7F: G***, kibuzzard-639A1F7F, F.Cu at (92.4, 97.6)
- added kibuzzard-639A1F94: G***, kibuzzard-639A1F94, F.Cu at (82.2, 97.6)
- added kibuzzard-639A1FC8: G***, kibuzzard-639A1FC8, F.Cu at (87.4, 97.4)
- added kibuzzard-639A1FDB: G***, kibuzzard-639A1FDB, F.Cu at (89.8, 97.4)
- added kibuzzard-639A1FE7: G***, kibuzzard-639A1FE7, F.Cu at (94.8, 97.6)
- added kibuzzard-639A20B2: G***, kibuzzard-639A20B2, F.Cu at (64.0, 95.6)
- added kibuzzard-639A20B2: G***, kibuzzard-639A20B2, F.Cu at (85.2, 78.8)
- added kibuzzard-639A20C5: G***, kibuzzard-639A20C5, F.Cu at (70.4, 98.6)
- added kibuzzard-639A2114: G***, kibuzzard-639A2114, F.Cu at (85.2, 90.6)
- moved FID2 21.7 mm to (110.8, 54.0)
- moved FID3 19.3 mm to (94.4, 53.8)
- moved J5 0.20 mm to (73.2, 95.4)
Connections:
- J2 pad 1: /MIC_out -> Net-(J2-Pad1)
- U8 pad 3: /MIC_out -> Net-(J2-Pad1)
Routing:
- net /MIC_out: track 62.5 -> 46.6 mm, vias 2 -> 1
- net Net-(J2-Pad1): track 0.00 -> 3.71 mm
- net +5V: track 124.6 -> 127.7 mm
- net PD2: track 56.9 -> 55.0 mm
- net GND: track 123.0 -> 124.7 mm
- added copper zone on F.Cu, net +3V3
