File: HW/cross_band_handy_walkie_talkie_V1/cross_band_handy_walkie_talkie_V1.kicad_pcb (KiCad board)
At the start: 4 copper layers, 100 x 50 mm, 134 parts, among them J1 Conn_01x06, J14 SMA, J15 SMA, J2 Conn_01x03, J3 Conn_01x03, J4 Conn_01x03, J5 Conn_01x03, J6 USB_C_Receptacle, J7 Conn_01x04, J8 RFShield_OnePiece, J9 Conn_01x02, Q1 MMBT3904, Q2 MMBT3904, SW1 MCU_RESET, U1 CH340C, U10 LM386, U11 TS5A63157DBV, U12 TS5A63157DBV, U13 SA818S, U14 SA818S, U2 ESP32-A1S, U3 AMS1117-3.3, U4 PCA9554APW, U5 SRV05-4, U7 MAX9814, U8 TS5A63157DBV, U9 TS5A63157DBV

Commit message: j
Parts:
- removed C35, C36: 100n, Capacitor_SMD:C_0603_1608Metric_Pad1.08x0.95mm_HandSolder
- removed JP2, JP3: ., Jumper:SolderJumper-3_P2.0mm_Open_TrianglePad1.0x1.5mm_NumberLabels
- removed U11, U12: TS5A63157DBV, Package_TO_SOT_SMD:SOT-23-6
- added C23: 1u, Capacitor_SMD:C_0603_1608Metric_Pad1.08x0.95mm_HandSolder, F.Cu at (183.2, 64.2)
- added R18: 10k, Resistor_SMD:R_0603_1608Metric_Pad0.98x0.95mm_HandSolder, F.Cu at (187.5, 61.7)
- added R8: 10k, Resistor_SMD:R_0603_1608Metric_Pad0.98x0.95mm_HandSolder, F.Cu at (183.2, 61.7)
- C7: value DNP -> 1u
Connections:
- C17 pad 2: /esp_audio_OUTPUT -> HPOUT_R
- C19 pad 2: AUDIO_OUT -> LINE_L
- C7 pad 1: /EN -> HPOUT_L
- C7 pad 2: GND -> Net-(U2-Pad27)
- D4 pad 2: /GPIO_23 -> RX2
- TP7 pad 1: /GPIO_22 -> TX1
- U13 pad 18: Net-(U11-Pad3) -> unconnected-(U13-Pad18)
- U13 pad 3: Net-(U12-Pad1) -> unconnected-(U13-Pad3)
- U13 pad 6: Net-(U13-Pad6) -> PD2
- U14 pad 18: Net-(U11-Pad1) -> unconnected-(U14-Pad18)
- U14 pad 3: Net-(U12-Pad3) -> unconnected-(U14-Pad3)
- U14 pad 6: Net-(U14-Pad6) -> PD1
- U2 pad 10: AUDIO_ON1 -> /GPIO_15
- U2 pad 12: RX2 -> /GPIO_04
- U2 pad 21: Net-(C19-Pad1) -> Net-(U2-Pad21)
- U2 pad 27: unconnected-(U2-Pad27) -> Net-(U2-Pad27)
- U2 pad 29: TX1 -> /GPIO_05
- U2 pad 30: AUDIO_ON2 -> /GPIO_18
- U2 pad 31: /GPIO_23 -> RX2
- U2 pad 32: SDA -> /GPIO_19
- U2 pad 33: /GPIO_22 -> TX1
- U2 pad 34: SCL -> RX1
- U2 pad 5: /GPIO_34 -> TX2
- U2 pad 7: PTT2 -> /GPIO_14
- U2 pad 9: PTT1 -> /GPIO_13
- U4 pad 10: /switch2 -> PD2
- U4 pad 11: /switch3 -> H/L2
- U4 pad 12: /switch4 -> PD2
- U4 pad 4: PD1 -> PTT1
- U4 pad 5: H/L1 -> PD1
- U4 pad 6: PD2 -> H/L1
- U4 pad 7: H/L2 -> PD1
- U4 pad 9: /switch1 -> PTT2
Routing:
- net +3V3: track 177.9 -> 0.00 mm, vias 3 -> 0
- net GND: track 176.9 -> 0.00 mm, vias 126 -> 0
- net +5V: track 135.3 -> 0.00 mm, vias 11 -> 0
- net Net-(U11-Pad1): track 88.7 -> 0.00 mm, vias 3 -> 0
- net H/L2: track 60.5 -> 0.00 mm, vias 3 -> 0
- net /switch4: track 58.0 -> 0.00 mm, vias 2 -> 0
- net RF_AUDIO_INPUT: track 52.5 -> 0.00 mm, vias 2 -> 0
- net /GPIO_12: track 49.0 -> 0.00 mm, vias 1 -> 0
- net PD2: track 48.7 -> 0.00 mm, vias 2 -> 0
- net PTT1: track 48.7 -> 0.00 mm, vias 5 -> 0
- net Net-(U12-Pad1): track 48.1 -> 0.00 mm, vias 5 -> 0
- net /BOOT: track 45.9 -> 0.00 mm, vias 3 -> 0
- net /MIC_AMPLIFIER_OUTPUT: track 43.7 -> 0.00 mm, vias 1 -> 0
- net AUDIO_ON2: track 41.2 -> 0.00 mm, vias 1 -> 0
- net AUDIO_ON1: track 39.2 -> 0.00 mm, vias 1 -> 0
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