File: HW/cross_band_handy_walkie_talkie_ES8388/cross_band_handy_walkie_talkie_ES8388.kicad_sch (KiCad schematic)
At the start: 60 parts

Commit message: t
Parts:
- gave numbers to parts that had none: 60

Commit message: b
Parts:
- removed C1: DNP, Capacitor_SMD:C_0603_1608Metric_Pad1.08x0.95mm_HandSolder, symbol Device:C_Small
- removed C11, C12, C9: 100n, Capacitor_SMD:C_0603_1608Metric_Pad1.08x0.95mm_HandSolder, symbol Device:C_Small
- added BT?: Battery_Cell, Connector_PinHeader_2.54mm:PinHeader_1x02_P2.54mm_Vertical, symbol Device:Battery_Cell
- added C? (x7): 10u, Capacitor_SMD:C_0805_2012Metric, symbol Device:C_Small
- added C? (x3): 1u, Capacitor_SMD:C_0603_1608Metric_Pad1.08x0.95mm_HandSolder, symbol Device:C_Small
- added C?: 100n, Capacitor_SMD:C_0603_1608Metric_Pad1.08x0.95mm_HandSolder, symbol Device:C_Small
- added D? (x4): LED_Small, LED_SMD:LED_0805_2012Metric, symbol Device:LED_Small
- added L?: L_Small, symbol Device:L_Small
- added R? (x3): 5k1, Resistor_SMD:R_0603_1608Metric_Pad0.98x0.95mm_HandSolder, symbol Device:R_Small
- added R? (x3): 1k, Resistor_SMD:R_0805_2012Metric, symbol Device:R
- added U?: TP5000, Package_DFN_QFN:QFN-16-1EP_4x4mm_P0.65mm_EP2.5x2.5mm_ThermalVias, symbol My_custom_lib:TP5000
- added U?: AMS1117-3.3, Package_TO_SOT_SMD:SOT-223-3_TabPin2, symbol Regulator_Linear:AMS1117-3.3
Connections:
- net +3V3: now also C?.1, C?.2, D?.2 (A), R?.1, R?.1, U?.2 (VO)
- net +5V: now also C?.1, C?.1, C?.1, C?.2, D?.2 (A), R?.1, U?.1 (VIN), U?.16 (VIN), U?.2 (VIN), U?.3 (VI)
- net GND: now also BT?.2 (-), C?.1, C?.1, C?.2, C?.2, C?.2, C?.2, C?.2, C?.2, C?.2, C?.2, C?.2, R?.2, R?.2, U?.1 (GND), U?.12 (RTRICK), U?.6 (GND), U?.7 (GND)
- net Tranceiver_Audio_IN_2: now reaches U4.18 (MIC_IN)
- net Tranceiver_Audio_OUT_2: now reaches U4.3 (AF(Audio_OUT))
- net Tranceiver_Audio_IN_1: now reaches U3.18 (MIC_IN)
- net Tranceiver_Audio_OUT_1: now reaches U3.3 (AF(Audio_OUT))
- net GPIO_5 renamed G0
- net GPIO_6 renamed G1
- new net: C?.1, C?.1, L?.2, R?.2, U?.8 (VS)
- new net: D?.1 (K), U?.14 (~{CHRG})
- new net: D?.2 (A), D?.2 (A), R?.2
- new net: BT?.1 (+), C?.1, C?.1, R?.1, U?.9 (BAT)
- new net: C?.1, U?.10 (VREG)
- new net: D?.1 (K), U?.15 (~{STDBY})
- new net: L?.1, U?.3 (LX), U?.4 (LX), U?.5 (LX)
- new net: D?.1 (K), R?.1 (x2)
- new net SCL: R?.2
- new net SDA: R?.2
Other:
- note added: "3V3 LDO"
- moved on the sheet: C2, C3, C4, C5, C6, H1, H2, H3, H4, R1, R20, R21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

Commit message: f
Parts:
- removed BT?: Battery_Cell, Connector_PinHeader_2.54mm:PinHeader_1x02_P2.54mm_Vertical, symbol Device:Battery_Cell
- removed C13, C? (x7): 10u, Capacitor_SMD:C_0805_2012Metric, symbol Device:C_Small
- removed C? (x2): 1u, Capacitor_SMD:C_0603_1608Metric_Pad1.08x0.95mm_HandSolder, symbol Device:C_Small
- removed C?: 100n, Capacitor_SMD:C_0603_1608Metric_Pad1.08x0.95mm_HandSolder, symbol Device:C_Small
- removed D? (x2): LED_Small, LED_SMD:LED_0805_2012Metric, symbol Device:LED_Small
- removed FL1, FL2: LFCN-160, Filter:Filter_Mini-Circuits_FV1206, symbol RF_Filter:LFCN-160
- removed J3, J4: SMA, Connector_Coaxial:SMA_Amphenol_901-144_Vertical, symbol Connector:Conn_Coaxial
- removed L?: L_Small, symbol Device:L_Small
- removed R13, R14, R15, R26, R27: 10k, Resistor_SMD:R_0603_1608Metric_Pad0.98x0.95mm_HandSolder, symbol Device:R_Small
- removed R?: 1k, Resistor_SMD:R_0805_2012Metric, symbol Device:R
- removed R?: 5k1, Resistor_SMD:R_0603_1608Metric_Pad0.98x0.95mm_HandSolder, symbol Device:R_Small
- removed U3, U4: SA818S, Z_mycustom_footprint_lib:SA818S, symbol My_custom_lib:SA818S
- removed U?: TP5000, Package_DFN_QFN:QFN-16-1EP_4x4mm_P0.65mm_EP2.5x2.5mm_ThermalVias, symbol My_custom_lib:TP5000
- removed U?: AMS1117-3.3, Package_TO_SOT_SMD:SOT-223-3_TabPin2, symbol Regulator_Linear:AMS1117-3.3
- added BT1: Battery_Cell, Connector_PinHeader_2.54mm:PinHeader_1x02_P2.54mm_Vertical, symbol Device:Battery_Cell
- added C11, C12, C46, C47, C50, C51, C52, C9: 10u, Capacitor_SMD:C_0805_2012Metric, symbol Device:C_Small
- added C53: 100n, Capacitor_SMD:C_0603_1608Metric_Pad1.08x0.95mm_HandSolder, symbol Device:C_Small
- added D3: D_Schottky, Diode_SMD:D_SMA_Handsoldering, symbol Device:D_Schottky
- added D4, D5: LED_Small, LED_SMD:LED_0805_2012Metric, symbol Device:LED_Small
- added J3: Conn_01x02, Connector_PinHeader_2.54mm:PinHeader_1x02_P2.54mm_Vertical, symbol Connector_Generic:Conn_01x02
- added L4: L_Small, symbol Device:L_Small
- added L5: L_Small, Inductor_SMD:L_0603_1608Metric, symbol Device:L_Small
- added Q1: nMOS, Package_TO_SOT_SMD:SOT-23, symbol Device:Q_NMOS_GSD
- added R15: 1k, Resistor_SMD:R_0805_2012Metric, symbol Device:R
- added R19, R20, R36, R40: 10k, Resistor_SMD:R_0402_1005Metric, symbol Device:R_Small
- added R30: 10k, Resistor_SMD:R_0603_1608Metric_Pad0.98x0.95mm_HandSolder, symbol Device:R_Small
- added U3: AMS1117-3.3, Package_TO_SOT_SMD:SOT-223-3_TabPin2, symbol Regulator_Linear:AMS1117-3.3
- added U4: TP5000, Package_DFN_QFN:QFN-16-1EP_4x4mm_P0.65mm_EP2.5x2.5mm_ThermalVias, symbol My_custom_lib:TP5000
- D1, D2: renamed from D?; value LED_Small -> green
- R14: renamed from R12; footprint Resistor_SMD:R_0603_1608Metric_Pad0.98x0.95mm_HandSolder -> Resistor_SMD:R_0402_1005Metric; LCSC C25804 -> C25744
- R16: value 10k -> 5k1; LCSC C25804 -> C23186
- R17, R18: footprint Resistor_SMD:R_0603_1608Metric_Pad0.98x0.95mm_HandSolder -> Resistor_SMD:R_0402_1005Metric; LCSC C25804 -> C25744
- gave numbers to parts that had none: 5
- renumbered C2 to C1, C3 to C2, C4 to C3, C5 to C4, C6 to C5, C7 to C6, C8 to C7, R8 to R10, R9 to R11, R10 to R12, R11 to R13, R19 to R21, R20 to R24, R21 to R25, R22 to R26, R23 to R27, R24 to R28, R25 to R29, R4 to R6, R5 to R7, R6 to R8, R7 to R9
Connections:
- net +3V3: now also C11.1, C50.1, L5.2, R19.2, R20.2, R36.2, R40.2, U3.2 (VO); no longer R16.2
- net +5V: now also C47.1, C9.1, R15.1, U3.3 (VI), U4.1 (VIN), U4.16 (VIN), U4.2 (VIN); no longer C10.1
- net CARD_DETECT: now also R40.1; no longer R18.1
- net CLK: now also R36.1; no longer R17.1
- net CMD: now also R20.1; no longer R16.1
- net DATA_1: now also R17.1
- net DATA_2: now also R18.1
- net DATA_3: now also R19.1
- net GND: now also BT1.2 (-), C11.2, C12.2, C46.2, C47.2, C50.2, C51.2, C52.2, C53.2, C9.2, D3.2 (A), J3.1 (Pin_1), Q1.2 (S), R30.1, U3.1 (GND), U4.12 (RTRICK), U4.6 (GND), U4.7 (GND)
- new net: D5.1 (K), U4.15 (~{STDBY})
- new net: D4.2 (A), D5.2 (A), R15.2
- new net: BT1.1 (+), C10.1, C51.1, C52.1, L5.1, R16.1, U4.9 (BAT)
- new net: C12.1, C46.1, L4.2, R16.2, U4.8 (VS)
- new net: C53.1, U4.10 (VREG)
- new net: Q1.1 (G), R30.2
- new net: J3.2 (Pin_2), U4.11 (TS)
- new net: D4.1 (K), U4.14 (~{CHRG})
- new net: D3.1 (K), L4.1, U4.3 (LX), U4.4 (LX), U4.5 (LX)
- new net CS: Q1.3 (D), U4.13 (CS)
Other:
- note added: "RShunt (Ω) IBAT (mA) 1 100 0.2 500 0.1 1000 0.067 1500 0.05 2000"
- note added: "leds on the PTT lines leds on the PD lines led on SD CS"
- note removed: "750mA max current"
- note removed: "RF MODULES"
- note removed: "SA818-1"
- note removed: "SA818-2"

Commit message: f
Parts:
- added D8: D_Schottky, Diode_SMD:D_SMA_Handsoldering, symbol Device:D_Schottky
- added J9: Conn_01x03, Connector_PinHeader_2.54mm:PinHeader_1x03_P2.54mm_Vertical, symbol Connector_Generic:Conn_01x03
- D4, D5: value LED_Small -> green
- R16: value 5k1 -> 0R2
Connections:
- net +3V3: now also D8.2 (A)
- net +5V: now also D8.1 (K), J9.3 (Pin_3)
- net at Q1.1 (G), R30.2: now also J9.2 (Pin_2)
- no-connect marks 15 -> 16
Other:
- note added: "500mA @3.6V 1.8W => 400mA @5V 2W"
- note added: "AUDIO"
- note added: "SD card"
- note removed: "leds on the PTT lines leds on the PD lines led on SD CS"
- moved on the sheet: BT1, C10, C11, C12, C46, C47, C50, C51, C52, C53, C7, C8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

Commit message: l
Parts:
- removed D8: D_Schottky, Diode_SMD:D_SMA_Handsoldering, symbol Device:D_Schottky
- removed L5: L_Small, Inductor_SMD:L_0603_1608Metric, symbol Device:L_Small
- added L1: 4u7, Z_mycustom_footprint_lib:Inductor_2.5x2x1.2mm, symbol Device:L_Small
- added R43: 0R1, Resistor_SMD:R_1206_3216Metric, symbol Device:R_Small
- D4: value green -> red; footprint LED_SMD:LED_0805_2012Metric -> LED_SMD:LED_0603_1608Metric; LCSC C2297 -> C2286
- L4: value L_Small -> 4u7; footprint (none) -> Z_mycustom_footprint_lib:Inductor_2.5x2x1.2mm; LCSC (none) -> C3002553
- R16: value 0R2 -> 0R1; footprint Resistor_SMD:R_0603_1608Metric_Pad0.98x0.95mm_HandSolder -> Resistor_SMD:R_1206_3216Metric; LCSC C23186 -> C25334
Connections:
- net +3V3: now also L1.2
- net at BT1.1 (+), C10.1, C51.1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: now also L1.1, R43.1; no longer R16.1
- new net: R16.1, R43.2
Other:
- moved on the sheet: BT1, R16

Commit message: n
Parts:
- removed C46, C47, C50, C51, C52: 10u, Capacitor_SMD:C_0805_2012Metric, symbol Device:C_Small
- added C13, C17: 1u, Capacitor_SMD:C_0402_1005Metric, symbol Device:C_Small
- added C14, C15, C16, C57, C58, C59: 10u, Capacitor_SMD:C_0603_1608Metric, symbol Device:C_Small
- C10, C11, C12, C3, C4, C7, C9: footprint Capacitor_SMD:C_0805_2012Metric -> Capacitor_SMD:C_0603_1608Metric; LCSC C15850 -> C96446
- C5, C53: value 100n -> 1u; footprint Capacitor_SMD:C_0603_1608Metric_Pad1.08x0.95mm_HandSolder -> Capacitor_SMD:C_0402_1005Metric; LCSC C14663 -> C52923
- R2, R22, R23, R3: footprint Resistor_SMD:R_0603_1608Metric_Pad0.98x0.95mm_HandSolder -> Resistor_SMD:R_0402_1005Metric; LCSC C23186 -> C25905
Connections:
- net +3V3: now also C5.2, C14.1, C15.1, C57.1, C58.1, C59.1; no longer C11.1, C5.1, C7.1
- net +5V: now also C7.1
- net D+: now also U1.1 (IO1); no longer U1.4 (IO3)
- net GND: now also C5.1, C53.1, C13.1, C14.2, C15.2, C16.2, C17.1, C57.2, C58.2, C59.2; no longer C5.2, C53.2
- net GPIO_12: now also R26.1; no longer R29.1
- net GPIO_14: now also R29.1; no longer R26.1
- net GPIO_45: now also J9.2 (Pin_2), Q1.1 (G), R30.2
- net at BT1.1 (+), C10.1, L1.1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: now also C11.1, C16.1, C17.2
- net at C12.1, L4.2, R16.2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: now also C13.2
- net at U4.10 (VREG): now also C53.2; no longer C53.1
- no-connect marks 16 -> 15

Commit message: b
Parts:
- removed J3: Conn_01x02, Connector_PinHeader_2.54mm:PinHeader_1x02_P2.54mm_Vertical, symbol Connector_Generic:Conn_01x02
- removed J9: Conn_01x03, Connector_PinHeader_2.54mm:PinHeader_1x03_P2.54mm_Vertical, symbol Connector_Generic:Conn_01x03
- added C61, C62: 10u, Capacitor_SMD:C_0603_1608Metric, symbol Device:C_Small
- added Q2, Q3, Q4: AO3401A, Package_TO_SOT_SMD:SOT-23, symbol Transistor_FET:AO3401A
- added R46: 10k, Resistor_SMD:R_0603_1608Metric_Pad0.98x0.95mm_HandSolder, symbol Device:R_Small
- added TP1, TP2: TestPoint, TestPoint:TestPoint_Pad_1.0x1.0mm, symbol Connector:TestPoint
Connections:
- net +3V3: now also C61.1, C62.1, Q3.2 (S), Q4.2 (S); no longer C57.1, C58.1, C59.1, L1.2, U3.2 (VO)
- net +5V: now also Q2.1 (G), Q3.1 (G), R46.2
- net GND: now also C61.2, C62.2, Q4.1 (G), R46.1
- net at U4.11 (TS): now also TP2.1
- new net: C58.1, C59.1, L1.2, Q2.2 (S)
- new net: Q2.3 (D), Q3.3 (D)
- new net: C57.1, Q4.3 (D), U3.2 (VO)
- no-connect marks 15 -> 14
Other:
- note removed: "3V3 LDO"
- moved on the sheet: BT1, C10, C11, C12, C13, C16, C17, C53, C57, C58, C59, C7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

Commit message: g
Parts:
- R46: footprint Resistor_SMD:R_0603_1608Metric_Pad0.98x0.95mm_HandSolder -> Resistor_SMD:R_0402_1005Metric; LCSC C25804 -> C25744
Changed lines of the file:
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@@
+    (pin "2")
+  )
+  (symbol (lib_id "Device:R_Small") (at 314.96 205.74 0) (mirror x) (unit 1)
+    (in_bom yes) (on_board yes)
+    (property "Reference" "R46" (id 0) (at 313.69 204.47 0)
+      (effects (font (size 1.27 1.27)) (justify right))
+    )
+    (property "Value" "10k" (id 1) (at 313.69 207.01 0)
+      (effects (font (size 1.27 1.27)) (justify right))
+    )
+    (property "Footprint" "Resistor_SMD:R_0402_1005Metric" (id 2) (at 314.96 205.74 0)
+      (effects (font (size 1.27 1.27)) hide)
+    )
+    (property "Datasheet" "~" (id 3) (at 314.96 205.74 0)
+      (effects (font (size 1.27 1.27)) hide)
+    )
+    (property "LCSC" "C25744" (id 4) (at 314.96 205.74 90)
+      (effects (font (size 1.27 1.27)) hide)
+    )
+    (pin "1")
     (pin "2")
   )
@@
     )
     (property "LCSC" "C2297" (id 4) (at 289.56 40.64 90)
-      (effects (font (size 1.27 1.27)) hide)
-    )
-    (pin "1")
-    (pin "2")
-  )
-  (symbol (lib_id "Device:R_Small") (at 314.96 205.74 0) (mirror x) (unit 1)
-    (in_bom yes) (on_board yes) (fields_autoplaced)
-    (property "Reference" "R46" (id 0) (at 312.42 204.4699 0)
-      (effects (font (size 1.27 1.27)) (justify right))
-    )
-    (property "Value" "10k" (id 1) (at 312.42 207.0099 0)
-      (effects (font (size 1.27 1.27)) (justify right))
-    )
-    (property "Footprint" "Resistor_SMD:R_0603_1608Metric_Pad0.98x0.95mm_HandSolder" (id 2) (at 314.96 205.74 0)
-      (effects (font (size 1.27 1.27)) hide)
-    )
-    (property "Datasheet" "~" (id 3) (at 314.96 205.74 0)
-      (effects (font (size 1.27 1.27)) hide)
-    )
-    (property "LCSC" "C25804" (id 4) (at 314.96 205.74 90)
       (effects (font (size 1.27 1.27)) hide)
     )
@@
       (reference "R45") (unit 1) (value "10k") (footprint "Resistor_SMD:R_0603_1608Metric_Pad0.98x0.95mm_HandSolder")
     )
-    (path "/8982463c-c3fa-4800-ae20-7eea17cdf06e"
-      (reference "R46") (unit 1) (value "10k") (footprint "Resistor_SMD:R_0603_1608Metric_Pad0.98x0.95mm_HandSolder")
+    (path "/7aa18316-618b-46b7-b925-fdbc1b5fae1c"
+      (reference "R46") (unit 1) (value "10k") (footprint "Resistor_SMD:R_0402_1005Metric")
     )
     (path "/b92fe6ff-d6b8-4da3-890c-5c9328d5748e/6b541878-701e-4e8c-ad50-4ac4a2855c34"
