File: HW/cross_band_handy_walkie_talkie_ES8388/cross_band_handy_walkie_talkie_ES8388.kicad_sch (KiCad schematic)
At the start: 87 parts, among them J1 USB_C_Receptacle, J2 Micro_SD_Card_Det, Q1 nMOS, Q2 AO3401A, Q3 AO3401A, Q4 AO3401A, SW1 MCU_RESET, SW2 MCU_RESET, U1 SRV05-4, U2 ESP32-S3-WROOM-1, U3 AMS1117-3.3, U4 TP5000

Commit message: f
Parts:
- added R47, R48, R49, R50: 10, Resistor_SMD:R_0402_1005Metric, symbol Device:R_Small
- FB1: footprint (none) -> Resistor_SMD:R_0805_2012Metric
Connections:
- net AMP_L: now also R48.1
- net AMP_R: now also R47.1
- net G0: now also R50.1; no longer U2.5 (GPIO5/TOUCH5/ADC1_CH4)
- net G1: now also R49.1; no longer U2.6 (GPIO6/TOUCH6/ADC1_CH5)
- new net GPIO_5: R50.2, U2.5 (GPIO5/TOUCH5/ADC1_CH4)
- new net GPIO_6: R49.2, U2.6 (GPIO6/TOUCH6/ADC1_CH5)
Changed lines of the file:
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@@
     (stroke (width 0) (type default) (color 0 0 0 0))
   )
+  (wire (pts (xy -21.59 229.87) (xy -26.67 229.87))
+    (stroke (width 0) (type default) (color 0 0 0 0))
+  )
   (wire (pts (xy 83.82 257.81) (xy 83.82 261.62))
     (stroke (width 0) (type default) (color 0 0 0 0))
@@
     (stroke (width 0) (type default) (color 0 0 0 0))
   )
+  (wire (pts (xy -21.59 232.41) (xy -26.67 232.41))
+    (stroke (width 0) (type default) (color 0 0 0 0))
+  )
   (wire (pts (xy 83.82 248.92) (xy 83.82 250.19))
     (stroke (width 0) (type default) (color 0 0 0 0))
@@
     )
   )
-  (global_label "GPIO_5" (shape bidirectional) (at -31.75 232.41 0) (fields_autoplaced)
+  (global_label "GPIO_5" (shape bidirectional) (at -21.59 232.41 0) (fields_autoplaced)
     (effects (font (size 1.27 1.27)) (justify left))
-    (property "Intersheet References" "${INTERSHEET_REFS}" (id 0) (at -22.6845 232.4894 0)
+    (property "Intersheet References" "${INTERSHEET_REFS}" (id 0) (at -12.5245 232.4894 0)
       (effects (font (size 1.27 1.27)) (justify left) hide)
     )
@@
     )
   )
-  (global_label "GPIO_6" (shape bidirectional) (at -31.75 229.87 0) (fields_autoplaced)
+  (global_label "GPIO_6" (shape bidirectional) (at -21.59 229.87 0) (fields_autoplaced)
     (effects (font (size 1.27 1.27)) (justify left))
-    (property "Intersheet References" "${INTERSHEET_REFS}" (id 0) (at -22.6845 229.9494 0)
+    (property "Intersheet References" "${INTERSHEET_REFS}" (id 0) (at -12.5245 229.9494 0)
       (effects (font (size 1.27 1.27)) (justify left) hide)
     )
@@
     (pin "1")
   )
+  (symbol (lib_id "Device:R_Small") (at -29.21 229.87 90) (unit 1)
+    (in_bom yes) (on_board yes)
+    (property "Reference" "R49" (id 0) (at -34.29 228.6 90))
+    (property "Value" "10" (id 1) (at -25.4 228.6 90))
+    (property "Footprint" "Resistor_SMD:R_0402_1005Metric" (id 2) (at -29.21 229.87 0)
+      (effects (font (size 1.27 1.27)) hide)
+    )
+    (property "Datasheet" "https://jlcpcb.com/partdetail/25820-0402WGF100JTCE/C25077" (id 3) (at -29.21 229.87 0)
+      (effects (font (size 1.27 1.27)) hide)
+    )
+    (property "LCSC" "C25077" (id 4) (at -29.21 229.87 90)
+      (effects (font (size 1.27 1.27)) hide)
+    )
+    (pin "1")
+    (pin "2")
+  )
   (symbol (lib_id "Transistor_FET:AO3401A") (at 328.93 193.04 90) (unit 1)
     (in_bom yes) (on_board yes) (fields_autoplaced)
@@
     (pin "2")
   )
+  (symbol (lib_id "Device:R_Small") (at -29.21 219.71 90) (unit 1)
+    (in_bom yes) (on_board yes)
+    (property "Reference" "R47" (id 0) (at -34.29 218.44 90))
+    (property "Value" "10" (id 1) (at -25.4 218.44 90))
+    (property "Footprint" "Resistor_SMD:R_0402_1005Metric" (id 2) (at -29.21 219.71 0)
+      (effects (font (size 1.27 1.27)) hide)
+    )
+    (property "Datasheet" "https://jlcpcb.com/partdetail/25820-0402WGF100JTCE/C25077" (id 3) (at -29.21 219.71 0)
+      (effects (font (size 1.27 1.27)) hide)
+    )
+    (property "LCSC" "C25077" (id 4) (at -29.21 219.71 90)
+      (effects (font (size 1.27 1.27)) hide)
+    )
+    (pin "1")
+    (pin "2")
+  )
   (symbol (lib_id "power:GND") (at 186.69 212.09 0) (mirror y) (unit 1)
     (in_bom yes) (on_board yes) (fields_autoplaced)
@@
     (pin "2")
   )
+  (symbol (lib_id "Device:R_Small") (at -29.21 232.41 90) (unit 1)
+    (in_bom yes) (on_board yes)
+    (property "Reference" "R50" (id 0) (at -34.29 231.14 90))
+    (property "Value" "10" (id 1) (at -25.4 231.14 90))
+    (property "Footprint" "Resistor_SMD:R_0402_1005Metric" (id 2) (at -29.21 232.41 0)
+      (effects (font (size 1.27 1.27)) hide)
+    )
+    (property "Datasheet" "https://jlcpcb.com/partdetail/25820-0402WGF100JTCE/C25077" (id 3) (at -29.21 232.41 0)
+      (effects (font (size 1.27 1.27)) hide)
+    )
+    (property "LCSC" "C25077" (id 4) (at -29.21 232.41 90)
+      (effects (font (size 1.27 1.27)) hide)
+    )
+    (pin "1")
+    (pin "2")
+  )
   (symbol (lib_id "Device:C_Small") (at 52.07 220.98 0) (mirror y) (unit 1)
     (in_bom yes) (on_board yes)
@@
     (property "Reference" "FB1" (id 0) (at 302.2219 29.21 90))
     (property "Value" "FerriteBead_Small" (id 1) (at 302.2219 31.75 90))
-    (property "Footprint" "" (id 2) (at 302.26 37.338 90)
+    (property "Footprint" "Resistor_SMD:R_0805_2012Metric" (id 2) (at 302.26 37.338 90)
       (effects (font (size 1.27 1.27)) hide)
     )
@@
     (pin "1")
   )
+  (symbol (lib_id "Device:R_Small") (at -29.21 222.25 90) (unit 1)
+    (in_bom yes) (on_board yes)
+    (property "Reference" "R48" (id 0) (at -34.29 220.98 90))
+    (property "Value" "10" (id 1) (at -25.4 220.98 90))
+    (property "Footprint" "Resistor_SMD:R_0402_1005Metric" (id 2) (at -29.21 222.25 0)
+      (effects (font (size 1.27 1.27)) hide)
+    )
+    (property "Datasheet" "https://jlcpcb.com/partdetail/25820-0402WGF100JTCE/C25077" (id 3) (at -29.21 222.25 0)
+      (effects (font (size 1.27 1.27)) hide)
+    )
+    (property "LCSC" "C25077" (id 4) (at -29.21 222.25 90)
+      (effects (font (size 1.27 1.27)) hide)
+    )
+    (pin "1")
+    (pin "2")
+  )
   (symbol (lib_id "power:GND") (at 378.46 212.09 0) (unit 1)
     (in_bom yes) (on_board yes) (fields_autoplaced)
@@
     )
     (path "/7ed5df86-46f1-4eb6-b428-6aa00fc10581"
-      (reference "FB1") (unit 1) (value "FerriteBead_Small") (footprint "")
+      (reference "FB1") (unit 1) (value "FerriteBead_Small") (footprint "Resistor_SMD:R_0805_2012Metric")
     )
     (path "/46bc8e46-a5bf-4c81-ba9c-1dc5a7bb013b"
@@
       (reference "R46") (unit 1) (value "10k") (footprint "Resistor_SMD:R_0402_1005Metric")
     )
+    (path "/2f3f6bb2-60de-4f96-8895-f0880e053a54"
+      (reference "R47") (unit 1) (value "10") (footprint "Resistor_SMD:R_0402_1005Metric")
+    )
+    (path "/acd56cfa-3a6b-4f8d-a122-8cda6fef0833"
+      (reference "R48") (unit 1) (value "10") (footprint "Resistor_SMD:R_0402_1005Metric")
+    )
+    (path "/27adda3e-73e3-4c98-aff5-541fe265b971"
+      (reference "R49") (unit 1) (value "10") (footprint "Resistor_SMD:R_0402_1005Metric")
+    )
+    (path "/4d82f358-b350-4168-9d6f-17ae28a43c9c"
+      (reference "R50") (unit 1) (value "10") (footprint "Resistor_SMD:R_0402_1005Metric")
+    )
     (path "/b92fe6ff-d6b8-4da3-890c-5c9328d5748e/6b541878-701e-4e8c-ad50-4ac4a2855c34"

Commit message: e
Parts:
- removed R24: 27, Resistor_SMD:R_0402_1005Metric, symbol Device:R_Small
Connections:
- net GND: now also U4.17 (PAD)
- net RAW_3v3: now reaches C57.1, Q4.3 (D), U3.2 (VO)
- net buck_out: now reaches D3.1 (K), L4.1, U4.3 (LX), U4.4 (LX), U4.5 (LX)
Other:
- sheet Audio_Codec ports: added none; removed RESET
Changed lines of the file:
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@@
     (stroke (width 0) (type default) (color 0 0 0 0))
   )
-  (wire (pts (xy 96.52 168.91) (xy 104.14 168.91))
-    (stroke (width 0) (type default) (color 0 0 0 0))
-  )
   (wire (pts (xy 166.37 38.1) (xy 160.02 38.1))
     (stroke (width 0) (type default) (color 0 0 0 0))
@@
     (stroke (width 0) (type default) (color 0 0 0 0))
   )
-  (wire (pts (xy 109.22 168.91) (xy 114.3 168.91))
-    (stroke (width 0) (type default) (color 0 0 0 0))
-  )
   (wire (pts (xy 300.99 50.8) (xy 302.26 50.8))
     (stroke (width 0) (type default) (color 0 0 0 0))
@@
     (effects (font (size 1.27 1.27)) (justify left bottom))
   )
+  (label "buck_out" (at 226.695 180.34 180)
+    (effects (font (size 1.27 1.27)) (justify right bottom))
+  )
   (label "DATA_1" (at 52.07 264.16 0)
     (effects (font (size 1.27 1.27)) (justify left bottom))
@@
     (effects (font (size 1.27 1.27)) (justify right bottom))
   )
+  (label "RAW_3v3" (at 361.315 201.93 0)
+    (effects (font (size 1 1)) (justify left bottom))
+  )
   (label "CARD_DETECT" (at 73.66 228.6 0)
     (effects (font (size 1.27 1.27)) (justify left bottom))
@@
     )
   )
-  (global_label "GPIO_48" (shape bidirectional) (at 96.52 168.91 180) (fields_autoplaced)
+  (global_label "GPIO_48" (shape bidirectional) (at -32.385 124.46 180) (fields_autoplaced)
     (effects (font (size 1.27 1.27)) (justify right))
-    (property "Intersheet References" "${INTERSHEET_REFS}" (id 0) (at 86.245 168.8306 0)
+    (property "Intersheet References" "${INTERSHEET_REFS}" (id 0) (at -42.66 124.3806 0)
       (effects (font (size 1.27 1.27)) (justify right) hide)
     )
@@
     (pin "15")
     (pin "16")
+    (pin "17")
     (pin "2")
     (pin "3")
@@
     (pin "1")
   )
-  (symbol (lib_id "Device:R_Small") (at 106.68 168.91 90) (unit 1)
-    (in_bom yes) (on_board yes)
-    (property "Reference" "R24" (id 0) (at 101.6 167.64 90))
-    (property "Value" "27" (id 1) (at 110.49 167.64 90))
-    (property "Footprint" "Resistor_SMD:R_0402_1005Metric" (id 2) (at 106.68 168.91 0)
-      (effects (font (size 1.27 1.27)) hide)
-    )
-    (property "Datasheet" "https://jlcpcb.com/partdetail/25835-0402WGF220JTCE/C25092" (id 3) (at 106.68 168.91 0)
-      (effects (font (size 1.27 1.27)) hide)
-    )
-    (property "LCSC" "C25092" (id 4) (at 106.68 168.91 90)
-      (effects (font (size 1.27 1.27)) hide)
-    )
-    (pin "1")
-    (pin "2")
-  )
   (symbol (lib_id "Device:C_Small") (at 233.68 207.01 0) (mirror x) (unit 1)
     (in_bom yes) (on_board yes)
@@
       (effects (font (size 1.27 1.27)) (justify left top) hide)
     )
-    (pin "RESET" input (at 114.3 168.91 180)
-      (effects (font (size 1.27 1.27)) (justify left))
-    )
     (pin "MCLK" input (at 114.3 171.45 180)
       (effects (font (size 1.27 1.27)) (justify left))
@@
       (reference "R23") (unit 1) (value "5k1") (footprint "Resistor_SMD:R_0402_1005Metric")
     )
-    (path "/b057acb8-e653-4b32-b3b1-e9428339c274"
-      (reference "R24") (unit 1) (value "27") (footprint "Resistor_SMD:R_0402_1005Metric")
-    )
     (path "/880ff5d8-a106-4ac0-a969-88f64c405503"

Commit message: n
Parts:
- added J9: Conn_01x04, Connector_PinHeader_2.54mm:PinHeader_1x04_P2.54mm_Vertical, symbol Connector_Generic:Conn_01x04
Connections:
- net GPIO_9 is gone; now on net AUDIO_ON1: U2.17 (GPIO9/TOUCH9/ADC1_CH8/FSPIHD/SUBSPIHD)
- net SCL is gone; now on net GPIO_35: R23.2
- net SDA is gone; now on net GPIO_36: R22.2
- net +3V3: now also J9.4 (Pin_4)
- net GND: now also J9.1 (Pin_1)
- net GPIO_35: now also J9.3 (Pin_3)
- net GPIO_36: now also J9.2 (Pin_2)

Commit message: g
Connections:
- net GPIO_13 is gone; now on net AUDIO_ON1: U2.21 (GPIO13/TOUCH13/ADC2_CH2/FSPIQ/FSPIIO7/SUBSPIQ)
- net GPIO_4 is gone; now on net AUDIO_ON2: U2.4 (GPIO4/TOUCH4/ADC1_CH3)
- net AUDIO_ON1: no longer U2.17 (GPIO9/TOUCH9/ADC1_CH8/FSPIHD/SUBSPIHD)
- net GPIO_15: now also R48.2
- net GPIO_16: now also Q1.1 (G), R30.2
- net GPIO_45: no longer Q1.1 (G), R30.2
- net GPIO_5: now also R47.2; no longer R50.2
- net GPIO_6: now also R50.2; no longer R49.2
- net GPIO_7: now also R49.2
- new net GPIO_9: U2.17 (GPIO9/TOUCH9/ADC1_CH8/FSPIHD/SUBSPIHD)
Other:
- moved on the sheet: R47, R48

Commit message: r
Parts:
- added BT2: Battery_Cell, Connector_JST:JST_XH_B2B-XH-AM_1x02_P2.50mm_Vertical, symbol Device:Battery_Cell
- added R24: 10, Resistor_SMD:R_0402_1005Metric, symbol Device:R_Small
Connections:
- net AMP_L: now also R49.1; no longer R48.1
- net G1: now also R48.1; no longer R49.1
- net GND: now also BT2.2 (-)
- net GPIO_18: now also R24.2
- net at BT1.1 (+), C10.1, C11.1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: now also BT2.1 (+)
- new net PTT3: R24.1
Other:
- moved on the sheet: BT1, C16, C17

Commit message: y
Parts:
- added D8: red, LED_SMD:LED_0603_1608Metric, symbol Device:LED_Small
- added J10: Conn_01x04, Connector_PinHeader_2.54mm:PinHeader_1x03_P2.54mm_Vertical, symbol Connector_Generic:Conn_01x04
- added R45: 1k, Resistor_SMD:R_0603_1608Metric, symbol Device:R
Connections:
- net GND: now also D8.2 (A), J10.1 (Pin_1)
- net GPIO_43: now also J10.3 (Pin_3)
- net GPIO_44: now also J10.2 (Pin_2)
- net +BATT: now reaches BT1.1 (+), BT2.1 (+), C10.1, C11.1, C16.1, C17.2, L1.1, R43.1, U4.9 (BAT)
- net +BATT: now also R45.2
- new net: D8.1 (K), R45.1
- no-connect marks 14 -> 16
Other:
- note added: "COMMON RF POWER SET PIN"
- note added: "EXTERNAL PTT PIN"
- note added: "MODULE 1"
- note added: "MODULE 2"
- note added: "POWER AMPLIFIER"
- note added: "POWER SUPPLY: BMS + CHARGEING + REGULATION"
- note added: "RF MODULE PIN SETUP"
- note added: "reversed on purpose"
- title: (none) -> Cross band handy walkie talkie V2
- moved on the sheet: BT1, BT2, C10, C11, C12, C13, C16, C17, C53, C57, C58, C59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

Commit message: b
Parts:
- added TP10, TP11, TP12, TP13, TP4, TP5, TP6, TP7, TP9: TestPoint, TestPoint:TestPoint_Pad_1.0x1.0mm, symbol Connector:TestPoint
Connections:
- net +3V3: now also TP7.1
- net GND: now also TP10.1, TP11.1, TP4.1, TP5.1, TP6.1, TP9.1
- net GPIO_43: now also TP12.1
- net GPIO_44: now also TP13.1
