File: HW/cross_band_handy_walkie_talkie_ES8388/cross_band_handy_walkie_talkie_ES8388.kicad_sch (KiCad schematic)
At the start: 105 parts, among them J1 USB_C_Receptacle, J10 Conn_01x04, J2 Micro_SD_Card_Det, J9 Conn_01x04, Q1 nMOS, Q2 AO3401A, Q3 AO3401A, Q4 AO3401A, SW1 MCU_RESET, SW2 MCU_RESET, U1 SRV05-4, U2 ESP32-S3-WROOM-1, U3 AMS1117-3.3, U4 TP5000

Commit message: b
Parts:
- added Q6: nMOS, Package_TO_SOT_SMD:SOT-23, symbol Device:Q_NMOS_GSD
- added R52, R53: 10k, Resistor_SMD:R_0402_1005Metric, symbol Device:R_Small
Connections:
- net +BATT: now also D8.1 (K); no longer R45.2
- net GND: now also R45.1, Q6.2 (S), R53.2; no longer D8.2 (A), Q4.1 (G)
- net RAW_3v3: now also Q6.1 (G), R53.1
- net BATT_filtered: now reaches C58.1, C59.1, L1.2, Q2.2 (S)
- net BATT_filtered: now also R52.2
- new net: Q4.1 (G), Q6.3 (D), R52.1
- new net: D8.2 (A), R45.2
Other:
- note added: "BOOT & ENABLE BUTTONS"
- note added: "Emergency UART programer"
- note added: "I am out of pins..."
- note added: "I2C"
- note added: "USB+ESC TVS + Indicator LEDs"
- moved on the sheet: BT1, BT2, C1, C10, C11, C2, C3, C4, C5, C57, C58, C59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

Commit message: f
Connections:
- no-connect marks 16 -> 17
Other:
- moved on the sheet: TP1
Changed lines of the file:
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@@
   (no_connect (at 355.6 71.12))
   (no_connect (at 247.65 265.43))
+  (no_connect (at 260.35 93.98))
   (no_connect (at 355.6 78.74))
   (no_connect (at 355.6 93.98))
@@
     (pin "1")
   )
-  (symbol (lib_id "Connector:TestPoint") (at -17.78 99.06 270) (unit 1)
+  (symbol (lib_id "Connector:TestPoint") (at 260.35 93.98 270) (unit 1)
     (in_bom no) (on_board no) (fields_autoplaced)
-    (property "Reference" "TP1" (id 0) (at -11.43 99.0599 90)
+    (property "Reference" "TP1" (id 0) (at 266.7 93.9799 90)
       (effects (font (size 1.27 1.27)) (justify left))
     )
-    (property "Value" "TestPoint" (id 1) (at -15.7479 102.87 0)
+    (property "Value" "TestPoint" (id 1) (at 262.3821 97.79 0)
       (effects (font (size 1.27 1.27)) (justify left) hide)
     )
-    (property "Footprint" "TestPoint:TestPoint_Pad_1.0x1.0mm" (id 2) (at -17.78 104.14 0)
+    (property "Footprint" "TestPoint:TestPoint_Pad_1.0x1.0mm" (id 2) (at 260.35 99.06 0)
       (effects (font (size 1.27 1.27)) hide)
     )
-    (property "Datasheet" "~" (id 3) (at -17.78 104.14 0)
+    (property "Datasheet" "~" (id 3) (at 260.35 99.06 0)
       (effects (font (size 1.27 1.27)) hide)
     )

Commit message: R
Parts:
- added SW3: SW_SPDT, Z_mycustom_footprint_lib:MSK-12d19, symbol Switch:SW_SPDT
Connections:
- net BATT_filtered: now also SW3.1 (A); no longer C58.1, C59.1, L1.2
- new net: C58.1, C59.1, L1.2, SW3.2 (B)
- no-connect marks 17 -> 18
Other:
- moved on the sheet: C57, C61, C62, C7, Q2, Q3, Q4, Q6, R46, R52, R53, TP10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

Commit message: b
Parts:
- L1, L4: LCSC C3002553 -> C602016
Changed lines of the file:
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@@
       (effects (font (size 1.27 1.27)) hide)
     )
-    (property "LCSC" "C3002553" (id 4) (at 240.03 191.77 90)
+    (property "LCSC" "C602016" (id 4) (at 240.03 191.77 90)
       (effects (font (size 1.27 1.27)) hide)
     )
@@
       (effects (font (size 1.27 1.27)) hide)
     )
-    (property "LCSC" "C3002553" (id 4) (at 198.12 191.77 90)
-      (effects (font (size 1.27 1.27)) hide)
-    )
+    (property "LCSC" "C602016" (id 4) (at 198.12 191.77 90)
+      (effects (font (size 1.27 1.27)) hide)
+    )
