File: HW/cross_band_handy_walkie_talkie_ES8388/Audio_Codec.kicad_sch (KiCad schematic)
At the start: 46 parts

Commit message: t
Parts:
- removed C? (x6): 1u, Capacitor_SMD:C_0603_1608Metric_Pad1.08x0.95mm_HandSolder, symbol Device:C_Small
- removed C? (x6): 100n, Capacitor_SMD:C_0603_1608Metric_Pad1.08x0.95mm_HandSolder, symbol Device:C_Small
- removed C? (x3): 10u, Capacitor_SMD:C_0805_2012Metric, symbol Device:C_Small
- removed J? (x2): AUDIO, Connector_PinHeader_2.54mm:PinHeader_1x03_P2.54mm_Vertical, symbol Connector_Generic:Conn_01x03
- removed R? (x7): 1k, Resistor_SMD:R_0603_1608Metric_Pad0.98x0.95mm_HandSolder, symbol Device:R_Small
- removed R?: 2k7, Resistor_SMD:R_0603_1608Metric_Pad0.98x0.95mm_HandSolder, symbol Device:R_Small
- removed TP?: TestPoint_THT, TestPoint:TestPoint_Loop_D2.60mm_Drill0.9mm_Beaded, symbol Connector:TestPoint
- removed U?: TLV320AIC3254, Package_DFN_QFN:QFN-32-1EP_5x5mm_P0.5mm_EP3.1x3.1mm_ThermalVias, symbol My_custom_lib:TLV320AIC3254
- added C24, C25, C27, C28, C30, C31, C34, C35, C? (x6): 1u, Capacitor_SMD:C_0603_1608Metric_Pad1.08x0.95mm_HandSolder, symbol Device:C_Small
- added C? (x8): 10u, Capacitor_SMD:C_0805_2012Metric, symbol Device:C_Small
- added JP1: 3p, Jumper:SolderJumper-3_P1.3mm_Bridged12_Pad1.0x1.5mm, symbol Jumper:Jumper_3_Bridged12
- gave numbers to parts that had none: 19
Connections:
- net +3V3: now also U6.2 (DVDD), U6.3 (PVDD), C?.1, C?.1, C?.2, C?.2, JP1.3 (B); no longer C32.1, C33.1
- net +5V: now also C?.1, C?.1
- net BCLK: now also U6.5 (SCLK)
- net DIN: now also U6.6 (DSDIN)
- net DOUT: now also U6.8 (ASDOUT)
- net GND: now also U6.13 (HPGND), C?.1, C?.1, C?.1, C?.1, C?.1, C?.1, C?.2, C?.2, C?.2, C?.2, C?.2, C?.2, C?.2, C?.2, JP1.1 (A); no longer U6.17 (AVDD)
- net MCLK: now also U6.1 (MCLK)
- net SCL: now also U6.28 (CCLK)
- net SDA: now also U6.27 (CDATA)
- net WCLK: now also U6.7 (LRCK)
- net at C29.1, J5.T: no longer R28.1
- net at R31.1: no longer R30.1
- net at L1.2, U5.9 (AVDD): now also C?.1
- net at U6.10 (VREF): now also C?.1
- net at U6.11 (ROUT1): now also C31.2
- net at U6.12 (LOUT1): now also C30.2
- net at U6.14 (ROUT2): now also C34.1
- net at U6.15 (LOUT2): now also C35.1
- net at U6.16 (HPVDD): now also C?.1, C?.2
- net at U6.19 (ADCVREF): now also C32.1, C?.2
- net at U6.20 (VMID): now also C33.1, C?.2
- net at U6.21 (RIN2): now also C28.1
- net at U6.22 (LIN2): now also C27.1
- net at U6.23 (RIN1): now also C25.1
- net at U6.24 (LIN1): now also C24.1
- net at U6.26 (CE): now also JP1.2 (C)
- new net: C?.1, C?.2, U6.17 (AVDD)
Other:
- note removed: "0011000"
- moved on the sheet: C16, C18, C19, C20, C21, C22, C23, C26, C29, C32, C33, J5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

Commit message: b
Parts:
- removed R28: 100k, Resistor_SMD:R_0805_2012Metric, symbol Device:R
- removed R30: 1k, Resistor_SMD:R_0603_1608Metric_Pad0.98x0.95mm_HandSolder, symbol Device:R_Small
- removed R31: 2k7, Resistor_SMD:R_0603_1608Metric_Pad0.98x0.95mm_HandSolder, symbol Device:R_Small
- added C? (x2): 10u, Capacitor_SMD:C_0805_2012Metric, symbol Device:C_Small
- added C? (x2): 1u, Capacitor_SMD:C_0603_1608Metric_Pad1.08x0.95mm_HandSolder, symbol Device:C_Small
- added J?: Conn_01x04, symbol Connector_Generic:Conn_01x04
- added JP?: 3p, Jumper:SolderJumper-3_P1.3mm_Bridged12_Pad1.0x1.5mm, symbol Jumper:Jumper_3_Bridged12
- added L? (x2): L_Small, Inductor_SMD:L_0603_1608Metric, symbol Device:L_Small
- added R? (x4): 2k2, Resistor_SMD:R_0603_1608Metric_Pad0.98x0.95mm_HandSolder, symbol Device:R_Small
Connections:
- net +3V3: now also C?.1, C?.1, JP?.1 (A), L?.1, L?.1; no longer C?.1, C?.1, C?.2, C?.2, U6.2 (DVDD), U6.3 (PVDD)
- net +5V: now also JP?.3 (B); no longer C16.1, C?.1, C?.1, L1.1, U5.13 (PVDD), U5.3 (PVDD)
- net GND: now also C?.2, C?.2
- net L_out1: now reaches C30.1
- net L_out1: now also R?.2
- net Jack_MIC_INPUT_1: now reaches J5.S
- net Jack_MIC_INPUT_1: now also C27.2
- net at C34.2: now also C26.2
- net at U5.16 (OUTR+): now also J?.3 (Pin_3)
- net at U5.17 (OUTR-): now also J?.4 (Pin_4)
- net at U5.2 (OUTL+): now also J?.1 (Pin_1)
- net at U5.5 (OUTL-): now also J?.2 (Pin_2)
- net at C?.1, L1.2, U5.9 (AVDD): now also C16.1, C?.1, U5.13 (PVDD), U5.3 (PVDD)
- net at C29.2: now also C35.2
- net R_out1: now reaches C31.1
- net R_out1: now also R?.2
- net Tranceiver_Audio_IN_2: now reaches C25.2
- net Tranceiver_Audio_IN_1: now reaches C24.2
- net Audio_OUT_L: no longer names the net of C18.1, C19.1
- net Audio_OUT_L: now also R?.1, R?.2
- net Audio_OUT_R: no longer names the net of C21.1, C22.1
- net Audio_OUT_R: now also R?.1, R?.1
- net GPIO_4 renamed AMP_L
- net AMP_L: no longer U5.8 (~{SDR})
- net GPIO_5 renamed G1
- net GPIO_6 renamed G0
- new net: C?.1, C?.1, C?.2, C?.2, L?.2, L?.2, U6.2 (DVDD), U6.3 (PVDD)
- new net: C?.1, R?.1
- new net: C?.1, JP?.2 (C), L1.1
- new net: C?.2, R?.2
- new net AMP_R: U5.8 (~{SDR})
- new net Tranceiver_Audio_OUT_1: C?.2
- new net Tranceiver_Audio_OUT_2: C?.1
Other:
- note added: "001000x"
- note added: "RC cut off 2k2 + 4n7 15399 Hz"
- moved on the sheet: C16, C18, C19, C20, C21, C22, C23, C24, C25, C26, C27, C28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

Commit message: f
Parts:
- removed C25, C27, C31, C34, C35: 1u, Capacitor_SMD:C_0603_1608Metric_Pad1.08x0.95mm_HandSolder, symbol Device:C_Small
- removed R29: 100k, Resistor_SMD:R_0805_2012Metric, symbol Device:R
- added C26, C33, C36: 22u, Capacitor_SMD:C_0805_2012Metric, symbol Device:C_Small
- added C54, C57: 10u, Capacitor_SMD:C_0805_2012Metric, symbol Device:C_Small
- added C55, C56: 1u, Capacitor_SMD:C_0603_1608Metric_Pad1.08x0.95mm_HandSolder, symbol Device:C_Small
- added D6, D7: red, LED_SMD:LED_0603_1608Metric, symbol Device:LED_Small
- added FL1, FL2: LFCN-160, Filter:Filter_Mini-Circuits_FV1206, symbol RF_Filter:LFCN-160
- added J4: Conn_01x06, Connector_PinHeader_2.54mm:PinHeader_1x06_P2.54mm_Vertical, symbol Connector_Generic:Conn_01x06
- added J7, J8: SMA, Connector_Coaxial:SMA_Amphenol_901-144_Vertical, symbol Connector:Conn_Coaxial
- added R31, R37, R42: 10k, Resistor_SMD:R_0603_1608Metric_Pad0.98x0.95mm_HandSolder, symbol Device:R_Small
- added R38, R39: 1k, Resistor_SMD:R_0805_2012Metric, symbol Device:R
- added R41: 2k2, Resistor_SMD:R_0603_1608Metric_Pad0.98x0.95mm_HandSolder, symbol Device:R_Small
- added RV1, RV2, RV3, RV4: 10k, symbol Device:R_Potentiometer
- added U7, U8: SA818S, Z_mycustom_footprint_lib:SA818S, symbol My_custom_lib:SA818S
- C24, C28, C30: value 1u -> 22u; footprint Capacitor_SMD:C_0603_1608Metric_Pad1.08x0.95mm_HandSolder -> Capacitor_SMD:C_0805_2012Metric; LCSC C15849 -> C45783
- gave numbers to parts that had none: 26
- renumbered C16 to C15, C18 to C25, C19 to C27, C20 to C29, C21 to C31, C22 to C32, C23 to C35, C32 to C43, C33 to C44, C26 to C48, C29 to C49, J5 to J6, JP1 to JP2, U6 to U5, U5 to U6
Connections:
- net +3V3: now also J4.1 (Pin_1), R41.1, R42.1
- net +5V: now also C54.1, C55.2, C56.1, C57.2, U7.8 (VBATT), U8.8 (VBATT)
- net GND: now also C54.2, C55.1, C56.2, C57.1, FL1.2 (GND), FL1.4 (GND), FL2.2 (GND), FL2.4 (GND), J4.2 (Pin_2), J4.5 (Pin_5), J7.2 (Ext), J8.2 (Ext), R31.1, R37.2, R38.2, R39.2, RV1.1, RV2.3, RV3.3, RV4.3, U7.10 (GND), U7.9 (GND), U8.10 (GND), U8.9 (GND)
- net JACK_DETECT: now also R42.2
- net Jack_MIC_INPUT_1: now also C26.2, R41.2
- net L_out1: now also C36.1; no longer C30.1
- net R_out1: now also C33.1
- net Tranceiver_Audio_IN_1: now also U8.18 (MIC_IN); no longer C24.2
- net Tranceiver_Audio_IN_2: now also U7.18 (MIC_IN)
- net Tranceiver_Audio_OUT_1: now also RV1.3, RV4.1, U8.3 (AF(Audio_OUT)); no longer C17.2
- net Tranceiver_Audio_OUT_2: now also RV2.1, RV3.1, U7.3 (AF(Audio_OUT)); no longer C37.1
- net at U5.12 (LOUT1): now also C36.2; no longer C30.2
- net 3V33: now reaches C20.2, C21.1, C22.1, C23.2, L2.2, L3.2, U5.2 (DVDD), U5.3 (PVDD)
- net 3V33: now also C38.2, C39.1, C40.1, C41.2, U5.16 (HPVDD), U5.17 (AVDD)
- net at U5.14 (ROUT2): now also C48.2
- net at U5.21 (RIN2): now also C30.1; no longer C28.1
- net LINE_IN2: now reaches C28.2
- net LINE_IN2: now also RV3.2
- net at C35.2: now also U6.18 (INR+); no longer U6.17 (OUTR-)
- net at C25.2: now also U6.19 (INL-); no longer U6.20 (INL+)
- net at C31.2: now also U6.17 (OUTR-); no longer U6.18 (INR+)
- net at C29.2: now also U6.20 (INL+); no longer U6.19 (INL-)
- net at U5.11 (ROUT1): now also C33.2
- net at U5.15 (LOUT2): now also C49.2
- net at U5.22 (LIN2): now also C28.1
- net at U5.23 (RIN1): now also C26.1
- new net: D7.1 (K), R39.1
- new net: C37.1, RV2.2
- new net: C17.2, RV1.2
- new net: D6.1 (K), R38.1
- new net AMPLIFIED_AUDIO_OUT: J4.3 (Pin_3)
- new net AUDIO_ON1: U8.1 (Audio_ON)
- new net AUDIO_ON2: U7.1 (Audio_ON)
- new net H/L1: U8.7 (H/L)
- new net H/L2: U7.7 (H/L)
- new net LINE_IN1: C24.2, RV4.2
- new net MIC-AMP_IN: J4.6 (Pin_6)
- new net MIC_EST_PTT: J4.4 (Pin_4)
- new net MIC_INPUT_2: C30.2
- new net PD1: R31.2, U8.6 (PD)
- new net PD2: R37.1, U7.6 (PD)
- new net PTT1: D6.2 (A), U8.5 (PTT)
- new net PTT2: D7.2 (A), U7.5 (PTT)
- new net RX1: U8.17 (TXD(TX))
- new net RX2: U7.17 (TXD(TX))
- new net TX1: U8.16 (RXD_(RX))
- new net TX2: U7.16 (RXD_(RX))
- new net ant1: FL1.1 (IN), U7.12 (ANT)
- new net ant2: FL1.3 (OUT), J7.1 (In)
- new net ant3: FL2.1 (IN), U8.12 (ANT)
- new net ant4: FL2.3 (OUT), J8.1 (In)
Other:
- note added: "750mA max current"
- note added: "AUDIO IO"
- note added: "MIC bias resistor???"
- note added: "RF MODULES"
- note added: "SA818-1"
- note added: "SA818-2"
- moved on the sheet: C13, C14, C15, C16, C17, C25, C27, C29, C31, C32, C35, C37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

Commit message: f
Parts:
- RV1, RV2, RV3, RV4: footprint (none) -> Potentiometer_SMD:Potentiometer_Bourns_3314J_Vertical; LCSC (none) -> C36376
Connections:
- net GND: now also RV4.1; no longer RV4.3
- net Tranceiver_Audio_OUT_1: now also RV4.3; no longer RV4.1
Other:
- moved on the sheet: C54
Changed lines of the file:
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@@
     (stroke (width 0) (type default) (color 0 0 0 0))
   )
-  (wire (pts (xy 193.04 220.98) (xy 200.66 220.98))
+  (wire (pts (xy 195.58 220.98) (xy 200.66 220.98))
     (stroke (width 0) (type default) (color 0 0 0 0))
   )
@@
     (stroke (width 0) (type default) (color 0 0 0 0))
   )
-  (wire (pts (xy 193.04 227.33) (xy 193.04 229.87))
+  (wire (pts (xy 195.58 227.33) (xy 195.58 229.87))
     (stroke (width 0) (type default) (color 0 0 0 0))
   )
@@
     (stroke (width 0) (type default) (color 0 0 0 0))
   )
-  (wire (pts (xy 193.04 220.98) (xy 193.04 222.25))
+  (wire (pts (xy 195.58 220.98) (xy 195.58 222.25))
     (stroke (width 0) (type default) (color 0 0 0 0))
   )
@@
     (pin "1")
   )
-  (symbol (lib_id "power:GND") (at 193.04 229.87 0) (unit 1)
+  (symbol (lib_id "power:GND") (at 195.58 229.87 0) (unit 1)
     (in_bom yes) (on_board yes) (fields_autoplaced)
-    (property "Reference" "#PWR095" (id 0) (at 193.04 236.22 0)
+    (property "Reference" "#PWR095" (id 0) (at 195.58 236.22 0)
       (effects (font (size 1.27 1.27)) hide)
     )
-    (property "Value" "GND" (id 1) (at 193.04 234.95 0)
+    (property "Value" "GND" (id 1) (at 195.58 234.95 0)
       (effects (font (size 1.27 1.27)) hide)
     )
-    (property "Footprint" "" (id 2) (at 193.04 229.87 0)
+    (property "Footprint" "" (id 2) (at 195.58 229.87 0)
       (effects (font (size 1.27 1.27)) hide)
     )
-    (property "Datasheet" "" (id 3) (at 193.04 229.87 0)
+    (property "Datasheet" "" (id 3) (at 195.58 229.87 0)
       (effects (font (size 1.27 1.27)) hide)
     )
@@
     (pin "1")
   )
-  (symbol (lib_id "Device:R_Potentiometer") (at 320.04 106.68 90) (unit 1)
-    (in_bom yes) (on_board yes) (fields_autoplaced)
-    (property "Reference" "RV2" (id 0) (at 320.04 110.49 90))
-    (property "Value" "10k" (id 1) (at 320.04 113.03 90))
-    (property "Footprint" "" (id 2) (at 320.04 106.68 0)
-      (effects (font (size 1.27 1.27)) hide)
-    )
-    (property "Datasheet" "~" (id 3) (at 320.04 106.68 0)
-      (effects (font (size 1.27 1.27)) hide)
-    )
-    (pin "1")
-    (pin "2")
-    (pin "3")
-  )
   (symbol (lib_id "My_custom_lib:SA818S") (at 93.98 238.76 0) (mirror y) (unit 1)
     (in_bom yes) (on_board yes) (fields_autoplaced)
@@
     (pin "1")
   )
+  (symbol (lib_id "Device:R_Potentiometer") (at 226.06 129.54 270) (unit 1)
+    (in_bom yes) (on_board yes) (fields_autoplaced)
+    (property "Reference" "RV3" (id 0) (at 226.06 123.19 90))
+    (property "Value" "10k" (id 1) (at 226.06 125.73 90))
+    (property "Footprint" "Potentiometer_SMD:Potentiometer_Bourns_3314J_Vertical" (id 2) (at 226.06 129.54 0)
+      (effects (font (size 1.27 1.27)) hide)
+    )
+    (property "Datasheet" "~" (id 3) (at 226.06 129.54 0)
+      (effects (font (size 1.27 1.27)) hide)
+    )
+    (property "LCSC" "C36376" (id 4) (at 226.06 129.54 90)
+      (effects (font (size 1.27 1.27)) hide)
+    )
+    (pin "1")
+    (pin "2")
+    (pin "3")
+  )
   (symbol (lib_id "power:GND") (at 219.71 157.48 0) (mirror y) (unit 1)
     (in_bom yes) (on_board yes) (fields_autoplaced)
@@
     (pin "2")
   )
-  (symbol (lib_id "Device:R_Potentiometer") (at 226.06 154.94 270) (mirror x) (unit 1)
-    (in_bom yes) (on_board yes) (fields_autoplaced)
-    (property "Reference" "RV4" (id 0) (at 226.06 158.115 90))
-    (property "Value" "10k" (id 1) (at 226.06 160.655 90))
-    (property "Footprint" "" (id 2) (at 226.06 154.94 0)
-      (effects (font (size 1.27 1.27)) hide)
-    )
-    (property "Datasheet" "~" (id 3) (at 226.06 154.94 0)
-      (effects (font (size 1.27 1.27)) hide)
-    )
-    (pin "1")
-    (pin "2")
-    (pin "3")
-  )
   (symbol (lib_id "power:+3V3") (at 69.85 63.5 0) (unit 1)
     (in_bom yes) (on_board yes) (fields_autoplaced)
@@
   )
   (symbol (lib_id "My_custom_lib:TPA2012D2") (at 360.68 83.82 0) (unit 1)
-    (in_bom yes) (on_board yes) (fields_autoplaced)
-    (property "Reference" "U6" (id 0) (at 365.2394 64.77 0)
+    (in_bom yes) (on_board yes)
+    (property "Reference" "U6" (id 0) (at 367.03 102.87 0)
       (effects (font (size 1.27 1.27)) (justify left))
     )
-    (property "Value" "TPA2012D2" (id 1) (at 365.2394 67.31 0)
+    (property "Value" "TPA2012D2" (id 1) (at 367.03 105.41 0)
       (effects (font (size 1.27 1.27)) (justify left))
     )
@@
     (property "Reference" "RV1" (id 0) (at 306.07 36.83 90))
     (property "Value" "10k" (id 1) (at 306.07 39.37 90))
-    (property "Footprint" "" (id 2) (at 306.07 43.18 0)
+    (property "Footprint" "Potentiometer_SMD:Potentiometer_Bourns_3314J_Vertical" (id 2) (at 306.07 43.18 0)
       (effects (font (size 1.27 1.27)) hide)
     )
@@
       (effects (font (size 1.27 1.27)) hide)
     )
+    (property "LCSC" "C36376" (id 4) (at 306.07 43.18 90)
+      (effects (font (size 1.27 1.27)) hide)
+    )
     (pin "1")
     (pin "2")
@@
     (pin "2")
   )
-  (symbol (lib_id "Device:R_Potentiometer") (at 226.06 129.54 270) (unit 1)
-    (in_bom yes) (on_board yes) (fields_autoplaced)
-    (property "Reference" "RV3" (id 0) (at 226.06 123.825 90))
-    (property "Value" "10k" (id 1) (at 226.06 126.365 90))
-    (property "Footprint" "" (id 2) (at 226.06 129.54 0)
-      (effects (font (size 1.27 1.27)) hide)
-    )
-    (property "Datasheet" "~" (id 3) (at 226.06 129.54 0)
-      (effects (font (size 1.27 1.27)) hide)
-    )
-    (pin "1")
-    (pin "2")
-    (pin "3")
-  )
   (symbol (lib_id "Device:C_Small") (at 132.08 134.62 90) (mirror x) (unit 1)
     (in_bom yes) (on_board yes)
@@
     (pin "1")
   )
-  (symbol (lib_id "Device:C_Small") (at 193.04 224.79 0) (unit 1)
+  (symbol (lib_id "Device:C_Small") (at 195.58 224.79 0) (unit 1)
     (in_bom yes) (on_board yes)
-    (property "Reference" "C54" (id 0) (at 186.69 224.79 0)
+    (property "Reference" "C54" (id 0) (at 189.23 224.79 0)
       (effects (font (size 1.27 1.27)) (justify left))
     )
-    (property "Value" "10u" (id 1) (at 186.69 227.33 0)
+    (property "Value" "10u" (id 1) (at 189.23 227.33 0)
       (effects (font (size 1.27 1.27)) (justify left))
     )
-    (property "Footprint" "Capacitor_SMD:C_0805_2012Metric" (id 2) (at 193.04 224.79 0)
+    (property "Footprint" "Capacitor_SMD:C_0805_2012Metric" (id 2) (at 195.58 224.79 0)
       (effects (font (size 1.27 1.27)) hide)
     )
-    (property "Datasheet" "~" (id 3) (at 193.04 224.79 0)
+    (property "Datasheet" "~" (id 3) (at 195.58 224.79 0)
       (effects (font (size 1.27 1.27)) hide)
     )
-    (property "LCSC" "C15850" (id 4) (at 193.04 224.79 0)
+    (property "LCSC" "C15850" (id 4) (at 195.58 224.79 0)
       (effects (font (size 1.27 1.27)) hide)
     )
@@
     (pin "1")
   )
+  (symbol (lib_id "Device:R_Potentiometer") (at 320.04 106.68 90) (unit 1)
+    (in_bom yes) (on_board yes) (fields_autoplaced)
+    (property "Reference" "RV2" (id 0) (at 320.04 110.49 90))
+    (property "Value" "10k" (id 1) (at 320.04 113.03 90))
+    (property "Footprint" "Potentiometer_SMD:Potentiometer_Bourns_3314J_Vertical" (id 2) (at 320.04 106.68 0)
+      (effects (font (size 1.27 1.27)) hide)
+    )
+    (property "Datasheet" "~" (id 3) (at 320.04 106.68 0)
+      (effects (font (size 1.27 1.27)) hide)
+    )
+    (property "LCSC" "C36376" (id 4) (at 320.04 106.68 90)
+      (effects (font (size 1.27 1.27)) hide)
+    )
+    (pin "1")
+    (pin "2")
+    (pin "3")
+  )
   (symbol (lib_id "Device:L_Small") (at 92.71 59.69 90) (unit 1)
     (in_bom yes) (on_board yes) (fields_autoplaced)
@@
     (pin "2")
   )
+  (symbol (lib_id "Device:R_Potentiometer") (at 226.06 154.94 90) (unit 1)
+    (in_bom yes) (on_board yes) (fields_autoplaced)
+    (property "Reference" "RV4" (id 0) (at 226.06 158.75 90))
+    (property "Value" "10k" (id 1) (at 226.06 161.29 90))
+    (property "Footprint" "Potentiometer_SMD:Potentiometer_Bourns_3314J_Vertical" (id 2) (at 226.06 154.94 0)
+      (effects (font (size 1.27 1.27)) hide)
+    )
+    (property "Datasheet" "~" (id 3) (at 226.06 154.94 0)
+      (effects (font (size 1.27 1.27)) hide)
+    )
+    (property "LCSC" "C36376" (id 4) (at 226.06 154.94 90)
+      (effects (font (size 1.27 1.27)) hide)
+    )
+    (pin "1")
+    (pin "2")
+    (pin "3")
+  )
   (symbol (lib_id "Device:R") (at 146.05 266.7 0) (unit 1)
