File: HW/cross_band_handy_walkie_talkie_ES8388/Audio_Codec.kicad_sch (KiCad schematic)
At the start: 71 parts, among them J4 Conn_01x06, J5 Conn_01x04, J6 AudioJack4_SwitchTR1, J7 SMA, J8 SMA, U5 ES8388, U6 TPA2012D2, U7 SA818S, U8 SA818S

Commit message: l
Parts:
- removed L1: L_Small, Inductor_SMD:L_0603_1608Metric, symbol Device:L_Small
- J4: now left out of the parts list
- J5: footprint (none) -> TerminalBlock:TerminalBlock_bornier-4_P5.08mm
- L2, L3: value L_Small -> 4u7; footprint Inductor_SMD:L_0603_1608Metric -> Z_mycustom_footprint_lib:Inductor_2.5x2x1.2mm; LCSC C13415 -> C3002553
Connections:
- net +3V3: no longer L2.1
- net 3V33: no longer L2.2
- net at C13.1, JP1.2 (C): now also L2.1
- net at C14.1, C15.1, C16.1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: now also L2.2
- net AMPLIFIED_AUDIO_OUT renamed EXT_SPEAKER+
Changed lines of the file:
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@@
   (junction (at 331.47 71.12) (diameter 0) (color 0 0 0 0)
   )
-  (junction (at 86.36 67.31) (diameter 0) (color 0 0 0 0)
-  )
   (junction (at 361.95 104.14) (diameter 0) (color 0 0 0 0)
   )
@@
   (junction (at 74.93 67.31) (diameter 0) (color 0 0 0 0)
   )
-  (junction (at 101.6 67.31) (diameter 0) (color 0 0 0 0)
-  )
   (no_connect (at 143.51 85.09))
   (no_connect (at 173.99 72.39))
@@
     (stroke (width 0) (type default) (color 0 0 0 0))
   )
-  (wire (pts (xy 99.06 67.31) (xy 101.6 67.31))
+  (wire (pts (xy 99.06 67.31) (xy 107.95 67.31))
     (stroke (width 0) (type default) (color 0 0 0 0))
   )
@@
     (stroke (width 0) (type default) (color 0 0 0 0))
   )
-  (wire (pts (xy 83.82 67.31) (xy 86.36 67.31))
+  (wire (pts (xy 83.82 67.31) (xy 90.17 67.31))
     (stroke (width 0) (type default) (color 0 0 0 0))
   )
@@
     (stroke (width 0) (type default) (color 0 0 0 0))
   )
-  (wire (pts (xy 101.6 59.69) (xy 101.6 67.31))
-    (stroke (width 0) (type default) (color 0 0 0 0))
-  )
   (wire (pts (xy 242.57 96.52) (xy 242.57 86.36))
     (stroke (width 0) (type default) (color 0 0 0 0))
@@
     (stroke (width 0) (type default) (color 0 0 0 0))
   )
-  (wire (pts (xy 86.36 67.31) (xy 90.17 67.31))
-    (stroke (width 0) (type default) (color 0 0 0 0))
-  )
   (polyline (pts (xy 151.13 199.39) (xy 274.32 199.39))
     (stroke (width 0) (type default) (color 0 0 0 0))
@@
     (stroke (width 0) (type default) (color 0 0 0 0))
   )
-  (wire (pts (xy 330.2 217.17) (xy 351.79 217.17))
+  (wire (pts (xy 330.2 217.17) (xy 347.98 217.17))
     (stroke (width 0) (type default) (color 0 0 0 0))
   )
@@
     (stroke (width 0) (type default) (color 0 0 0 0))
   )
-  (wire (pts (xy 86.36 59.69) (xy 86.36 67.31))
-    (stroke (width 0) (type default) (color 0 0 0 0))
-  )
-  (wire (pts (xy 90.17 59.69) (xy 86.36 59.69))
-    (stroke (width 0) (type default) (color 0 0 0 0))
-  )
   (wire (pts (xy 107.95 73.66) (xy 107.95 74.93))
     (stroke (width 0) (type default) (color 0 0 0 0))
@@
     (stroke (width 0) (type default) (color 0 0 0 0))
   )
-  (wire (pts (xy 95.25 59.69) (xy 101.6 59.69))
-    (stroke (width 0) (type default) (color 0 0 0 0))
-  )
   (wire (pts (xy 326.39 52.07) (xy 326.39 55.88))
     (stroke (width 0) (type default) (color 0 0 0 0))
@@
     (stroke (width 0) (type default) (color 0 0 0 0))
   )
-  (wire (pts (xy 101.6 67.31) (xy 107.95 67.31))
-    (stroke (width 0) (type default) (color 0 0 0 0))
-  )
   (text "RC cut off\n2k2 + 4n7\n15399 Hz" (at 301.625 63.5 0)
     (effects (font (size 1.27 1.27)) (justify left bottom))
@@
     (effects (font (size 1.27 1.27)) (justify right bottom))
   )
-  (label "AMPLIFIED_AUDIO_OUT" (at 351.79 217.17 0)
-    (effects (font (size 1.27 1.27)) (justify left bottom))
-  )
   (label "ant3" (at 69.85 238.76 0)
     (effects (font (size 1.27 1.27)) (justify left bottom))
@@
     (pin "1")
   )
-  (symbol (lib_id "Device:L_Small") (at 92.71 67.31 90) (unit 1)
-    (in_bom yes) (on_board yes) (fields_autoplaced)
-    (property "Reference" "L3" (id 0) (at 92.71 62.23 90))
-    (property "Value" "L_Small" (id 1) (at 92.71 64.77 90))
-    (property "Footprint" "Inductor_SMD:L_0603_1608Metric" (id 2) (at 92.71 67.31 0)
-      (effects (font (size 1.27 1.27)) hide)
-    )
-    (property "Datasheet" "~" (id 3) (at 92.71 67.31 0)
-      (effects (font (size 1.27 1.27)) hide)
-    )
-    (property "LCSC" "C13415" (id 4) (at 92.71 67.31 90)
-      (effects (font (size 1.27 1.27)) hide)
-    )
-    (pin "1")
-    (pin "2")
-  )
   (symbol (lib_id "Connector:AudioJack4_SwitchTR1") (at 101.6 129.54 0) (unit 1)
     (in_bom yes) (on_board yes) (fields_autoplaced)
@@
     (pin "1")
   )
+  (symbol (lib_id "Device:L_Small") (at 342.9 52.07 90) (unit 1)
+    (in_bom yes) (on_board yes) (fields_autoplaced)
+    (property "Reference" "L2" (id 0) (at 342.9 46.99 90))
+    (property "Value" "4u7" (id 1) (at 342.9 49.53 90))
+    (property "Footprint" "Z_mycustom_footprint_lib:Inductor_2.5x2x1.2mm" (id 2) (at 342.9 52.07 0)
+      (effects (font (size 1.27 1.27)) hide)
+    )
+    (property "Datasheet" "~" (id 3) (at 342.9 52.07 0)
+      (effects (font (size 1.27 1.27)) hide)
+    )
+    (property "LCSC" "C3002553" (id 4) (at 342.9 52.07 90)
+      (effects (font (size 1.27 1.27)) hide)
+    )
+    (pin "1")
+    (pin "2")
+  )
   (symbol (lib_id "power:GND") (at 351.79 219.71 0) (unit 1)
     (in_bom yes) (on_board yes)
@@
     (pin "2")
   )
-  (symbol (lib_id "Device:L_Small") (at 342.9 52.07 90) (unit 1)
-    (in_bom yes) (on_board yes) (fields_autoplaced)
-    (property "Reference" "L1" (id 0) (at 342.9 46.99 90))
-    (property "Value" "L_Small" (id 1) (at 342.9 49.53 90))
-    (property "Footprint" "Inductor_SMD:L_0603_1608Metric" (id 2) (at 342.9 52.07 0)
-      (effects (font (size 1.27 1.27)) hide)
-    )
-    (property "Datasheet" "~" (id 3) (at 342.9 52.07 0)
-      (effects (font (size 1.27 1.27)) hide)
-    )
-    (property "LCSC" "C13415" (id 4) (at 342.9 52.07 90)
-      (effects (font (size 1.27 1.27)) hide)
-    )
-    (pin "1")
-    (pin "2")
-  )
   (symbol (lib_id "Device:C_Small") (at 200.66 224.79 0) (mirror x) (unit 1)
     (in_bom yes) (on_board yes)
@@
     (pin "3")
   )
+  (symbol (lib_id "Device:L_Small") (at 92.71 67.31 90) (unit 1)
+    (in_bom yes) (on_board yes) (fields_autoplaced)
+    (property "Reference" "L3" (id 0) (at 92.71 62.23 90))
+    (property "Value" "4u7" (id 1) (at 92.71 64.77 90))
+    (property "Footprint" "Z_mycustom_footprint_lib:Inductor_2.5x2x1.2mm" (id 2) (at 92.71 67.31 0)
+      (effects (font (size 1.27 1.27)) hide)
+    )
+    (property "Datasheet" "~" (id 3) (at 92.71 67.31 0)
+      (effects (font (size 1.27 1.27)) hide)
+    )
+    (property "LCSC" "C3002553" (id 4) (at 92.71 67.31 90)
+      (effects (font (size 1.27 1.27)) hide)
+    )
+    (pin "1")
+    (pin "2")
+  )
   (symbol (lib_id "Connector_Generic:Conn_01x06") (at 325.12 217.17 180) (unit 1)
-    (in_bom yes) (on_board yes)
+    (in_bom no) (on_board no)
     (property "Reference" "J4" (id 0) (at 317.5 213.36 0))
     (property "Value" "Conn_01x06" (id 1) (at 317.5 215.9 0))
@@
     (pin "3")
   )
-  (symbol (lib_id "Device:L_Small") (at 92.71 59.69 90) (unit 1)
-    (in_bom yes) (on_board yes) (fields_autoplaced)
-    (property "Reference" "L2" (id 0) (at 92.71 54.61 90))
-    (property "Value" "L_Small" (id 1) (at 92.71 57.15 90))
-    (property "Footprint" "Inductor_SMD:L_0603_1608Metric" (id 2) (at 92.71 59.69 0)
-      (effects (font (size 1.27 1.27)) hide)
-    )
-    (property "Datasheet" "~" (id 3) (at 92.71 59.69 0)
-      (effects (font (size 1.27 1.27)) hide)
-    )
-    (property "LCSC" "C13415" (id 4) (at 92.71 59.69 90)
-      (effects (font (size 1.27 1.27)) hide)
-    )
-    (pin "1")
-    (pin "2")
-  )
   (symbol (lib_id "Device:C_Small") (at 107.95 71.12 0) (mirror y) (unit 1)
     (in_bom yes) (on_board yes)
@@
       (effects (font (size 1.27 1.27)) (justify left))
     )
-    (property "Footprint" "" (id 2) (at 392.43 78.74 0)
+    (property "Footprint" "TerminalBlock:TerminalBlock_bornier-4_P5.08mm" (id 2) (at 392.43 78.74 0)
       (effects (font (size 1.27 1.27)) hide)
     )

Commit message: n
Parts:
- removed C13, C14, C15, C16, C57: 10u, Capacitor_SMD:C_0805_2012Metric, symbol Device:C_Small
- removed C17: 1u, Capacitor_SMD:C_0603_1608Metric_Pad1.08x0.95mm_HandSolder, symbol Device:C_Small
- added C46, C51: 1u, Capacitor_SMD:C_0402_1005Metric, symbol Device:C_Small
- added C47, C50, C52, C60: 10u, Capacitor_SMD:C_0603_1608Metric, symbol Device:C_Small
- C18, C19, C21, C22, C39, C44, C54: footprint Capacitor_SMD:C_0805_2012Metric -> Capacitor_SMD:C_0603_1608Metric; LCSC C15850 -> C96446
- C20, C23, C35, C37, C38, C42, C45: footprint Capacitor_SMD:C_0603_1608Metric_Pad1.08x0.95mm_HandSolder -> Capacitor_SMD:C_0402_1005Metric; LCSC C15849 -> C52923
- C25, C29, C31, C41: value 1u -> 10u; footprint Capacitor_SMD:C_0603_1608Metric_Pad1.08x0.95mm_HandSolder -> Capacitor_SMD:C_0603_1608Metric; LCSC C15849 -> C96446
- C27, C32: footprint Capacitor_SMD:C_0603_1608Metric_Pad1.08x0.95mm_HandSolder -> Capacitor_SMD:C_0402_1005Metric; LCSC C53987 -> C1538
- C34, C40, C43: value 10u -> 1u; footprint Capacitor_SMD:C_0805_2012Metric -> Capacitor_SMD:C_0402_1005Metric; LCSC C15850 -> C52923
- R32, R33, R34, R35, R41: footprint Resistor_SMD:R_0603_1608Metric_Pad0.98x0.95mm_HandSolder -> Resistor_SMD:R_0402_1005Metric; LCSC C4190 -> C25879
Connections:
- net +3V3: now also C25.1, R34.1; no longer C18.1, C19.1, R41.1
- net +5V: now also C52.1
- net 3V33: now also C29.1, C31.1, C34.2, C43.1, C44.1, C45.2; no longer C21.1, C22.1, C23.2, C38.2, C40.1, C41.2
- net GND: now also C25.2, C29.2, C31.2, C34.1, C37.1, C40.1, C41.2, RV1.3, RV2.1, C46.2, C47.2, C50.2, C51.1, C52.2, C60.2; no longer C23.1, C29.1, C34.2, C35.1, C38.1, C40.2, C41.1, C42.1, RV1.1, RV2.3
- net Jack_MIC_INPUT_1: now also R34.2; no longer R41.2
- net L_out1: now also R35.1; no longer R34.2
- net R_out1: now also R33.1; no longer R33.2
- net Tranceiver_Audio_OUT_1: now also RV1.1; no longer RV1.3
- net Tranceiver_Audio_OUT_2: now also RV2.3; no longer RV2.1
- net at U5.10 (VREF): now also C41.1; no longer C34.1
- net Power_amp_Vcc_intermediate: now reaches JP1.2 (C), L2.1
- net Power_amp_Vcc_intermediate: now also C18.1
- net Power_amp_Vcc: now reaches L2.2, U6.13 (PVDD), U6.3 (PVDD), U6.9 (AVDD)
- net Power_amp_Vcc: now also C19.1, C21.1, C22.1, C60.1
- net at R32.1: now also C23.2
- net at C27.1, R32.2: now also C35.1, R33.2; no longer C25.1, R33.1
- net at C35.2: now also U6.19 (INL-); no longer U6.18 (INR+)
- net at J5.3 (Pin_3): now also U6.14 (OUTR+); no longer U6.16 (OUTR+)
- net at U6.17 (INR-): now also C38.2; no longer C31.2
- net at J5.4 (Pin_4): now also U6.11 (OUTR-); no longer U6.17 (OUTR-)
- net at U6.20 (INL+): now also C37.2; no longer C29.2
- net at RV1.2: now also C23.1
- net at R35.2: now also C32.1, C38.1, R41.1; no longer C37.2
- net at RV2.2: now also C42.2; no longer C37.1
- new net: C42.1, R41.2
- new net: C46.1, C47.1, U5.19 (ADCVREF)
- new net: C40.2, U6.16 (INR+)
- new net: C50.1, C51.2, U5.20 (VMID)
Other:
- moved on the sheet: C20, RV1, RV2

Commit message: b
Parts:
- removed J5: Conn_01x04, TerminalBlock:TerminalBlock_bornier-4_P5.08mm, symbol Connector_Generic:Conn_01x04
- added J3, J5: Screw_Terminal_01x02, TerminalBlock_Altech:Altech_AK300_1x02_P5.00mm_45-Degree, symbol Connector:Screw_Terminal_01x02
- added R44, R45: 10k, Resistor_SMD:R_0603_1608Metric_Pad0.98x0.95mm_HandSolder, symbol Device:R_Small
Connections:
- net GND: now also R44.1, R45.2
- net H/L1: now also R44.2
- net H/L2: now also R45.1
- net at U6.11 (OUTR-): now also J5.1 (Pin_1)
- net at U6.14 (OUTR+): now also J5.2 (Pin_2)
- net at U6.2 (OUTL+): now also J3.1 (Pin_1)
- net at U6.5 (OUTL-): now also J3.2 (Pin_2)
Changed lines of the file:
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@@
   (junction (at 331.47 71.12) (diameter 0) (color 0 0 0 0)
   )
+  (junction (at 168.91 269.24) (diameter 0) (color 0 0 0 0)
+  )
   (junction (at 361.95 104.14) (diameter 0) (color 0 0 0 0)
   )
@@
     (stroke (width 0) (type default) (color 0 0 0 0))
   )
+  (wire (pts (xy 171.45 261.62) (xy 171.45 262.89))
+    (stroke (width 0) (type default) (color 0 0 0 0))
+  )
   (wire (pts (xy 106.68 124.46) (xy 111.76 124.46))
     (stroke (width 0) (type default) (color 0 0 0 0))
@@
     (stroke (width 0) (type default) (color 0 0 0 0))
   )
+  (wire (pts (xy 171.45 267.97) (xy 171.45 269.24))
+    (stroke (width 0) (type default) (color 0 0 0 0))
+  )
   (wire (pts (xy 177.8 72.39) (xy 184.15 72.39))
     (stroke (width 0) (type default) (color 0 0 0 0))
@@
     (stroke (width 0) (type default) (color 0 0 0 0))
   )
-  (wire (pts (xy 375.92 85.09) (xy 375.92 81.28))
-    (stroke (width 0) (type default) (color 0 0 0 0))
-  )
   (wire (pts (xy 347.98 214.63) (xy 330.2 214.63))
     (stroke (width 0) (type default) (color 0 0 0 0))
@@
     (stroke (width 0) (type default) (color 0 0 0 0))
   )
-  (wire (pts (xy 387.35 83.82) (xy 387.35 90.17))
+  (wire (pts (xy 387.35 87.63) (xy 387.35 90.17))
     (stroke (width 0) (type default) (color 0 0 0 0))
   )
@@
     (stroke (width 0) (type default) (color 0 0 0 0))
   )
+  (wire (pts (xy 168.91 269.24) (xy 168.91 270.51))
+    (stroke (width 0) (type default) (color 0 0 0 0))
+  )
   (wire (pts (xy 182.88 95.25) (xy 182.88 96.52))
     (stroke (width 0) (type default) (color 0 0 0 0))
@@
     (stroke (width 0) (type default) (color 0 0 0 0))
   )
-  (wire (pts (xy 374.65 85.09) (xy 375.92 85.09))
+  (wire (pts (xy 374.65 85.09) (xy 387.35 85.09))
     (stroke (width 0) (type default) (color 0 0 0 0))
   )
@@
     (stroke (width 0) (type default) (color 0 0 0 0))
   )
+  (wire (pts (xy 168.91 261.62) (xy 168.91 262.89))
+    (stroke (width 0) (type default) (color 0 0 0 0))
+  )
   (wire (pts (xy 336.55 59.69) (xy 336.55 60.96))
     (stroke (width 0) (type default) (color 0 0 0 0))
@@
     (stroke (width 0) (type default) (color 0 0 0 0))
   )
+  (wire (pts (xy 168.91 267.97) (xy 168.91 269.24))
+    (stroke (width 0) (type default) (color 0 0 0 0))
+  )
   (wire (pts (xy 142.24 77.47) (xy 143.51 77.47))
     (stroke (width 0) (type default) (color 0 0 0 0))
@@
     (stroke (width 0) (type default) (color 0 0 0 0))
   )
-  (wire (pts (xy 375.92 81.28) (xy 387.35 81.28))
-    (stroke (width 0) (type default) (color 0 0 0 0))
-  )
   (wire (pts (xy 336.55 52.07) (xy 340.36 52.07))
     (stroke (width 0) (type default) (color 0 0 0 0))
@@
     (stroke (width 0) (type default) (color 0 0 0 0))
   )
+  (wire (pts (xy 171.45 269.24) (xy 168.91 269.24))
+    (stroke (width 0) (type default) (color 0 0 0 0))
+  )
   (wire (pts (xy 198.12 92.71) (xy 198.12 96.52))
     (stroke (width 0) (type default) (color 0 0 0 0))
@@
     )
   )
+  (global_label "H{slash}L1" (shape input) (at 168.91 261.62 90) (fields_autoplaced)
+    (effects (font (size 1.27 1.27)) (justify left))
+    (property "Intersheet References" "${INTERSHEET_REFS}" (id 0) (at 168.8306 254.3083 90)
+      (effects (font (size 1.27 1.27)) (justify left) hide)
+    )
+  )
   (global_label "G0" (shape input) (at 377.19 95.25 0) (fields_autoplaced)
     (effects (font (size 1.27 1.27)) (justify left))
@@
     )
   )
+  (global_label "H{slash}L2" (shape input) (at 171.45 261.62 90) (fields_autoplaced)
+    (effects (font (size 1.27 1.27)) (justify left))
+    (property "Intersheet References" "${INTERSHEET_REFS}" (id 0) (at 171.3706 254.3083 90)
+      (effects (font (size 1.27 1.27)) (justify left) hide)
+    )
+  )
   (global_label "AMP_R" (shape input) (at 342.9 95.25 180) (fields_autoplaced)
     (effects (font (size 1.27 1.27)) (justify right))
@@
     (pin "1")
   )
+  (symbol (lib_id "Connector:Screw_Terminal_01x02") (at 392.43 76.2 0) (unit 1)
+    (in_bom yes) (on_board yes) (fields_autoplaced)
+    (property "Reference" "J3" (id 0) (at 394.97 76.1999 0)
+      (effects (font (size 1.27 1.27)) (justify left))
+    )
+    (property "Value" "Screw_Terminal_01x02" (id 1) (at 394.97 78.7399 0)
+      (effects (font (size 1.27 1.27)) (justify left))
+    )
+    (property "Footprint" "TerminalBlock_Altech:Altech_AK300_1x02_P5.00mm_45-Degree" (id 2) (at 392.43 76.2 0)
+      (effects (font (size 1.27 1.27)) hide)
+    )
+    (property "Datasheet" "~" (id 3) (at 392.43 76.2 0)
+      (effects (font (size 1.27 1.27)) hide)
+    )
+    (pin "1")
+    (pin "2")
+  )
   (symbol (lib_id "Device:C_Small") (at 349.25 57.15 0) (mirror y) (unit 1)
     (in_bom yes) (on_board yes)
@@
     (pin "1")
   )
+  (symbol (lib_id "power:GND") (at 168.91 270.51 0) (mirror y) (unit 1)
+    (in_bom yes) (on_board yes) (fields_autoplaced)
+    (property "Reference" "#PWR0114" (id 0) (at 168.91 276.86 0)
+      (effects (font (size 1.27 1.27)) hide)
+    )
+    (property "Value" "GND" (id 1) (at 168.91 275.59 0)
+      (effects (font (size 1.27 1.27)) hide)
+    )
+    (property "Footprint" "" (id 2) (at 168.91 270.51 0)
+      (effects (font (size 1.27 1.27)) hide)
+    )
+    (property "Datasheet" "" (id 3) (at 168.91 270.51 0)
+      (effects (font (size 1.27 1.27)) hide)
+    )
+    (pin "1")
+  )
   (symbol (lib_id "Device:C_Small") (at 383.54 57.15 0) (mirror y) (unit 1)
     (in_bom yes) (on_board yes)
@@
     (pin "9")
   )
+  (symbol (lib_id "Connector:Screw_Terminal_01x02") (at 392.43 87.63 0) (mirror x) (unit 1)
+    (in_bom yes) (on_board yes)
+    (property "Reference" "J5" (id 0) (at 396.24 85.09 0))
+    (property "Value" "Screw_Terminal_01x02" (id 1) (at 405.13 87.63 0))
+    (property "Footprint" "TerminalBlock_Altech:Altech_AK300_1x02_P5.00mm_45-Degree" (id 2) (at 392.43 87.63 0)
+      (effects (font (size 1.27 1.27)) hide)
+    )
+    (property "Datasheet" "~" (id 3) (at 392.43 87.63 0)
+      (effects (font (size 1.27 1.27)) hide)
+    )
+    (pin "1")
+    (pin "2")
+  )
   (symbol (lib_id "Device:C_Small") (at 83.82 71.12 0) (mirror y) (unit 1)
     (in_bom yes) (on_board yes)
@@
     (pin "2")
   )
+  (symbol (lib_id "Device:R_Small") (at 168.91 265.43 0) (mirror x) (unit 1)
+    (in_bom yes) (on_board yes) (fields_autoplaced)
+    (property "Reference" "R44" (id 0) (at 166.37 264.1599 0)
+      (effects (font (size 1.27 1.27)) (justify right))
+    )
+    (property "Value" "10k" (id 1) (at 166.37 266.6999 0)
+      (effects (font (size 1.27 1.27)) (justify right))
+    )
+    (property "Footprint" "Resistor_SMD:R_0603_1608Metric_Pad0.98x0.95mm_HandSolder" (id 2) (at 168.91 265.43 0)
+      (effects (font (size 1.27 1.27)) hide)
+    )
+    (property "Datasheet" "~" (id 3) (at 168.91 265.43 0)
+      (effects (font (size 1.27 1.27)) hide)
+    )
+    (property "LCSC" "C25804" (id 4) (at 168.91 265.43 90)
+      (effects (font (size 1.27 1.27)) hide)
+    )
+    (pin "1")
+    (pin "2")
+  )
   (symbol (lib_id "power:GND") (at 154.94 273.05 0) (unit 1)
     (in_bom yes) (on_board yes) (fields_autoplaced)
@@
     (pin "3")
   )
+  (symbol (lib_id "Device:R_Small") (at 171.45 265.43 0) (unit 1)
+    (in_bom yes) (on_board yes) (fields_autoplaced)
+    (property "Reference" "R45" (id 0) (at 173.99 264.1599 0)
+      (effects (font (size 1.27 1.27)) (justify left))
+    )
+    (property "Value" "10k" (id 1) (at 173.99 266.6999 0)
+      (effects (font (size 1.27 1.27)) (justify left))
+    )
+    (property "Footprint" "Resistor_SMD:R_0603_1608Metric_Pad0.98x0.95mm_HandSolder" (id 2) (at 171.45 265.43 0)
+      (effects (font (size 1.27 1.27)) hide)
+    )
+    (property "Datasheet" "~" (id 3) (at 171.45 265.43 0)
+      (effects (font (size 1.27 1.27)) hide)
+    )
+    (property "LCSC" "C25804" (id 4) (at 171.45 265.43 90)
+      (effects (font (size 1.27 1.27)) hide)
+    )
+    (pin "1")
+    (pin "2")
+  )
   (symbol (lib_id "power:GND") (at 233.68 102.87 0) (mirror y) (unit 1)
     (in_bom yes) (on_board yes) (fields_autoplaced)
@@
     (pin "1")
   )
-  (symbol (lib_id "Connector_Generic:Conn_01x04") (at 392.43 78.74 0) (unit 1)
-    (in_bom yes) (on_board yes) (fields_autoplaced)
-    (property "Reference" "J5" (id 0) (at 394.97 78.7399 0)
-      (effects (font (size 1.27 1.27)) (justify left))
-    )
-    (property "Value" "Conn_01x04" (id 1) (at 394.97 81.2799 0)
-      (effects (font (size 1.27 1.27)) (justify left))
-    )
-    (property "Footprint" "TerminalBlock:TerminalBlock_bornier-4_P5.08mm" (id 2) (at 392.43 78.74 0)
-      (effects (font (size 1.27 1.27)) hide)
-    )
-    (property "Datasheet" "~" (id 3) (at 392.43 78.74 0)
-      (effects (font (size 1.27 1.27)) hide)
-    )
-    (pin "1")
-    (pin "2")
-    (pin "3")
-    (pin "4")
-  )
 )

Commit message: f
Connections:
- net GND: now also RV1.1, RV2.3, RV3.1, RV4.3; no longer RV1.3, RV2.1, RV3.3, RV4.1
- net Tranceiver_Audio_OUT_1: now also RV1.3, RV4.1; no longer RV1.1, RV4.3
- net Tranceiver_Audio_OUT_2: now also RV2.1, RV3.3; no longer RV2.3, RV3.1
Other:
- moved on the sheet: C18, C19, C20, C21, C22, C23, C24, C25, C26, C27, C28, C29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
