File: HW/cross_band_handy_walkie_talkie_ES8388/Audio_Codec.kicad_sch (KiCad schematic)
At the start: 73 parts, among them J3 Screw_Terminal_01x02, J4 Conn_01x06, J5 Screw_Terminal_01x02, J6 AudioJack4_SwitchTR1, J7 SMA, J8 SMA, U5 ES8388, U6 TPA2012D2, U7 SA818S, U8 SA818S

Commit message: f
Parts:
- R38, R39: footprint Resistor_SMD:R_0805_2012Metric -> Resistor_SMD:R_0603_1608Metric; LCSC C17513 -> C21190
Changed lines of the file:
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@@
       (effects (font (size 1.27 1.27)) (justify left))
     )
-    (property "Footprint" "Resistor_SMD:R_0805_2012Metric" (id 2) (at 153.162 266.7 90)
+    (property "Footprint" "Resistor_SMD:R_0603_1608Metric" (id 2) (at 153.162 266.7 90)
       (effects (font (size 1.27 1.27)) hide)
     )
@@
       (effects (font (size 1.27 1.27)) hide)
     )
-    (property "LCSC" "C17513" (id 4) (at 154.94 266.7 0)
+    (property "LCSC" "C21190" (id 4) (at 154.94 266.7 0)
       (effects (font (size 1.27 1.27)) hide)
     )
@@
       (effects (font (size 1.27 1.27)) (justify left))
     )
-    (property "Footprint" "Resistor_SMD:R_0805_2012Metric" (id 2) (at 144.272 266.7 90)
+    (property "Footprint" "Resistor_SMD:R_0603_1608Metric" (id 2) (at 144.272 266.7 90)
       (effects (font (size 1.27 1.27)) hide)
     )
@@
       (effects (font (size 1.27 1.27)) hide)
     )
-    (property "LCSC" "C17513" (id 4) (at 146.05 266.7 0)
-      (effects (font (size 1.27 1.27)) hide)
-    )
+    (property "LCSC" "C21190" (id 4) (at 146.05 266.7 0)
+      (effects (font (size 1.27 1.27)) hide)
+    )

Commit message: e
Connections:
- net LINE_IN1: now also C28.2; no longer C24.2
- net LINE_IN2: now also C24.2; no longer C28.2
- net A_audio_4: now reaches C30.1, U5.21 (RIN2)
- net A_audio_3: now reaches C28.1, U5.22 (LIN2)
- net R_out1_: now reaches C33.2, U5.11 (ROUT1)
- net L_out1_: now reaches C36.2, U5.12 (LOUT1)
- net A_audio_2: now reaches C26.1, U5.23 (RIN1)
- net A_audio_1: now reaches C24.1, U5.24 (LIN1)
Changed lines of the file:
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@@
     (effects (font (size 1.27 1.27)) (justify right bottom))
+  )
+  (label "R_out1_" (at 105.41 69.85 0)
+    (effects (font (size 0.2 0.2)) (justify left bottom))
+  )
+  (label "A_audio_3" (at 142.24 59.69 0)
+    (effects (font (size 0.2 0.2)) (justify left bottom))
+  )
+  (label "L_out1_" (at 105.41 72.39 0)
+    (effects (font (size 0.2 0.2)) (justify left bottom))
   )
   (label "Power_amp_Vcc_intermediate" (at 307.975 48.895 180)
     (effects (font (size 0.4 0.4)) (justify right bottom))
   )
+  (label "A_audio_2" (at 142.24 57.15 0)
+    (effects (font (size 0.2 0.2)) (justify left bottom))
+  )
   (label "Jack_MIC_INPUT_1" (at 162.56 55.88 0)
     (effects (font (size 1.27 1.27)) (justify left bottom))
@@
     (effects (font (size 1.27 1.27)) (justify left bottom))
   )
+  (label "A_audio_4" (at 142.24 62.23 0)
+    (effects (font (size 0.2 0.2)) (justify left bottom))
+  )
   (label "MIC_INPUT_2" (at 162.56 63.5 0)
     (effects (font (size 1.27 1.27)) (justify left bottom))
@@
     (effects (font (size 1.27 1.27)) (justify left bottom))
   )
+  (label "A_audio_1" (at 142.24 54.61 0)
+    (effects (font (size 0.2 0.2)) (justify left bottom))
+  )
   (global_label "LINE_IN1" (shape input) (at 290.83 147.955 0) (fields_autoplaced)
     (effects (font (size 1.27 1.27)) (justify left))
@@
     )
   )
-  (global_label "LINE_IN1" (shape input) (at 162.56 52.07 0) (fields_autoplaced)
-    (effects (font (size 1.27 1.27)) (justify left))
-    (property "Intersheet References" "${INTERSHEET_REFS}" (id 0) (at 173.1979 51.9906 0)
+  (global_label "LINE_IN1" (shape input) (at 162.56 59.69 0) (fields_autoplaced)
+    (effects (font (size 1.27 1.27)) (justify left))
+    (property "Intersheet References" "${INTERSHEET_REFS}" (id 0) (at 173.1979 59.6106 0)
       (effects (font (size 1.27 1.27)) (justify left) hide)
     )
@@
     )
   )
-  (global_label "LINE_IN2" (shape input) (at 162.56 59.69 0) (fields_autoplaced)
-    (effects (font (size 1.27 1.27)) (justify left))
-    (property "Intersheet References" "${INTERSHEET_REFS}" (id 0) (at 173.1979 59.6106 0)
-      (effects (font (size 1.27 1.27)) (justify left) hide)
-    )
+  (global_label "LINE_IN2" (shape input) (at 162.56 52.07 0) (fields_autoplaced)
+    (effects (font (size 1.27 1.27)) (justify left))
+    (property "Intersheet References" "${INTERSHEET_REFS}" (id 0) (at 173.1979 51.9906 0)
+      (effects (font (size 1.27 1.27)) (justify left) hide)
+    )

Commit message: r
Parts:
- removed R45: 10k, Resistor_SMD:R_0603_1608Metric_Pad0.98x0.95mm_HandSolder, symbol Device:R_Small
- added C63: 22u, Capacitor_SMD:C_0805_2012Metric, symbol Device:C_Small
Connections:
- net EXT_SPEAKER+ is gone; now on net MIC_INPUT_2: J4.3 (Pin_3)
- net H/L2 is gone; now on net H/L1: U7.7 (H/L)
- net Speaker_L+: now reaches J3.1 (Pin_1), U6.2 (OUTL+)
- net Speaker_L+: now also C63.2
- net Speaker_L-: now reaches J3.2 (Pin_2), U6.5 (OUTL-)
- net Speaker_R-: now reaches J5.1 (Pin_1), U6.11 (OUTR-)
- net Speaker_R+: now reaches J5.2 (Pin_2), U6.14 (OUTR+)
- net MIC-AMP_IN renamed PTT3
- net MIC_EST_PTT: no longer names the net of J4.4 (Pin_4)
- net MIC_EST_PTT: now also C63.1
Other:
- moved on the sheet: C18, C19, C21, C22, C23, C27, C32, C35, C37, C38, C40, C42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

Commit message: y
Parts:
- removed C49: 1u, Capacitor_SMD:C_0603_1608Metric_Pad1.08x0.95mm_HandSolder, symbol Device:C_Small
- added TP3: TestPoint, TestPoint:TestPoint_Pad_1.0x1.0mm, symbol Connector:TestPoint
Connections:
- net at C48.1, J6.R1: now also J6.T
- net at U5.15 (LOUT2): now also TP3.1
- no-connect marks 2 -> 4
Other:
- title: (none) -> Cross band handy walkie talkie V2
Changed lines of the file:
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@@
 (kicad_sch (version 20211123) (generator eeschema)
   (paper "A3")
+  (title_block
+    (title "Cross band handy walkie talkie V2")
+    (date "2023-03-19")
+    (comment 1 "Author: Kecs Robert Alfred")
+    (comment 2 "Reviewed by: Andreas Spiess")
+  )
   (junction (at 303.53 91.44) (diameter 0) (color 0 0 0 0)
   )
@@
   (junction (at 347.98 53.34) (diameter 0) (color 0 0 0 0)
   )
+  (junction (at 93.98 109.22) (diameter 0) (color 0 0 0 0)
+  )
   (junction (at 303.53 83.82) (diameter 0) (color 0 0 0 0)
   )
   (junction (at 298.45 72.39) (diameter 0) (color 0 0 0 0)
   )
+  (junction (at 116.84 114.3) (diameter 0) (color 0 0 0 0)
+  )
   (junction (at 185.42 67.31) (diameter 0) (color 0 0 0 0)
   )
@@
   )
   (no_connect (at 110.49 64.77))
+  (no_connect (at 101.6 114.3))
+  (no_connect (at 73.66 111.76))
   (no_connect (at 140.97 52.07))
   (wire (pts (xy 321.31 53.34) (xy 321.31 55.88))
@@
     (stroke (width 0) (type default) (color 0 0 0 0))
   )
+  (wire (pts (xy 116.84 114.3) (xy 143.51 114.3))
+    (stroke (width 0) (type default) (color 0 0 0 0))
+  )
   (wire (pts (xy 67.31 67.31) (xy 110.49 67.31))
     (stroke (width 0) (type default) (color 0 0 0 0))
@@
     (stroke (width 0) (type default) (color 0 0 0 0))
   )
-  (wire (pts (xy 73.66 109.22) (xy 96.52 109.22))
+  (wire (pts (xy 73.66 109.22) (xy 93.98 109.22))
     (stroke (width 0) (type default) (color 0 0 0 0))
   )
@@
     (stroke (width 0) (type default) (color 0 0 0 0))
   )
+  (wire (pts (xy 93.98 109.22) (xy 93.98 114.3))
+    (stroke (width 0) (type default) (color 0 0 0 0))
+  )
   (wire (pts (xy 355.6 60.96) (xy 355.6 62.23))
     (stroke (width 0) (type default) (color 0 0 0 0))
@@
     (stroke (width 0) (type default) (color 0 0 0 0))
   )
-  (wire (pts (xy 73.66 114.3) (xy 96.52 114.3))
+  (wire (pts (xy 73.66 114.3) (xy 93.98 114.3))
     (stroke (width 0) (type default) (color 0 0 0 0))
   )
@@
     (stroke (width 0) (type default) (color 0 0 0 0))
   )
-  (wire (pts (xy 101.6 114.3) (xy 143.51 114.3))
+  (wire (pts (xy 101.6 114.3) (xy 116.84 114.3))
     (stroke (width 0) (type default) (color 0 0 0 0))
   )
@@
     (stroke (width 0) (type default) (color 0 0 0 0))
   )
+  (wire (pts (xy 116.84 111.76) (xy 116.84 114.3))
+    (stroke (width 0) (type default) (color 0 0 0 0))
+  )
   (wire (pts (xy 317.5 72.39) (xy 314.96 72.39))
     (stroke (width 0) (type default) (color 0 0 0 0))
@@
   )
   (wire (pts (xy 292.1 92.71) (xy 292.1 95.25))
+    (stroke (width 0) (type default) (color 0 0 0 0))
+  )
+  (wire (pts (xy 93.98 109.22) (xy 96.52 109.22))
     (stroke (width 0) (type default) (color 0 0 0 0))
   )
@@
     (pin "2")
   )
-  (symbol (lib_id "Device:C_Small") (at 99.06 114.3 90) (mirror x) (unit 1)
-    (in_bom yes) (on_board yes)
-    (property "Reference" "C49" (id 0) (at 97.79 116.84 90)
-      (effects (font (size 1.27 1.27)) (justify left))
-    )
-    (property "Value" "1u" (id 1) (at 102.87 116.84 90)
-      (effects (font (size 1.27 1.27)) (justify left))
-    )
-    (property "Footprint" "Capacitor_SMD:C_0603_1608Metric_Pad1.08x0.95mm_HandSolder" (id 2) (at 99.06 114.3 0)
-      (effects (font (size 1.27 1.27)) hide)
-    )
-    (property "Datasheet" "https://jlcpcb.com/partdetail/16531-CL10A105KB8NNNC/C15849" (id 3) (at 99.06 114.3 0)
-      (effects (font (size 1.27 1.27)) hide)
-    )
-    (property "LCSC" "C15849" (id 4) (at 99.06 114.3 0)
-      (effects (font (size 1.27 1.27)) hide)
-    )
-    (pin "1")
-    (pin "2")
-  )
   (symbol (lib_id "Device:C_Small") (at 165.1 78.74 0) (mirror y) (unit 1)
     (in_bom yes) (on_board yes)
@@
     (pin "2")
   )
+  (symbol (lib_id "Connector:TestPoint") (at 116.84 111.76 0) (unit 1)
+    (in_bom no) (on_board yes) (fields_autoplaced)
+    (property "Reference" "TP3" (id 0) (at 119.38 108.4579 0)
+      (effects (font (size 1.27 1.27)) (justify left))
+    )
+    (property "Value" "TestPoint" (id 1) (at 120.65 109.7279 0)
+      (effects (font (size 1.27 1.27)) (justify left) hide)
+    )
+    (property "Footprint" "TestPoint:TestPoint_Pad_1.0x1.0mm" (id 2) (at 121.92 111.76 0)
+      (effects (font (size 1.27 1.27)) hide)
+    )
+    (property "Datasheet" "~" (id 3) (at 121.92 111.76 0)
+      (effects (font (size 1.27 1.27)) hide)
+    )
+    (pin "1")
+  )
   (symbol (lib_id "Device:R_Small") (at 168.91 265.43 0) (mirror x) (unit 1)

Commit message: b
Parts:
- added TP8: TestPoint, TestPoint:TestPoint_Pad_1.0x1.0mm, symbol Connector:TestPoint
Connections:
- net at C48.2, U5.14 (ROUT2): now also TP8.1
Changed lines of the file:
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@@
   (junction (at 165.1 72.39) (diameter 0) (color 0 0 0 0)
+  )
+  (junction (at 109.22 102.87) (diameter 0) (color 0 0 0 0)
   )
   (junction (at 303.53 72.39) (diameter 0) (color 0 0 0 0)
@@
     (stroke (width 0) (type default) (color 0 0 0 0))
   )
+  (wire (pts (xy 114.3 102.87) (xy 109.22 102.87))
+    (stroke (width 0) (type default) (color 0 0 0 0))
+  )
   (wire (pts (xy 317.5 72.39) (xy 314.96 72.39))
     (stroke (width 0) (type default) (color 0 0 0 0))
@@
     (stroke (width 0) (type default) (color 0 0 0 0))
   )
-  (wire (pts (xy 109.22 77.47) (xy 109.22 109.22))
+  (wire (pts (xy 109.22 77.47) (xy 109.22 102.87))
     (stroke (width 0) (type default) (color 0 0 0 0))
   )
@@
   )
   (wire (pts (xy 67.31 67.31) (xy 67.31 68.58))
+    (stroke (width 0) (type default) (color 0 0 0 0))
+  )
+  (wire (pts (xy 109.22 102.87) (xy 109.22 109.22))
     (stroke (width 0) (type default) (color 0 0 0 0))
   )
@@
       (effects (font (size 1.27 1.27)) hide)
     )
+    (pin "1")
+  )
+  (symbol (lib_id "Connector:TestPoint") (at 114.3 102.87 270) (unit 1)
+    (in_bom no) (on_board yes) (fields_autoplaced)
+    (property "Reference" "TP8" (id 0) (at 120.65 102.8699 90)
+      (effects (font (size 1.27 1.27)) (justify left))
+    )
+    (property "Value" "TestPoint" (id 1) (at 116.3321 106.68 0)
+      (effects (font (size 1.27 1.27)) (justify left) hide)
+    )
+    (property "Footprint" "TestPoint:TestPoint_Pad_1.0x1.0mm" (id 2) (at 114.3 107.95 0)
+      (effects (font (size 1.27 1.27)) hide)
+    )
+    (property "Datasheet" "~" (id 3) (at 114.3 107.95 0)
+      (effects (font (size 1.27 1.27)) hide)
+    )

Commit message: b
Parts:
- removed R44: 10k, Resistor_SMD:R_0603_1608Metric_Pad0.98x0.95mm_HandSolder, symbol Device:R_Small
- added JP4: 3p, Jumper:SolderJumper-3_P1.3mm_Bridged12_Pad1.0x1.5mm, symbol Jumper:Jumper_3_Bridged12
- added Q5: nMOS, Package_TO_SOT_SMD:SOT-23, symbol Device:Q_NMOS_GSD
- added R44: 1k, Resistor_SMD:R_0603_1608Metric, symbol Device:R
- added R51: 10k, Resistor_SMD:R_0603_1608Metric_Pad0.98x0.95mm_HandSolder, symbol Device:R_Small
Connections:
- net +3V3: now also JP4.1 (A), R51.2
- net +5V: now also JP4.3 (B); no longer C52.1, C54.1, C55.2, C56.1, U7.8 (VBATT), U8.8 (VBATT)
- net GND: now also Q5.2 (S)
- net H/L1: now also R44.1
- new net: Q5.3 (D), R44.2
- new net RF_TX_power_set: Q5.1 (G), R51.1
- new net RF_power_buss: C52.1, C54.1, C55.2, C56.1, JP4.2 (C), U7.8 (VBATT), U8.8 (VBATT)
- no-connect marks 4 -> 3
Other:
- note added: "AUDIO CODEC"
- note added: "Audio POWER Amplifier"
- moved on the sheet: C18, C19, C21, C22, C23, C27, C32, C35, C37, C38, C40, C42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

Commit message: f
Connections:
- net RF_power_buss renamed RF_power_bus
Changed lines of the file:
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@@
   (junction (at 345.44 77.47) (diameter 0) (color 0 0 0 0)
+  )
+  (junction (at 86.36 223.52) (diameter 0) (color 0 0 0 0)
   )
   (junction (at 142.24 218.44) (diameter 0) (color 0 0 0 0)
@@
     (stroke (width 0) (type default) (color 0 0 0 0))
   )
+  (wire (pts (xy 86.36 223.52) (xy 90.17 223.52))
+    (stroke (width 0) (type default) (color 0 0 0 0))
+  )
   (wire (pts (xy 189.23 81.28) (xy 189.23 82.55))
     (stroke (width 0) (type default) (color 0 0 0 0))
@@
     (stroke (width 0) (type default) (color 0 0 0 0))
   )
-  (wire (pts (xy 86.36 226.06) (xy 86.36 223.52))
-    (stroke (width 0) (type default) (color 0 0 0 0))
-  )
   (polyline (pts (xy 24.13 20.32) (xy 24.13 118.11))
     (stroke (width 0) (type default) (color 0 0 0 0))
@@
   )
   (polyline (pts (xy 238.76 27.94) (xy 238.76 137.16))
+    (stroke (width 0) (type default) (color 0 0 0 0))
+  )
+  (wire (pts (xy 86.36 223.52) (xy 86.36 226.06))
     (stroke (width 0) (type default) (color 0 0 0 0))
   )
@@
     )
   )
-  (global_label "RF_power_buss" (shape input) (at 208.28 218.44 180) (fields_autoplaced)
+  (global_label "RF_power_bus" (shape input) (at 208.28 218.44 180) (fields_autoplaced)
     (effects (font (size 1.27 1.27)) (justify right))
-    (property "Intersheet References" "${INTERSHEET_REFS}" (id 0) (at 191.7155 218.5194 0)
+    (property "Intersheet References" "${INTERSHEET_REFS}" (id 0) (at 192.7436 218.3606 0)
       (effects (font (size 1.27 1.27)) (justify right) hide)
     )
@@
     )
   )
-  (global_label "RF_power_buss" (shape input) (at 86.36 223.52 0) (fields_autoplaced)
-    (effects (font (size 1.27 1.27)) (justify left))
-    (property "Intersheet References" "${INTERSHEET_REFS}" (id 0) (at 102.9245 223.4406 0)
-      (effects (font (size 1.27 1.27)) (justify left) hide)
-    )
+  (global_label "RF_power_bus" (shape input) (at 90.17 223.52 0) (fields_autoplaced)
+    (effects (font (size 1.27 1.27)) (justify left))
+    (property "Intersheet References" "${INTERSHEET_REFS}" (id 0) (at 105.7064 223.4406 0)
+      (effects (font (size 1.27 1.27)) (justify left) hide)
+    )

Commit message: b
Parts:
- L2, L3: LCSC C3002553 -> C602016
Changed lines of the file:
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@@
       (effects (font (size 1.27 1.27)) hide)
     )
-    (property "LCSC" "C3002553" (id 4) (at 327.66 63.5 90)
+    (property "LCSC" "C602016" (id 4) (at 327.66 63.5 90)
       (effects (font (size 1.27 1.27)) hide)
     )
@@
       (effects (font (size 1.27 1.27)) hide)
     )
-    (property "LCSC" "C3002553" (id 4) (at 59.69 46.99 90)
-      (effects (font (size 1.27 1.27)) hide)
-    )
+    (property "LCSC" "C602016" (id 4) (at 59.69 46.99 90)
+      (effects (font (size 1.27 1.27)) hide)
+    )
