File: HW/cross_band_handy_walkie_talkie_ES8388/Audio_Codec.kicad_sch (KiCad schematic)
At the start: 77 parts, among them J3 Screw_Terminal_01x02, J4 Conn_01x06, J5 Screw_Terminal_01x02, J6 AudioJack4_SwitchTR1, J7 SMA, J8 SMA, Q5 nMOS, U5 ES8388, U6 TPA2012D2, U7 SA818S, U8 SA818S

Commit message: r
Parts:
- U5: footprint Package_DFN_QFN:QFN-28-1EP_4x4mm_P0.4mm_EP2.4x2.4mm_ThermalVias -> Package_DFN_QFN:QFN-28-1EP_4x4mm_P0.45mm_EP2.4x2.4mm_ThermalVias
Changed lines of the file:
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@@
       (effects (font (size 1.27 1.27)))
     )
-    (property "Footprint" "Package_DFN_QFN:QFN-28-1EP_4x4mm_P0.4mm_EP2.4x2.4mm_ThermalVias" (at 125.73 69.85 0)
+    (property "Footprint" "Package_DFN_QFN:QFN-28-1EP_4x4mm_P0.45mm_EP2.4x2.4mm_ThermalVias" (at 125.73 69.85 0)
       (effects (font (size 1.27 1.27) italic) hide)
     )
