File: HW/cross_band_handy_walkie_talkie_ES8388/cross_band_handy_walkie_talkie_ES8388.kicad_pcb (KiCad board)
At the start: 2 copper layers, 90 parts, among them J1 USB_C_Receptacle, J2 Micro_SD_Card_Det, J3 SMA, J4 SMA, J5 AudioJack4_SwitchTR1, SW1 MCU_RESET, SW2 MCU_RESET, U1 SRV05-4, U2 ESP32-S3-WROOM-1, U3 SA818S, U4 SA818S, U5 TPA2012D2, U6 ES8388

Commit message: b
Parts:
- moved C15 79.7 mm to (168.6, 110.8)
- moved C16 79.7 mm to (174.0, 99.5)
- moved C17 79.7 mm to (182.7, 98.5)
- moved C19 79.7 mm to (178.0, 104.8)
- moved C20 79.7 mm to (168.6, 113.3)
- moved C30 79.7 mm to (164.2, 111.0)
- moved J5 79.7 mm to (157.2, 97.7)
- moved JP1 79.7 mm to (159.2, 111.6)
- moved R29 79.7 mm to (158.6, 115.1)
- moved C14 79.7 mm to (163.0, 114.9)
- moved C21 79.7 mm to (188.9, 93.0)
- moved C23 79.7 mm to (180.2, 96.0)
- moved C24 79.7 mm to (167.3, 115.8)
- moved C26 79.7 mm to (184.6, 93.0)
- moved C27 79.7 mm to (184.6, 95.6)
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
Commit message: f
Parts:
- removed J5: AudioJack4_SwitchTR1, Z_mycustom_footprint_lib:PJ-316A-6A
- added BT1: Battery_Cell, Connector_PinHeader_2.54mm:PinHeader_1x02_P2.54mm_Vertical, F.Cu at (353.4, 107.5)
- added C36: 22u, Capacitor_SMD:C_0805_2012Metric, F.Cu at (356.7, 71.0)
- added C37: 1u, Capacitor_SMD:C_0603_1608Metric_Pad1.08x0.95mm_HandSolder, F.Cu at (371.3, 64.5)
- added C38: 1u, Capacitor_SMD:C_0603_1608Metric_Pad1.08x0.95mm_HandSolder, F.Cu at (386.6, 47.6)
- added C39: 10u, Capacitor_SMD:C_0805_2012Metric, F.Cu at (388.3, 36.3)
- added C40: 10u, Capacitor_SMD:C_0805_2012Metric, F.Cu at (387.9, 42.3)
- added C41: 1u, Capacitor_SMD:C_0603_1608Metric_Pad1.08x0.95mm_HandSolder, F.Cu at (397.1, 39.9)
- added C42: 1u, Capacitor_SMD:C_0603_1608Metric_Pad1.08x0.95mm_HandSolder, F.Cu at (375.6, 61.3)
- added C43: 10u, Capacitor_SMD:C_0805_2012Metric, F.Cu at (347.8, 72.6)
- added C44: 10u, Capacitor_SMD:C_0805_2012Metric, F.Cu at (383.8, 36.3)
- added C45: 1u, Capacitor_SMD:C_0603_1608Metric_Pad1.08x0.95mm_HandSolder, F.Cu at (377.5, 55.8)
- added C46: 10u, Capacitor_SMD:C_0805_2012Metric, F.Cu at (362.0, 96.9)
- added C47: 10u, Capacitor_SMD:C_0805_2012Metric, F.Cu at (358.3, 113.9)
- added C48: 1u, Capacitor_SMD:C_0603_1608Metric_Pad1.08x0.95mm_HandSolder, F.Cu at (365.5, 73.1)
- added C49: 1u, Capacitor_SMD:C_0603_1608Metric_Pad1.08x0.95mm_HandSolder, F.Cu at (382.2, 52.1)
- added C50: 10u, Capacitor_SMD:C_0805_2012Metric, F.Cu at (366.9, 101.6)
- added C51: 10u, Capacitor_SMD:C_0805_2012Metric, F.Cu at (365.1, 106.0)
- added C52: 10u, Capacitor_SMD:C_0805_2012Metric, F.Cu at (392.9, 82.0)
- added C53: 100n, Capacitor_SMD:C_0603_1608Metric_Pad1.08x0.95mm_HandSolder, F.Cu at (401.7, 78.7)
- added C54: 10u, Capacitor_SMD:C_0805_2012Metric, F.Cu at (358.1, 68.0)
- added C55: 1u, Capacitor_SMD:C_0603_1608Metric_Pad1.08x0.95mm_HandSolder, F.Cu at (366.8, 68.0)
- added C56: 1u, Capacitor_SMD:C_0603_1608Metric_Pad1.08x0.95mm_HandSolder, F.Cu at (362.5, 67.7)
- added C57: 10u, Capacitor_SMD:C_0805_2012Metric, F.Cu at (383.8, 39.3)
- added D1: green, LED_SMD:LED_0805_2012Metric, F.Cu at (369.5, 104.6)
- added D2: green, LED_SMD:LED_0805_2012Metric, F.Cu at (344.7, 119.5)
- added D3: D_Schottky, Diode_SMD:D_SMA_Handsoldering, F.Cu at (346.0, 107.5)
- added D4: green, LED_SMD:LED_0805_2012Metric, F.Cu at (371.4, 101.6)
- added D5: green, LED_SMD:LED_0805_2012Metric, F.Cu at (340.2, 119.5)
- added D6: red, LED_SMD:LED_0603_1608Metric, F.Cu at (371.2, 67.1)
- added D7: red, LED_SMD:LED_0603_1608Metric, F.Cu at (375.5, 63.8)
- added D8: D_Schottky, Diode_SMD:D_SMA_Handsoldering, F.Cu at (378.5, 79.7)
- added J6: AudioJack4_SwitchTR1, Z_mycustom_footprint_lib:PJ-316A-6A, F.Cu at (365.5, 48.6)
- added J7: SMA, Connector_Coaxial:SMA_Amphenol_901-144_Vertical, F.Cu at (374.0, 30.1)
- added J8: SMA, Connector_Coaxial:SMA_Amphenol_901-144_Vertical, F.Cu at (383.4, 30.1)
- added J9: Conn_01x03, Connector_PinHeader_2.54mm:PinHeader_1x03_P2.54mm_Vertical, F.Cu at (365.2, 88.1)
- added JP2: 3p, Jumper:SolderJumper-3_P1.3mm_Bridged12_Pad1.0x1.5mm, F.Cu at (382.8, 42.8)
- added L2: L_Small, Inductor_SMD:L_0603_1608Metric, F.Cu at (381.7, 57.1)
- added L3: L_Small, Inductor_SMD:L_0603_1608Metric, F.Cu at (390.8, 47.9)
- added L5: L_Small, Inductor_SMD:L_0603_1608Metric, F.Cu at (393.3, 87.2)
- added Q1: nMOS, Package_TO_SOT_SMD:SOT-23, F.Cu at (362.3, 102.3)
- added R32: 2k2, Resistor_SMD:R_0603_1608Metric_Pad0.98x0.95mm_HandSolder, F.Cu at (392.7, 40.4)
- added R33: 2k2, Resistor_SMD:R_0603_1608Metric_Pad0.98x0.95mm_HandSolder, F.Cu at (382.2, 54.6)
- added R34: 2k2, Resistor_SMD:R_0603_1608Metric_Pad0.98x0.95mm_HandSolder, F.Cu at (392.2, 45.4)
- added R35: 2k2, Resistor_SMD:R_0603_1608Metric_Pad0.98x0.95mm_HandSolder, F.Cu at (397.1, 37.3)
- added R36: 10k, Resistor_SMD:R_0402_1005Metric, F.Cu at (366.3, 116.6)
- added R37: 10k, Resistor_SMD:R_0603_1608Metric_Pad0.98x0.95mm_HandSolder, F.Cu at (377.5, 58.3)
- added R38: 1k, Resistor_SMD:R_0805_2012Metric, F.Cu at (401.8, 29.9)
- added R39: 1k, Resistor_SMD:R_0805_2012Metric, F.Cu at (382.2, 49.4)
- added R40: 10k, Resistor_SMD:R_0402_1005Metric, F.Cu at (390.1, 91.1)
- added R41: 2k2, Resistor_SMD:R_0603_1608Metric_Pad0.98x0.95mm_HandSolder, F.Cu at (401.6, 32.6)
- added R42: 10k, Resistor_SMD:R_0603_1608Metric_Pad0.98x0.95mm_HandSolder, F.Cu at (387.8, 45.1)
- added RV1: 10k, Potentiometer_SMD:Potentiometer_Bourns_3314J_Vertical, F.Cu at (336.5, 70.2)
- added RV2: 10k, Potentiometer_SMD:Potentiometer_Bourns_3314J_Vertical, F.Cu at (342.5, 70.2)
- added RV3: 10k, Potentiometer_SMD:Potentiometer_Bourns_3314J_Vertical, F.Cu at (372.3, 38.6)
- added RV4: 10k, Potentiometer_SMD:Potentiometer_Bourns_3314J_Vertical, F.Cu at (330.4, 70.2)
- added U7: SA818S, Z_mycustom_footprint_lib:SA818S, F.Cu at (346.1, 35.7)
- added U8: SA818S, Z_mycustom_footprint_lib:SA818S, F.Cu at (346.1, 56.2)
- C1: value DNP -> 100n
- C11, C12, C14, C15, C3, C9: value 100n -> 10u; footprint Capacitor_SMD:C_0603_1608Metric_Pad1.08x0.95mm_HandSolder -> Capacitor_SMD:C_0805_2012Metric
- C17: value 100n -> 1u
- C18, C21, C34: value 1u -> 10u; footprint Capacitor_SMD:C_0603_1608Metric_Pad1.08x0.95mm_HandSolder -> Capacitor_SMD:C_0805_2012Metric
- C19, C22: value 4n7 -> 10u; footprint Capacitor_SMD:C_0603_1608Metric_Pad1.08x0.95mm_HandSolder -> Capacitor_SMD:C_0805_2012Metric
- C24, C26, C28, C30: value 1u -> 22u; footprint Capacitor_SMD:C_0603_1608Metric_Pad1.08x0.95mm_HandSolder -> Capacitor_SMD:C_0805_2012Metric
- C27: value 1u -> 4n7
- C32: value 10u -> 4n7; footprint Capacitor_SMD:C_0805_2012Metric -> Capacitor_SMD:C_0603_1608Metric_Pad1.08x0.95mm_HandSolder
- C33: value 10u -> 22u
- C5: value 10u -> 100n; footprint Capacitor_SMD:C_0805_2012Metric -> Capacitor_SMD:C_0603_1608Metric_Pad1.08x0.95mm_HandSolder
- C6: value 100n -> 15p
- C7: value 15p -> 10u; footprint Capacitor_SMD:C_0603_1608Metric_Pad1.08x0.95mm_HandSolder -> Capacitor_SMD:C_0805_2012Metric
- C8: value 10u -> 1u; footprint Capacitor_SMD:C_0805_2012Metric -> Capacitor_SMD:C_0603_1608Metric_Pad1.08x0.95mm_HandSolder
- J3: value SMA -> Conn_01x02; footprint Connector_Coaxial:SMA_Amphenol_901-144_Vertical -> Connector_PinHeader_2.54mm:PinHeader_1x02_P2.54mm_Vertical
- J4: value SMA -> Conn_01x06; footprint Connector_Coaxial:SMA_Amphenol_901-144_Vertical -> Connector_PinHeader_2.54mm:PinHeader_1x06_P2.54mm_Vertical
- R12, R13: value 10k -> 10; footprint Resistor_SMD:R_0603_1608Metric_Pad0.98x0.95mm_HandSolder -> Resistor_SMD:R_0402_1005Metric
- R14, R17, R18: footprint Resistor_SMD:R_0603_1608Metric_Pad0.98x0.95mm_HandSolder -> Resistor_SMD:R_0402_1005Metric
- R15, R4: value 10k -> 1k; footprint Resistor_SMD:R_0603_1608Metric_Pad0.98x0.95mm_HandSolder -> Resistor_SMD:R_0805_2012Metric
- R16: value 10k -> 0R2
- R19: value 10 -> 10k
- R20: value 27 -> 10k
- R22, R23: value 27 -> 5k1; footprint Resistor_SMD:R_0402_1005Metric -> Resistor_SMD:R_0603_1608Metric_Pad0.98x0.95mm_HandSolder
- R25: value 27 -> 10
- R26, R27: value 10k -> 27; footprint Resistor_SMD:R_0603_1608Metric_Pad0.98x0.95mm_HandSolder -> Resistor_SMD:R_0402_1005Metric
- R28, R29: value 100k -> 27; footprint Resistor_SMD:R_0805_2012Metric -> Resistor_SMD:R_0402_1005Metric
- R30: value 1k -> 10k
- R31: value 2k7 -> 10k
- R5: value 1Meg -> 1k; footprint Resistor_SMD:R_0603_1608Metric_Pad0.98x0.95mm_HandSolder -> Resistor_SMD:R_0805_2012Metric
- R6: value 10 -> 10k; footprint Resistor_SMD:R_0402_1005Metric -> Resistor_SMD:R_0603_1608Metric_Pad0.98x0.95mm_HandSolder
- R7: value 10 -> 1Meg; footprint Resistor_SMD:R_0402_1005Metric -> Resistor_SMD:R_0603_1608Metric_Pad0.98x0.95mm_HandSolder
- U3: value SA818S -> AMS1117-3.3; footprint Z_mycustom_footprint_lib:SA818S -> Package_TO_SOT_SMD:SOT-223-3_TabPin2; moved to F.Cu
- U4: value SA818S -> TP5000; footprint Z_mycustom_footprint_lib:SA818S -> Package_DFN_QFN:QFN-16-1EP_4x4mm_P0.65mm_EP2.5x2.5mm_ThermalVias; moved to F.Cu
- U5: value TPA2012D2 -> ES8388; footprint Package_DFN_QFN:QFN-20-1EP_4x4mm_P0.5mm_EP2.6x2.6mm_ThermalVias -> Package_DFN_QFN:QFN-28-1EP_4x4mm_P0.4mm_EP2.4x2.4mm_ThermalVias
- U6: value ES8388 -> TPA2012D2; footprint Package_DFN_QFN:QFN-28-1EP_4x4mm_P0.4mm_EP2.4x2.4mm_ThermalVias -> Package_DFN_QFN:QFN-20-1EP_4x4mm_P0.5mm_EP2.6x2.6mm_ThermalVias
- moved FL2 312.1 mm to (391.0, 27.7)
- moved C13 288.4 mm to (401.8, 26.9)
- moved U4 282.8 mm to (383.7, 87.7), turned to 0 degrees
- moved R18 280.5 mm to (384.9, 96.3)
- moved R24 280.0 mm to (397.1, 83.9)
- moved R20 277.8 mm to (401.0, 80.9)
- moved R12 276.8 mm to (373.1, 108.6)
- moved R10 272.2 mm to (390.1, 93.1)
- moved R23 267.8 mm to (389.0, 88.8)
- moved FL1 267.0 mm to (348.5, 68.8)
- moved C4 262.6 mm to (376.9, 95.1)
- moved R1 261.9 mm to (362.7, 116.8)
- moved R9 261.4 mm to (385.7, 94.3)
- moved R8 257.9 mm to (377.5, 106.0)
- moved R16 257.5 mm to (393.5, 84.7)
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Connections:
- C1 pad 1: /ESP_EN -> GND
- C1 pad 2: GND -> /ESP_EN
- C10 pad 1: +5V -> Net-(BT1-Pad1)
- C11 pad 1: +5V -> +3V3
- C12 pad 1: +5V -> Net-(C12-Pad1)
- C13 pad 1: GND -> Net-(C13-Pad1)
- C13 pad 2: +5V -> GND
- C14 pad 1: +5V -> Net-(C14-Pad1)
- C15 pad 1: Net-(C15-Pad1) -> Net-(C14-Pad1)
- C16 pad 1: +5V -> Net-(C14-Pad1)
- C17 pad 1: +5V -> Net-(C17-Pad1)
- C17 pad 2: GND -> Net-(C17-Pad2)
- C18 pad 1: Audio_OUT_L -> +3V3
- C18 pad 2: Net-(C18-Pad2) -> GND
- C19 pad 1: Audio_OUT_L -> +3V3
- C2 pad 1: GND -> /ESP_BOOT
- C2 pad 2: /ESP_EN -> GND
- C20 pad 2: Net-(C20-Pad2) -> /Audio_Codec/3V33
- C21 pad 1: Audio_OUT_R -> /Audio_Codec/3V33
- C21 pad 2: Net-(C21-Pad2) -> GND
- C22 pad 1: Audio_OUT_R -> /Audio_Codec/3V33
- C23 pad 2: Net-(C23-Pad2) -> /Audio_Codec/3V33
- C24 pad 2: unconnected-(C24-Pad2) -> LINE_IN1
- C25 pad 2: unconnected-(C25-Pad2) -> Net-(C25-Pad2)
- C26 pad 2: unconnected-(C26-Pad2) -> /Audio_Codec/Jack_MIC_INPUT_1
- C27 pad 1: Net-(C27-Pad1) -> Net-(C25-Pad1)
- C27 pad 2: unconnected-(C27-Pad2) -> GND
- C28 pad 2: unconnected-(C28-Pad2) -> LINE_IN2
- C29 pad 1: Net-(C29-Pad1) -> GND
- C29 pad 2: unconnected-(C29-Pad2) -> Net-(C29-Pad2)
- C3 pad 1: /ESP_BOOT -> +3V3
- C30 pad 1: unconnected-(C30-Pad1) -> Net-(C30-Pad1)
- C30 pad 2: Net-(C30-Pad2) -> /Audio_Codec/MIC_INPUT_2
- C31 pad 1: unconnected-(C31-Pad1) -> Net-(C31-Pad1)
- C32 pad 1: unconnected-(C32-Pad1) -> Net-(C31-Pad1)
- C33 pad 1: unconnected-(C33-Pad1) -> R_out1
- C33 pad 2: GND -> Net-(C33-Pad2)
- C34 pad 2: unconnected-(C34-Pad2) -> GND
- C35 pad 1: Net-(C35-Pad1) -> GND
- C35 pad 2: unconnected-(C35-Pad2) -> Net-(C35-Pad2)
- C6 pad 1: +3V3 -> Net-(C6-Pad1)
- C7 pad 1: Net-(C7-Pad1) -> +3V3
- C8 pad 1: +3V3 -> GND
- C8 pad 2: GND -> +3V3
- C9 pad 1: +3V3 -> +5V
- FL1 pad 1: /ant3 -> /Audio_Codec/ant1
- FL1 pad 3: /ant4 -> /Audio_Codec/ant2
- FL2 pad 1: /ant1 -> /Audio_Codec/ant3
- FL2 pad 3: /ant2 -> /Audio_Codec/ant4
- J1 pad S1: Net-(C7-Pad1) -> Net-(C6-Pad1)
- J3 pad 1: /ant4 -> GND
- J3 pad 2: GND -> Net-(J3-Pad2)
- J4 pad 1: /ant2 -> +3V3
- JP1 pad 1: GND -> +3V3
- JP1 pad 2: Net-(JP1-Pad2) -> Net-(C13-Pad1)
- JP1 pad 3: +3V3 -> +5V
- L1 pad 1: +5V -> Net-(C13-Pad1)
- L1 pad 2: Net-(C15-Pad1) -> Net-(C14-Pad1)
- R10 pad 1: /CMD -> /DATA_2
- R10 pad 2: GPIO_43 -> GPIO_1
- R11 pad 1: /CLK -> /DATA_3
- R11 pad 2: GPIO_44 -> GPIO_2
- R12 pad 1: /DATA_0 -> /CMD
- R12 pad 2: +3V3 -> GPIO_43
- R13 pad 1: /DATA_1 -> /CLK
- R13 pad 2: +3V3 -> GPIO_44
- R14 pad 1: /DATA_2 -> /DATA_0
- R15 pad 1: /DATA_3 -> +5V
- R15 pad 2: +3V3 -> Net-(D4-Pad2)
- R16 pad 1: /CMD -> Net-(BT1-Pad1)
- R16 pad 2: +3V3 -> Net-(C12-Pad1)
- R17 pad 1: /CLK -> /DATA_1
- R18 pad 1: /CARD_DETECT -> /DATA_2
- R19 pad 1: /CARD_DETECT -> /DATA_3
- R19 pad 2: GPIO_40 -> +3V3
- R20 pad 1: GPIO_48 -> /CMD
- R20 pad 2: /RESET -> +3V3
- R21 pad 1: GPIO_47 -> /CARD_DETECT
- R21 pad 2: /Audio_Codec/MCLK -> GPIO_40
- R22 pad 1: GPIO_14 -> +3V3
- R22 pad 2: /Audio_Codec/WCLK -> SDA
- R23 pad 1: GPIO_21 -> +3V3
- R23 pad 2: /Audio_Codec/BCLK -> SCL
- R24 pad 1: GPIO_11 -> GPIO_48
- R24 pad 2: /Audio_Codec/DOUT -> /RESET
- R25 pad 1: GPIO_12 -> GPIO_47
- R25 pad 2: /Audio_Codec/DIN -> /Audio_Codec/MCLK
- R26 pad 1: GND -> GPIO_14
- R26 pad 2: PD1 -> /Audio_Codec/WCLK
- R27 pad 1: PD2 -> GPIO_21
- R27 pad 2: GND -> /Audio_Codec/BCLK
- R28 pad 1: unconnected-(R28-Pad1) -> GPIO_11
- R28 pad 2: GND -> /Audio_Codec/DOUT
- R29 pad 1: +3V3 -> GPIO_12
- R29 pad 2: GPIO_13 -> /Audio_Codec/DIN
- R30 pad 1: unconnected-(R30-Pad1) -> GND
- R30 pad 2: unconnected-(R30-Pad2) -> Net-(Q1-Pad1)
- R31 pad 1: unconnected-(R31-Pad1) -> GND
- R31 pad 2: unconnected-(R31-Pad2) -> PD1
- R4 pad 1: /ESP_BOOT -> Net-(D1-Pad1)
- R4 pad 2: +3V3 -> GND
- R5 pad 1: GND -> Net-(D2-Pad1)
- R5 pad 2: Net-(C7-Pad1) -> GND
- R6 pad 1: /DATA_0 -> /ESP_BOOT
- R6 pad 2: GPIO_42 -> +3V3
- R7 pad 1: /DATA_1 -> GND
- R7 pad 2: GPIO_41 -> Net-(C6-Pad1)
- R8 pad 1: /DATA_2 -> /DATA_0
- R8 pad 2: GPIO_1 -> GPIO_42
- R9 pad 1: /DATA_3 -> /DATA_1
- R9 pad 2: GPIO_2 -> GPIO_41
- U2 pad 5: GPIO_5 -> G0
- U2 pad 6: GPIO_6 -> G1
- U3 pad 1: AUDIO_ON1 -> GND
- U3 pad 2: unconnected-(U3-Pad2) -> +3V3
- U3 pad 3: unconnected-(U3-Pad3) -> +5V
- U4 pad 1: AUDIO_ON2 -> +5V
- U4 pad 10: GND -> Net-(C53-Pad1)
- U4 pad 11: unconnected-(U4-Pad11) -> Net-(J3-Pad2)
- U4 pad 12: /ant1 -> GND
- U4 pad 13: unconnected-(U4-Pad13) -> /CS
- U4 pad 14: unconnected-(U4-Pad14) -> Net-(D4-Pad1)
- U4 pad 15: unconnected-(U4-Pad15) -> Net-(D5-Pad1)
- U4 pad 16: TX2 -> +5V
- U4 pad 17: RX2 -> (no net)
- U4 pad 2: unconnected-(U4-Pad2) -> +5V
- U4 pad 3: unconnected-(U4-Pad3) -> Net-(D3-Pad1)
- U4 pad 4: unconnected-(U4-Pad4) -> Net-(D3-Pad1)
- U4 pad 5: PTT2 -> Net-(D3-Pad1)
- U4 pad 6: PD2 -> GND
- U4 pad 7: H/L2 -> GND
- U4 pad 8: +5V -> Net-(C12-Pad1)
- U4 pad 9: GND -> Net-(BT1-Pad1)
- U5 pad 1: GPIO_5 -> /Audio_Codec/MCLK
- U5 pad 10: (no net) -> Net-(C34-Pad1)
- U5 pad 11: (no net) -> Net-(C33-Pad2)
- U5 pad 12: GND -> Net-(C36-Pad2)
- U5 pad 13: +5V -> GND
- U5 pad 14: (no net) -> Net-(C48-Pad2)
- U5 pad 15: GPIO_6 -> Net-(C49-Pad2)
- U5 pad 16: unconnected-(U5-Pad16) -> /Audio_Codec/3V33
- U5 pad 17: Net-(C23-Pad2) -> /Audio_Codec/3V33
- U5 pad 19: Net-(C20-Pad2) -> Net-(C42-Pad2)
- U5 pad 2: unconnected-(U5-Pad2) -> /Audio_Codec/3V33
- U5 pad 20: Net-(C18-Pad2) -> Net-(C44-Pad1)
- U5 pad 21: GND -> Net-(C30-Pad1)
- U5 pad 3: +5V -> /Audio_Codec/3V33
- U5 pad 5: unconnected-(U5-Pad5) -> /Audio_Codec/BCLK
- U5 pad 6: (no net) -> /Audio_Codec/DIN
- U5 pad 7: GPIO_4 -> /Audio_Codec/WCLK
- U5 pad 8: GPIO_4 -> /Audio_Codec/DOUT
- U5 pad 9: Net-(C15-Pad1) -> unconnected-(U5-Pad9)
- U6 pad 1: /Audio_Codec/MCLK -> G1
- U6 pad 10: unconnected-(U6-Pad10) -> (no net)
- U6 pad 11: Net-(C30-Pad2) -> (no net)
- U6 pad 12: Net-(C31-Pad2) -> GND
- U6 pad 13: GND -> Net-(C14-Pad1)
- U6 pad 14: Net-(C34-Pad1) -> (no net)
- U6 pad 15: Net-(C35-Pad1) -> G0
- U6 pad 16: unconnected-(U6-Pad16) -> Net-(J5-Pad3)
- U6 pad 17: GND -> Net-(C31-Pad2)
- U6 pad 19: unconnected-(U6-Pad19) -> Net-(C25-Pad2)
- U6 pad 2: +3V3 -> Net-(J5-Pad1)
- U6 pad 20: unconnected-(U6-Pad20) -> Net-(C29-Pad2)
- U6 pad 21: Net-(C28-Pad1) -> GND
- U6 pad 3: +3V3 -> Net-(C14-Pad1)
- U6 pad 5: /Audio_Codec/BCLK -> Net-(J5-Pad2)
- U6 pad 6: /Audio_Codec/DIN -> (no net)
- U6 pad 7: /Audio_Codec/WCLK -> AMP_L
- U6 pad 8: /Audio_Codec/DOUT -> AMP_R
- U6 pad 9: unconnected-(U6-Pad9) -> Net-(C14-Pad1)

Commit message: l
Parts:
- removed D8: D_Schottky, Diode_SMD:D_SMA_Handsoldering
- removed J4: Conn_01x06, Connector_PinHeader_2.54mm:PinHeader_1x06_P2.54mm_Vertical
- removed L5: L_Small, Inductor_SMD:L_0603_1608Metric
- added J5: Conn_01x04, TerminalBlock:TerminalBlock_bornier-4_P5.08mm, F.Cu at (369.5, 38.7)
- added L4: 4u7, Z_mycustom_footprint_lib:Inductor_2.5x2x1.2mm, F.Cu at (403.0, 88.9)
- added R43: 0R1, Resistor_SMD:R_1206_3216Metric, F.Cu at (355.3, 123.7)
- D4: value green -> red; footprint LED_SMD:LED_0805_2012Metric -> LED_SMD:LED_0603_1608Metric
- L1, L2, L3: value L_Small -> 4u7; footprint Inductor_SMD:L_0603_1608Metric -> Z_mycustom_footprint_lib:Inductor_2.5x2x1.2mm
- R16: value 0R2 -> 0R1; footprint Resistor_SMD:R_0603_1608Metric_Pad0.98x0.95mm_HandSolder -> Resistor_SMD:R_1206_3216Metric
- moved L1 67.2 mm to (396.3, 94.8)
- moved RV4 64.5 mm to (390.7, 47.3)
- moved R10 60.6 mm to (341.1, 128.8)
- moved FL2 60.6 mm to (356.6, 77.5)
- moved RV3 57.1 mm to (332.1, 79.0)
- moved C28 56.5 mm to (405.3, 35.7)
- moved SW1 55.8 mm to (334.6, 126.0)
- moved R42 55.0 mm to (347.6, 82.7)
- moved C53 54.4 mm to (369.1, 122.2)
- moved RV1 53.5 mm to (384.7, 47.0)
- moved C33 53.4 mm to (361.7, 76.7)
- moved R9 52.9 mm to (341.1, 122.8)
- moved C20 52.6 mm to (372.9, 72.5)
- moved R6 49.6 mm to (398.7, 90.9)
- moved C49 49.5 mm to (343.3, 82.7)
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Connections:
- L1 pad 1: Net-(C13-Pad1) -> Net-(BT1-Pad1)
- L1 pad 2: Net-(C14-Pad1) -> +3V3
- L2 pad 1: +3V3 -> Net-(C13-Pad1)
- L2 pad 2: /Audio_Codec/3V33 -> Net-(C14-Pad1)
- R16 pad 1: Net-(BT1-Pad1) -> Net-(R16-Pad1)

Commit message: n
Parts:
- added C58: 10u, Capacitor_SMD:C_0603_1608Metric, F.Cu at (104.5, 171.4)
- added C59: 10u, Capacitor_SMD:C_0603_1608Metric, F.Cu at (101.5, 171.4)
- added C60: 10u, Capacitor_SMD:C_0603_1608Metric, F.Cu at (167.2, 171.3)
- C10, C11, C12, C15, C16, C18, C19, C21, C22, C3, C39, C4, C44, C47, C50, C52, C54, C57, C7, C9: footprint Capacitor_SMD:C_0805_2012Metric -> Capacitor_SMD:C_0603_1608Metric
- C13, C34, C40, C43, C46, C51: value 10u -> 1u; footprint Capacitor_SMD:C_0805_2012Metric -> Capacitor_SMD:C_0402_1005Metric
- C14: footprint Capacitor_SMD:C_0805_2012Metric -> Capacitor_SMD:C_0603_1608Metric; moved to B.Cu
- C17, C20, C23, C27, C32, C35, C37, C38, C42, C45: footprint Capacitor_SMD:C_0603_1608Metric_Pad1.08x0.95mm_HandSolder -> Capacitor_SMD:C_0402_1005Metric
- C25, C29, C31, C41: value 1u -> 10u; footprint Capacitor_SMD:C_0603_1608Metric_Pad1.08x0.95mm_HandSolder -> Capacitor_SMD:C_0603_1608Metric
- C5, C53: value 100n -> 1u; footprint Capacitor_SMD:C_0603_1608Metric_Pad1.08x0.95mm_HandSolder -> Capacitor_SMD:C_0402_1005Metric
- C8, FL1, FL2, U7, U8: moved to B.Cu
- R2, R22, R23, R3, R32, R33, R34, R35, R41: footprint Resistor_SMD:R_0603_1608Metric_Pad0.98x0.95mm_HandSolder -> Resistor_SMD:R_0402_1005Metric
- moved C13 332.8 mm to (89.3, 189.2)
- moved L4 329.5 mm to (88.4, 187.2)
- moved R15 320.4 mm to (84.5, 173.4)
- moved C16 318.8 mm to (94.1, 185.2), turned to -90 degrees
- moved C12 317.9 mm to (91.8, 186.6)
- moved C17 314.3 mm to (92.9, 184.7), turned to 90 degrees
- moved L3 313.1 mm to (98.8, 115.0)
- moved C25 311.6 mm to (96.3, 113.5), turned to 90 degrees
- moved Q1 305.2 mm to (90.8, 168.6)
- moved L1 304.0 mm to (102.7, 173.9), turned to 90 degrees
- moved D4 300.0 mm to (89.4, 174.2), turned to 90 degrees
- moved R3 299.9 mm to (92.1, 98.5)
- moved C5 299.2 mm to (99.6, 82.4), turned to -90 degrees
- moved R35 298.8 mm to (147.4, 170.2), turned to -90 degrees
- moved D5 298.6 mm to (87.4, 174.4), turned to 90 degrees
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Connections:
- C11 pad 1: +3V3 -> Net-(BT1-Pad1)
- C12 pad 1: Net-(C12-Pad1) -> Net-(L4-Pad2)
- C13 pad 1: Net-(C13-Pad1) -> GND
- C13 pad 2: GND -> Net-(L4-Pad2)
- C14 pad 1: Net-(C14-Pad1) -> +3V3
- C15 pad 1: Net-(C14-Pad1) -> +3V3
- C16 pad 1: Net-(C14-Pad1) -> Net-(BT1-Pad1)
- C17 pad 1: Net-(C17-Pad1) -> GND
- C17 pad 2: Net-(C17-Pad2) -> Net-(BT1-Pad1)
- C18 pad 1: +3V3 -> /Audio_Codec/Power_amp_Vcc_intermediate
- C19 pad 1: +3V3 -> /Audio_Codec/Power_amp_Vcc
- C21 pad 1: /Audio_Codec/3V33 -> /Audio_Codec/Power_amp_Vcc
- C22 pad 1: /Audio_Codec/3V33 -> /Audio_Codec/Power_amp_Vcc
- C23 pad 1: GND -> Net-(RV1-Pad2)
- C23 pad 2: /Audio_Codec/3V33 -> Net-(R32-Pad1)
- C25 pad 1: Net-(C25-Pad1) -> +3V3
- C25 pad 2: Net-(C25-Pad2) -> GND
- C27 pad 1: Net-(C25-Pad1) -> Net-(C27-Pad1)
- C29 pad 1: GND -> /Audio_Codec/3V33
- C29 pad 2: Net-(C29-Pad2) -> GND
- C31 pad 1: Net-(C31-Pad1) -> /Audio_Codec/3V33
- C31 pad 2: Net-(C31-Pad2) -> GND
- C32 pad 1: Net-(C31-Pad1) -> Net-(C32-Pad1)
- C34 pad 1: Net-(C34-Pad1) -> GND
- C34 pad 2: GND -> /Audio_Codec/3V33
- C35 pad 1: GND -> Net-(C27-Pad1)
- C37 pad 1: Net-(C37-Pad1) -> GND
- C38 pad 1: GND -> Net-(C32-Pad1)
- C38 pad 2: /Audio_Codec/3V33 -> Net-(C38-Pad2)
- C40 pad 1: /Audio_Codec/3V33 -> GND
- C40 pad 2: GND -> Net-(C40-Pad2)
- C41 pad 1: GND -> Net-(U5-Pad10)
- C41 pad 2: /Audio_Codec/3V33 -> GND
- C42 pad 1: GND -> Net-(C42-Pad1)
- C42 pad 2: Net-(C42-Pad2) -> Net-(RV2-Pad2)
- C43 pad 1: Net-(C42-Pad2) -> /Audio_Codec/3V33
- C44 pad 1: Net-(C44-Pad1) -> /Audio_Codec/3V33
- C45 pad 2: Net-(C44-Pad1) -> /Audio_Codec/3V33
- C46 pad 1: Net-(C12-Pad1) -> Net-(U5-Pad19)
- C47 pad 1: +5V -> Net-(U5-Pad19)
- C5 pad 1: +3V3 -> GND
- C5 pad 2: GND -> +3V3
- C50 pad 1: +3V3 -> Net-(U5-Pad20)
- C51 pad 1: Net-(BT1-Pad1) -> GND
- C51 pad 2: GND -> Net-(U5-Pad20)
- C52 pad 1: Net-(BT1-Pad1) -> +5V
- C53 pad 1: Net-(C53-Pad1) -> GND
- C53 pad 2: GND -> Net-(U4-Pad10)
- C57 pad 1: GND -> +3V3
- C57 pad 2: +5V -> GND
- C7 pad 1: +3V3 -> +5V
- J9 pad 2: Net-(J9-Pad2) -> GPIO_45
- JP1 pad 2: Net-(C13-Pad1) -> /Audio_Codec/Power_amp_Vcc_intermediate
- L2 pad 1: Net-(C13-Pad1) -> /Audio_Codec/Power_amp_Vcc_intermediate
- L2 pad 2: Net-(C14-Pad1) -> /Audio_Codec/Power_amp_Vcc
- L4 pad 2: Net-(C12-Pad1) -> Net-(L4-Pad2)
- Q1 pad 1: Net-(J9-Pad2) -> GPIO_45
- R16 pad 2: Net-(C12-Pad1) -> Net-(L4-Pad2)
- R26 pad 1: GPIO_14 -> GPIO_12
- R29 pad 1: GPIO_12 -> GPIO_14
- R30 pad 2: Net-(J9-Pad2) -> GPIO_45
- R32 pad 1: Net-(C17-Pad1) -> Net-(R32-Pad1)
- R32 pad 2: Net-(C25-Pad1) -> Net-(C27-Pad1)
- R33 pad 1: Net-(C25-Pad1) -> R_out1
- R33 pad 2: R_out1 -> Net-(C27-Pad1)
- R34 pad 1: Net-(C31-Pad1) -> +3V3
- R34 pad 2: L_out1 -> /Audio_Codec/Jack_MIC_INPUT_1
- R35 pad 1: Net-(C31-Pad1) -> L_out1
- R35 pad 2: Net-(C37-Pad2) -> Net-(C32-Pad1)
- R41 pad 1: +3V3 -> Net-(C32-Pad1)
- R41 pad 2: /Audio_Codec/Jack_MIC_INPUT_1 -> Net-(C42-Pad1)
- RV1 pad 1: GND -> Tranceiver_Audio_OUT_1
- RV1 pad 2: Net-(C17-Pad2) -> Net-(RV1-Pad2)
- RV1 pad 3: Tranceiver_Audio_OUT_1 -> GND
- RV2 pad 1: Tranceiver_Audio_OUT_2 -> GND
- RV2 pad 2: Net-(C37-Pad1) -> Net-(RV2-Pad2)
- RV2 pad 3: GND -> Tranceiver_Audio_OUT_2
- U1 pad 1: unconnected-(U1-Pad1) -> D+
- U1 pad 4: D+ -> unconnected-(U1-Pad4)
- U4 pad 10: Net-(C53-Pad1) -> Net-(U4-Pad10)
- U4 pad 8: Net-(C12-Pad1) -> Net-(L4-Pad2)
- U5 pad 10: Net-(C34-Pad1) -> Net-(U5-Pad10)
- U5 pad 19: Net-(C42-Pad2) -> Net-(U5-Pad19)
- U5 pad 20: Net-(C44-Pad1) -> Net-(U5-Pad20)
- U6 pad 11: (no net) -> Net-(J5-Pad4)
- U6 pad 13: Net-(C14-Pad1) -> /Audio_Codec/Power_amp_Vcc
- U6 pad 14: (no net) -> Net-(J5-Pad3)
- U6 pad 16: Net-(J5-Pad3) -> Net-(C40-Pad2)
- U6 pad 17: Net-(C31-Pad2) -> Net-(C38-Pad2)
- U6 pad 19: Net-(C25-Pad2) -> Net-(C35-Pad2)
- U6 pad 20: Net-(C29-Pad2) -> Net-(C37-Pad2)
- U6 pad 3: Net-(C14-Pad1) -> /Audio_Codec/Power_amp_Vcc
- U6 pad 9: Net-(C14-Pad1) -> /Audio_Codec/Power_amp_Vcc
Other:
- copper layers 2 -> 4

Commit message: b
Parts:
- removed J9: Conn_01x03, Connector_PinHeader_2.54mm:PinHeader_1x03_P2.54mm_Vertical
- added C61: 10u, Capacitor_SMD:C_0603_1608Metric, F.Cu at (328.9, 132.5)
- added C62: 10u, Capacitor_SMD:C_0603_1608Metric, F.Cu at (328.3, 137.0)
- added Q2: AO3401A, Package_TO_SOT_SMD:SOT-23, F.Cu at (319.5, 133.5)
- added Q3: AO3401A, Package_TO_SOT_SMD:SOT-23, F.Cu at (319.5, 137.9)
- added Q4: AO3401A, Package_TO_SOT_SMD:SOT-23, F.Cu at (324.4, 133.5)
- added R44: 10k, Resistor_SMD:R_0603_1608Metric_Pad0.98x0.95mm_HandSolder, F.Cu at (313.5, 154.9)
- added R45: 10k, Resistor_SMD:R_0603_1608Metric_Pad0.98x0.95mm_HandSolder, F.Cu at (313.5, 157.4)
- added R46: 10k, Resistor_SMD:R_0603_1608Metric_Pad0.98x0.95mm_HandSolder, F.Cu at (324.1, 137.0)
- added TP2: TestPoint, TestPoint:TestPoint_Pad_1.0x1.0mm, F.Cu at (331.8, 135.3)
- J3: value Conn_01x02 -> Screw_Terminal_01x02; footprint Connector_PinHeader_2.54mm:PinHeader_1x02_P2.54mm_Vertical -> TerminalBlock_Altech:Altech_AK300_1x02_P5.00mm_45-Degree
- J5: value Conn_01x04 -> Screw_Terminal_01x02; footprint TerminalBlock:TerminalBlock_bornier-4_P5.08mm -> TerminalBlock_Altech:Altech_AK300_1x02_P5.00mm_45-Degree
- moved C52 204.8 mm to (120.5, 148.7)
- moved C55 204.8 mm to (120.5, 147.2)
- moved FL1 204.8 mm to (137.9, 141.9)
- moved J7 204.8 mm to (140.8, 133.2)
- moved U7 204.8 mm to (125.0, 131.0)
- moved C54 144.1 mm to (103.3, 114.0)
- moved C56 144.1 mm to (103.3, 115.6)
- moved FL2 144.1 mm to (85.4, 121.3)
- moved J8 144.1 mm to (83.5, 129.8)
- moved U8 144.1 mm to (99.0, 131.8)
- moved J3 37.7 mm to (128.3, 190.3), turned to 0 degrees
- moved J5 15.6 mm to (155.3, 189.2)
Connections:
- C57 pad 1: +3V3 -> Net-(C57-Pad1)
- C58 pad 1: +3V3 -> Net-(C58-Pad1)
- C59 pad 1: +3V3 -> Net-(C58-Pad1)
- J3 pad 1: GND -> Net-(U6-Pad2)
- J3 pad 2: Net-(J3-Pad2) -> Net-(U6-Pad5)
- J5 pad 1: Net-(J5-Pad1) -> Net-(U6-Pad11)
- J5 pad 2: Net-(J5-Pad2) -> Net-(U6-Pad14)
- L1 pad 2: +3V3 -> Net-(C58-Pad1)
- U3 pad 2: +3V3 -> Net-(C57-Pad1)
- U4 pad 11: Net-(J3-Pad2) -> Net-(U4-Pad11)
- U6 pad 11: Net-(J5-Pad4) -> Net-(U6-Pad11)
- U6 pad 14: Net-(J5-Pad3) -> Net-(U6-Pad14)
- U6 pad 2: Net-(J5-Pad1) -> Net-(U6-Pad2)
- U6 pad 5: Net-(J5-Pad2) -> Net-(U6-Pad5)
Other:
- board outline added: 80 x 79.4 mm

Commit message: g
Parts:
- R46: footprint Resistor_SMD:R_0603_1608Metric_Pad0.98x0.95mm_HandSolder -> Resistor_SMD:R_0402_1005Metric
- moved H1 299.2 mm to (55.0, 55.0)
- moved C2 293.4 mm to (70.6, 62.5), turned to 180 degrees
- moved C1 292.7 mm to (63.4, 62.7)
- moved U3 287.9 mm to (71.9, 81.0), turned to -90 degrees
- moved C7 286.2 mm to (69.7, 75.0), turned to 90 degrees
- moved C57 282.2 mm to (73.1, 75.8), turned to 0 degrees
- moved SW1 278.4 mm to (62.4, 57.1), turned to -90 degrees
- moved R6 278.3 mm to (75.1, 55.1)
- moved H4 277.8 mm to (55.0, 115.0)
- moved R1 269.9 mm to (75.1, 56.7), turned to 180 degrees
- moved C62 263.9 mm to (73.0, 70.2)
- moved C61 263.7 mm to (73.0, 68.6)
- moved R46 263.4 mm to (68.4, 74.0), turned to 90 degrees
- moved Q2 260.5 mm to (66.1, 73.1), turned to -90 degrees
- moved SW2 258.9 mm to (69.7, 57.1), turned to -90 degrees
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Other:
- board size 80 x 79.4 mm -> 80 x 70 mm

Commit message: f
Parts:
- added FB1: FerriteBead_Small, Resistor_SMD:R_0805_2012Metric, F.Cu at (64.3, 70.3)
- added R47: 10, Resistor_SMD:R_0402_1005Metric, F.Cu at (155.4, 77.0)
- added R48: 10, Resistor_SMD:R_0402_1005Metric, F.Cu at (158.3, 77.0)
- added R49: 10, Resistor_SMD:R_0402_1005Metric, F.Cu at (155.4, 75.0)
- added R50: 10, Resistor_SMD:R_0402_1005Metric, F.Cu at (158.3, 75.0)
- JP2: moved to B.Cu
- moved R5 194.2 mm to (53.3, 81.3)
- moved D1 194.1 mm to (53.4, 75.0)
- moved R4 185.7 mm to (53.4, 77.1)
- moved D2 180.9 mm to (53.4, 79.2)
- moved TP2 172.2 mm to (71.8, 107.3), turned to 180 degrees
- moved FID1 129.3 mm to (120.0, 55.0)
- moved C24 116.9 mm to (99.9, 85.4), turned to -90 degrees
- moved C49 105.2 mm to (115.2, 69.2), turned to 180 degrees
- moved RV4 104.1 mm to (103.7, 91.5), turned to 180 degrees
- moved JP2 101.1 mm to (95.7, 79.9), turned to -90 degrees
- moved C48 101.0 mm to (115.2, 67.0), turned to 180 degrees
- moved C26 98.9 mm to (103.5, 73.0)
- moved C28 93.5 mm to (103.5, 75.1)
- moved R42 87.9 mm to (120.6, 62.1)
- moved RV3 83.1 mm to (108.3, 77.0), turned to 180 degrees
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Connections:
- RV1 pad 1: Tranceiver_Audio_OUT_1 -> GND
- RV1 pad 3: GND -> Tranceiver_Audio_OUT_1
- RV2 pad 1: GND -> Tranceiver_Audio_OUT_2
- RV2 pad 3: Tranceiver_Audio_OUT_2 -> GND
- RV3 pad 1: Tranceiver_Audio_OUT_2 -> GND
- RV3 pad 3: GND -> Tranceiver_Audio_OUT_2
- RV4 pad 1: GND -> Tranceiver_Audio_OUT_1
- RV4 pad 3: Tranceiver_Audio_OUT_1 -> GND
- U2 pad 5: G0 -> GPIO_5
- U2 pad 6: G1 -> GPIO_6

Commit message: f
Parts:
- R38, R39: footprint Resistor_SMD:R_0805_2012Metric -> Resistor_SMD:R_0603_1608Metric
- moved R7 161.3 mm to (54.9, 60.7), turned to -90 degrees
- moved C6 155.8 mm to (53.3, 60.7), turned to 90 degrees
- moved C36 90.7 mm to (92.6, 89.6), turned to 180 degrees
- moved C33 86.0 mm to (92.6, 91.6), turned to 180 degrees
- moved C30 83.3 mm to (96.5, 83.0)
- moved R47 42.5 mm to (195.1, 91.9)
- moved R48 41.4 mm to (195.1, 95.9)
- moved R49 41.4 mm to (192.2, 93.9)
- moved R50 39.8 mm to (192.2, 95.9)
- moved R38 20.9 mm to (171.4, 95.4)
- moved R39 19.7 mm to (166.9, 98.4)
- moved R23 18.5 mm to (192.2, 91.9)
- moved R22 18.4 mm to (195.1, 93.9)
- moved R34 16.8 mm to (179.0, 97.4)
- moved R44 15.5 mm to (175.8, 92.2)
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Routing:
- added copper zone on B.Cu, net GND
- added copper zone on F.Cu, net GND
- added copper zone on In1.Cu, net GND
- added copper zone on In2.Cu, net GND
