File: HW/cross_band_handy_walkie_talkie_ES8388/cross_band_handy_walkie_talkie_ES8388.kicad_pcb (KiCad board)
At the start: 4 copper layers, 80 x 70 mm, 162 parts, among them J1 USB_C_Receptacle, J2 Micro_SD_Card_Det, J3 Screw_Terminal_01x02, J5 Screw_Terminal_01x02, J6 AudioJack4_SwitchTR1, J7 SMA, J8 SMA, Q1 nMOS, Q2 AO3401A, Q3 AO3401A, Q4 AO3401A, SW1 MCU_RESET, SW2 MCU_RESET, U1 SRV05-4, U2 ESP32-S3-WROOM-1, U3 AMS1117-3.3, U4 TP5000, U5 ES8388, U6 TPA2012D2, U7 SA818S, U8 SA818S

Commit message: e
Parts:
- removed R24: 27, Resistor_SMD:R_0402_1005Metric
- moved R34 70.3 mm to (112.5, 74.5), turned to -90 degrees
- moved C59 20.8 mm to (59.4, 103.5), turned to 180 degrees
- moved C58 19.6 mm to (62.4, 103.5), turned to 0 degrees
- moved L1 16.8 mm to (60.6, 106.0), turned to 90 degrees
- moved C10 14.4 mm to (59.3, 108.6), turned to 180 degrees
- moved C11 12.6 mm to (62.4, 108.6), turned to 0 degrees
- moved C24 8.90 mm to (100.2, 76.5), turned to 0 degrees
- moved C26 6.42 mm to (100.2, 78.5)
- moved C28 6.32 mm to (100.2, 80.5)
- moved C30 3.78 mm to (100.2, 82.6)
- moved C61 3.57 mm to (75.6, 71.1), turned to -90 degrees
- moved C49 2.68 mm to (114.9, 71.9)
- moved R7 1.87 mm to (56.8, 60.7), turned to 0 degrees
- moved FL1 1.54 mm to (122.8, 94.8)
- moved R42 1.03 mm to (120.7, 61.1), turned to -90 degrees
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Connections:
- net Net-(C24-Pad1) renamed /Audio_Codec/A_audio_1
- net Net-(C26-Pad1) renamed /Audio_Codec/A_audio_2
- net Net-(C28-Pad1) renamed /Audio_Codec/A_audio_3
- net Net-(C30-Pad1) renamed /Audio_Codec/A_audio_4
- net Net-(C33-Pad2) renamed /Audio_Codec/R_out1_
- net Net-(C36-Pad2) renamed /Audio_Codec/L_out1_
- net Net-(C57-Pad1) renamed /RAW_3v3
- net Net-(D3-Pad1) renamed /buck_out
- C24 pad 2: LINE_IN1 -> LINE_IN2
- C28 pad 2: LINE_IN2 -> LINE_IN1
- U4 pad 17: (no net) -> GND
Routing:
- net GND: track 0.00 -> 144.6 mm, vias 0 -> 77
- net +3V3: track 0.00 -> 67.9 mm, vias 0 -> 7
- net +5V: track 0.00 -> 54.5 mm, vias 0 -> 6
- net /Audio_Codec/Jack_MIC_INPUT_1: track 0.00 -> 38.1 mm
- net /ESP_BOOT: track 0.00 -> 33.7 mm, vias 0 -> 2
- net Tranceiver_Audio_OUT_1: track 0.00 -> 29.7 mm, vias 0 -> 1
- net D+: track 0.00 -> 25.4 mm
- net Net-(BT1-Pad1): track 0.00 -> 25.2 mm
- net D-: track 0.00 -> 25.0 mm
- net /DATA_1: track 0.00 -> 21.6 mm, vias 0 -> 2
- net /ESP_EN: track 0.00 -> 19.9 mm
- net /DATA_0: track 0.00 -> 19.4 mm, vias 0 -> 2
- net GPIO_13: track 0.00 -> 18.4 mm, vias 0 -> 2
- net VBUS: track 0.00 -> 16.5 mm
- net /CLK: track 0.00 -> 16.3 mm, vias 0 -> 2
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- added copper zone on F.Cu, net /RAW_3v3

Commit message: m
Routing:
- added copper zone on F.Cu, net /Audio_Codec/3V33
Changed lines of the file:
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@@
   (segment (start 92.255 78.4325) (end 92.255 77.755) (width 0.2933) (layer "F.Cu") (net 45))
   (segment (start 91.055 82.3075) (end 90.655 82.3075) (width 0.2933) (layer "F.Cu") (net 45))
-  (segment (start 88.685 84.73) (end 88.685 86.635) (width 0.2933) (layer "F.Cu") (net 45))
+  (segment (start 88.685 84.73) (end 88.685 86.635) (width 0.5) (layer "F.Cu") (net 45))
   (segment (start 90.48 87.22) (end 90.48 83.675) (width 0.2933) (layer "F.Cu") (net 45))
   (segment (start 92.55 77.17) (end 92.55 75.55) (width 0.2933) (layer "F.Cu") (net 45))
@@
     )
   )
+  (zone (net 45) (net_name "/Audio_Codec/3V33") (layer "F.Cu") (hatch edge 0.508)
+    (priority 1)
+    (connect_pads yes (clearance 0.3))
+    (min_thickness 0.2) (filled_areas_thickness no)
+    (fill yes (thermal_gap 0.3) (thermal_bridge_width 0.4))
+    (polygon
+      (pts
+        (xy 89.61 85.58)
+        (xy 89.63 83.09)
+        (xy 90.87 83.07)
+        (xy 90.82 84.91)
+        (xy 91.28 85.28)
+        (xy 91.28 88.25)
+        (xy 88.13 88.25)
+        (xy 88.16 85.58)
+      )
+    )
+  )
   (zone (net 2) (net_name "GND") (layer "F.Cu") (hatch edge 0.508)
     (priority 1)
     (connect_pads yes (clearance 0.3))
-    (min_thickness 0.2)
-    (fill (thermal_gap 0.3) (thermal_bridge_width 0.75))
+    (min_thickness 0.2) (filled_areas_thickness no)
+    (fill yes (thermal_gap 0.3) (thermal_bridge_width 0.75))
     (polygon
       (pts

Commit message: n
Parts:
- added J9: Conn_01x04, Connector_PinHeader_2.54mm:PinHeader_1x04_P2.54mm_Vertical, F.Cu at (114.4, 65.9)
- moved R22 99.5 mm to (99.7, 65.9), turned to 180 degrees
- moved R23 95.9 mm to (99.7, 66.9), turned to 180 degrees
- moved R47 35.0 mm to (162.4, 104.5), turned to 180 degrees
- moved R48 33.6 mm to (162.4, 103.5), turned to 180 degrees
- moved C48 2.34 mm to (114.1, 69.1)
- moved C36 0.63 mm to (92.9, 89.0)
- moved C33 0.14 mm to (92.7, 91.7)
Connections:
- D6 pad 2: PTT1 -> GPIO_4
- D7 pad 2: PTT2 -> GPIO_37
- R22 pad 2: SDA -> GPIO_36
- R23 pad 2: SCL -> GPIO_35
- R31 pad 2: PD1 -> GPIO_5
- R44 pad 2: H/L1 -> GPIO_6
- U5 pad 27: SDA -> GPIO_36
- U5 pad 28: SCL -> GPIO_35
- U7 pad 16: TX2 -> GPIO_38
- U7 pad 17: RX2 -> GPIO_39
- U7 pad 5: PTT2 -> GPIO_37
- U8 pad 1: AUDIO_ON1 -> GPIO_9
- U8 pad 16: TX1 -> GPIO_8
- U8 pad 17: RX1 -> GPIO_7
- U8 pad 5: PTT1 -> GPIO_4
- U8 pad 6: PD1 -> GPIO_5
- U8 pad 7: H/L1 -> GPIO_6
Routing:
- net +5V: track 54.5 -> 155.0 mm, vias 6 -> 10
- net +3V3: track 67.9 -> 157.5 mm, vias 7 -> 11
- net GND: track 144.6 -> 204.4 mm, vias 77 -> 115
- net GPIO_36: track 0.00 -> 32.2 mm
- net GPIO_37: track 0.00 -> 32.2 mm, vias 0 -> 4
- net GPIO_38: track 0.00 -> 30.1 mm, vias 0 -> 2
- net GPIO_35: track 0.00 -> 29.1 mm, vias 0 -> 1
- net GPIO_39: track 0.00 -> 28.8 mm, vias 0 -> 2
- net /Audio_Codec/R_out1_: track 0.00 -> 15.9 mm, vias 0 -> 2
- net Net-(C42-Pad2): track 0.00 -> 13.1 mm, vias 0 -> 2
- net /Audio_Codec/3V33: track 14.1 -> 27.2 mm, vias 0 -> 2
- net Net-(C23-Pad1): track 0.00 -> 12.9 mm, vias 0 -> 2
- net /Audio_Codec/L_out1_: track 0.00 -> 11.3 mm, vias 0 -> 2
- net /ESP_EN: track 19.9 -> 29.9 mm, vias 0 -> 2
- net L_out1: track 0.00 -> 4.42 mm
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- added copper zone on F.Cu, net +3V3

Commit message: g
Parts:
- added kibuzzard-6414CC1F: G***, kibuzzard-6414CC1F, F.Cu at (83.3, 92.5)
- added kibuzzard-6414CC2A: G***, kibuzzard-6414CC2A, F.Cu at (88.6, 92.5)
- FID2, FID3: moved to B.Cu
- moved R50 120.7 mm to (77.5, 58.2)
- moved R49 119.8 mm to (77.4, 59.5)
- moved D6 96.5 mm to (83.6, 89.9), turned to 90 degrees
- moved R31 96.0 mm to (84.6, 83.3), turned to 180 degrees
- moved R48 95.2 mm to (77.4, 60.8), turned to 0 degrees
- moved R44 91.5 mm to (85.4, 78.2), turned to 180 degrees
- moved D7 86.6 mm to (89.3, 89.9), turned to 90 degrees
- moved R38 86.4 mm to (85.2, 89.9), turned to 90 degrees
- moved FID2 84.2 mm to (88.7, 55.3), turned to 180 degrees
- moved R39 79.6 mm to (87.8, 89.9), turned to 90 degrees
- moved R45 72.4 mm to (103.5, 99.3)
- moved R37 70.0 mm to (101.4, 96.5)
- moved R47 66.9 mm to (95.5, 103.4), turned to -90 degrees
- moved FID3 57.5 mm to (123.5, 103.7), turned to 180 degrees
- moved J3 0.70 mm to (90.0, 111.0)
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Connections:
- D6 pad 2: GPIO_4 -> GPIO_8
- J6 pad TN: GPIO_13 -> /Audio_Codec/JACK_DETECT
- Q1 pad 1: GPIO_45 -> GPIO_16
- R30 pad 2: GPIO_45 -> GPIO_16
- R31 pad 2: GPIO_5 -> GPIO_17
- R37 pad 1: PD2 -> GPIO_45
- R42 pad 2: GPIO_13 -> /Audio_Codec/JACK_DETECT
- R44 pad 2: GPIO_6 -> GPIO_18
- R45 pad 1: H/L2 -> GPIO_48
- R47 pad 2: unconnected-(R47-Pad2) -> GPIO_5
- R48 pad 2: unconnected-(R48-Pad2) -> GPIO_15
- R49 pad 2: GPIO_6 -> GPIO_7
- R50 pad 2: GPIO_5 -> GPIO_6
- U7 pad 1: AUDIO_ON2 -> GPIO_4
- U7 pad 6: PD2 -> GPIO_45
- U7 pad 7: H/L2 -> GPIO_48
- U8 pad 1: GPIO_9 -> GPIO_13
- U8 pad 16: GPIO_8 -> GPIO_9
- U8 pad 17: GPIO_7 -> GPIO_10
- U8 pad 5: GPIO_4 -> GPIO_8
- U8 pad 6: GPIO_5 -> GPIO_17
- U8 pad 7: GPIO_6 -> GPIO_18
Routing:
- net GPIO_5: track 0.00 -> 118.3 mm, vias 0 -> 3
- net GPIO_16: track 0.00 -> 53.0 mm, vias 0 -> 3
- net GPIO_10: track 0.00 -> 45.1 mm, vias 0 -> 1
- net GPIO_9: track 0.00 -> 39.9 mm, vias 0 -> 1
- net GPIO_48: track 0.00 -> 37.8 mm, vias 0 -> 2
- net GPIO_4: track 0.00 -> 32.5 mm, vias 0 -> 1
- net Net-(C58-Pad1): track 8.03 -> 39.7 mm
- net GPIO_8: track 0.00 -> 31.6 mm, vias 0 -> 2
- net GPIO_45: track 1.82 -> 31.7 mm, vias 0 -> 3
- net +3V3: track 157.5 -> 184.1 mm, vias 11 -> 12
- net GPIO_17: track 0.00 -> 26.5 mm, vias 0 -> 3
- net Net-(J5-Pad2): track 0.00 -> 25.0 mm
- net GPIO_13: track 18.4 -> 43.1 mm, vias 2 -> 1
- net GPIO_18: track 0.00 -> 21.7 mm, vias 0 -> 2
- net Net-(J5-Pad1): track 0.00 -> 20.5 mm
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
Commit message: f
Parts:
- added kibuzzard-641623AE: G***, kibuzzard-641623AE, F.Cu at (59.4, 75.1)
- added kibuzzard-641623CB: G***, kibuzzard-641623CB, F.Cu at (58.8, 79.2)
- moved J7 3.30 mm to (124.0, 89.0)
- moved R34 2.66 mm to (112.3, 71.9)
- moved FL1 2.31 mm to (121.5, 96.7)
- moved J8 0.71 mm to (56.0, 89.0)
- moved C28 0.69 mm to (100.2, 81.2)
- moved C30 0.68 mm to (100.2, 83.2)
- moved C26 0.65 mm to (100.2, 79.2)
- moved C24 0.61 mm to (100.2, 77.1)
Routing:
- net G0: track 0.00 -> 60.6 mm, vias 0 -> 4
- net AMP_L: track 0.00 -> 58.6 mm, vias 0 -> 6
- net G1: track 0.00 -> 56.9 mm, vias 0 -> 4
- net Net-(C48-Pad2): track 0.00 -> 34.7 mm, vias 0 -> 2
- net GND: track 212.9 -> 247.4 mm, vias 123 -> 148
- net Net-(C49-Pad2): track 0.00 -> 32.8 mm, vias 0 -> 2
- net Net-(C6-Pad1): track 6.30 -> 32.2 mm
- net +3V3: track 184.1 -> 205.5 mm
- net Net-(BT1-Pad1): track 25.2 -> 28.9 mm
- net /Audio_Codec/Jack_MIC_INPUT_1: track 38.1 -> 41.2 mm
- net GPIO_37: track 45.4 -> 42.9 mm
- net /Audio_Codec/ant1: track 6.52 -> 4.27 mm
- net Net-(C58-Pad1): track 39.7 -> 41.4 mm
- net /Audio_Codec/L_out1_: track 10.9 -> 12.2 mm
- net /Audio_Codec/ant2: track 8.21 -> 6.99 mm
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- added copper zone on F.Cu, net +5V
- added copper zone on F.Cu, net /Audio_Codec/Power_amp_Vcc

Commit message: r
Parts:
- removed R45: 10k, Resistor_SMD:R_0603_1608Metric_Pad0.98x0.95mm_HandSolder
- added BT2: Battery_Cell, Connector_JST:JST_XH_B2B-XH-AM_1x02_P2.50mm_Vertical, F.Cu at (74.0, 115.0)
- added C63: 22u, Capacitor_SMD:C_0805_2012Metric, F.Cu at (88.0, 110.7)
- added J4: Conn_01x06, Connector_PinHeader_2.54mm:PinHeader_1x06_P2.54mm_Vertical, F.Cu at (84.2, 103.0)
- added R24: 10, Resistor_SMD:R_0402_1005Metric, F.Cu at (81.3, 115.2)
- moved R44 27.8 mm to (103.7, 99.2)
- moved BT1 4.87 mm to (65.0, 114.0)
- moved J3 3.00 mm to (93.0, 111.0)
- moved C30 1.72 mm to (98.8, 84.2), turned to -90 degrees
- moved R37 0.65 mm to (102.0, 96.4)
- moved R47 0.14 mm to (95.5, 103.2)
- moved R48 0.09 mm to (77.5, 60.8)
Connections:
- net GPIO_13 renamed AUDIO_ON1
- net GPIO_4 renamed AUDIO_ON2
- net Net-(J3-Pad1) renamed /Audio_Codec/Speaker_L+
- net Net-(J3-Pad2) renamed /Audio_Codec/Speaker_L-
- net Net-(J5-Pad1) renamed /Audio_Codec/Speaker_R-
- net Net-(J5-Pad2) renamed /Audio_Codec/Speaker_R+
- R44 pad 2: GPIO_18 -> GPIO_48
- R48 pad 1: AMP_L -> G1
- R49 pad 1: G1 -> AMP_L
- U8 pad 7: GPIO_18 -> GPIO_48
Routing:
- net /Audio_Codec/MIC_INPUT_2: track 0.00 -> 53.7 mm, vias 0 -> 3
- net GPIO_18: track 21.7 -> 57.7 mm, vias 2 -> 4
- net GND: track 247.4 -> 229.6 mm, vias 148 -> 165
- net GPIO_48: track 37.8 -> 54.4 mm, vias 2 -> 6
- net +3V3: track 205.5 -> 218.2 mm, vias 12 -> 14
- net GPIO_36: track 32.2 -> 39.3 mm
- net +5V: track 155.0 -> 162.1 mm, vias 10 -> 8
- net /RAW_3v3: track 10.8 -> 4.49 mm
- net GPIO_16: track 53.2 -> 59.0 mm, vias 3 -> 6
- net /Audio_Codec/Speaker_L+: track 16.5 -> 21.8 mm
- net Net-(BT1-Pad1): track 28.9 -> 33.9 mm
- net PTT3: track 0.00 -> 2.97 mm
- net GPIO_38: track 30.1 -> 33.1 mm, vias 2 -> 1
- net Net-(C63-Pad1): track 0.00 -> 2.81 mm
- net AMP_L: track 58.6 -> 61.4 mm
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