File: HW/cross_band_handy_walkie_talkie_ES8388/cross_band_handy_walkie_talkie_ES8388.kicad_pcb (KiCad board)
At the start: 4 copper layers, 80 x 70 mm, 169 parts, among them J1 USB_C_Receptacle, J2 Micro_SD_Card_Det, J3 Screw_Terminal_01x02, J4 Conn_01x06, J5 Screw_Terminal_01x02, J6 AudioJack4_SwitchTR1, J7 SMA, J8 SMA, J9 Conn_01x04, Q1 nMOS, Q2 AO3401A, Q3 AO3401A, Q4 AO3401A, SW1 MCU_RESET, SW2 MCU_RESET, U1 SRV05-4, U2 ESP32-S3-WROOM-1, U3 AMS1117-3.3, U4 TP5000, U5 ES8388, U6 TPA2012D2, U7 SA818S, U8 SA818S

Commit message: y
Parts:
- removed C49: 1u, Capacitor_SMD:C_0603_1608Metric_Pad1.08x0.95mm_HandSolder
- removed kibuzzard-6414CC1F: G***, kibuzzard-6414CC1F
- removed kibuzzard-6414CC2A: G***, kibuzzard-6414CC2A
- added D8: red, LED_SMD:LED_0603_1608Metric, F.Cu at (68.9, 116.3)
- added J10: Conn_01x04, Connector_PinHeader_2.54mm:PinHeader_1x03_P2.54mm_Vertical, F.Cu at (125.4, 61.4)
- added R45: 1k, Resistor_SMD:R_0603_1608Metric, F.Cu at (68.9, 114.8)
- added TP3: TestPoint, TestPoint:TestPoint_Pad_1.0x1.0mm, F.Cu at (114.5, 72.0)
- added kibuzzard-641A07F0: G***, kibuzzard-641A07F0, F.Cu at (88.5, 92.5)
- added kibuzzard-641A0805: G***, kibuzzard-641A0805, F.Cu at (82.9, 92.5)
- moved R42 4.29 mm to (120.3, 56.9)
- moved FID1 2.35 mm to (119.9, 52.6)
Connections:
- net Net-(BT1-Pad1) renamed +BATT
- J6 pad T: Net-(C49-Pad1) -> Net-(C48-Pad1)
- U5 pad 15: Net-(C49-Pad2) -> unconnected-(U5-Pad15)
Routing:
- net unconnected-(U5-Pad15): track 0.00 -> 32.8 mm, vias 0 -> 2
- net Net-(C49-Pad2): track 32.8 -> 0.00 mm, vias 2 -> 0
- net GPIO_44: track 1.79 -> 33.9 mm, vias 0 -> 1
- net GPIO_43: track 1.80 -> 31.0 mm, vias 0 -> 1
- net Net-(C48-Pad1): track 11.9 -> 20.1 mm
- net Net-(C49-Pad1): track 7.43 -> 0.00 mm
- net /Audio_Codec/JACK_DETECT: track 16.9 -> 21.3 mm
- net +BATT: track 33.9 -> 35.6 mm
- net /Audio_Codec/Jack_MIC_INPUT_1: track 41.2 -> 39.5 mm
- net Net-(D8-Pad1): track 0.00 -> 1.62 mm
- net +3V3: track 218.2 -> 218.9 mm
